File: eps_board/latch.kicad_sch (KiCad schematic)
At the start: 1 part, among them U64 CD4044BDR

Commit message: interim commit
Parts:
- added C1: 100n, Capacitor_SMD:C_0402_1005Metric_Pad0.74x0.62mm_HandSolder, symbol Device:C
Connections:
- net GND: now also C1.2
- net VIN: now also C1.1
Changed lines of the file:
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@@
+		)
+	)
+	(hierarchical_label "GND"
+		(shape input)
+		(at 162.56 78.105 180)
+		(fields_autoplaced yes)
+		(effects
+			(font
+				(size 1.27 1.27)
+			)
+			(justify right)
 		)
 	)
@@
 			)
 			(justify right)
+		)
+	)
+	(hierarchical_label "VIN"
+		(shape input)
+		(at 162.56 70.485 0)
+		(fields_autoplaced yes)
+		(effects
+			(font
+				(size 1.27 1.27)
+			)
+			(justify left)
 		)
 	)
@@
 					(unit 1)
 				)
+			)
+		)
+	)
+	(symbol
+		(lib_id "Device:C")
+		(at 162.56 74.295 0)
+		(unit 1)
+		(exclude_from_sim no)
+		(in_bom yes)
+		(on_board yes)
+		(dnp no)
+		(fields_autoplaced yes)
+		(property "Reference" "C1"
+			(at 166.37 73.0249 0)
+			(effects
+				(font
+					(size 1.27 1.27)
+				)
+				(justify left)
+			)
+		)
+		(property "Value" "100n"
+			(at 166.37 75.5649 0)
+			(effects
+				(font
+					(size 1.27 1.27)
+				)
+				(justify left)
+			)
+		)
+		(property "Footprint" "Capacitor_SMD:C_0402_1005Metric_Pad0.74x0.62mm_HandSolder"
+			(at 163.5252 78.105 0)
+			(effects
+				(font
+					(size 1.27 1.27)
+				)
+				(hide yes)
+			)
+		)
+		(property "Datasheet" "~"
+			(at 162.56 74.295 0)
+			(effects
+				(font
+					(size 1.27 1.27)
+				)
+				(hide yes)
+			)
+		)
+		(property "Description" "Unpolarized capacitor"
+			(at 162.56 74.295 0)
+			(effects
+				(font
+					(size 1.27 1.27)
+				)
+				(hide yes)
+			)
+		)
+		(pin "1"
+		)
+		(pin "2"
+		)
+		(instances
+			(project ""
+				(path "/05170af6-30ef-4c3a-b972-f098085da1bc/cb187d8a-b60d-4ae1-bb3e-5ed90a470051"
+					(reference "C1")
+					(unit 1)
+				)

Commit message: link battery to bus through switch, INA226 on I2C, and level shifter between vbat and MCU
Connections:
- net Q4: now reaches U64.1 (Q4)
- net R4: now reaches U64.14 (R4)
- net S4: now reaches U64.15 (S4)
- no-connect marks 3 -> 0
Changed lines of the file:
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@@
 	(generator_version "8.0")
 	(paper "A4")
-	(no_connect
-		(at 170.815 92.075)
-	)
-	(no_connect
-		(at 109.855 86.995)
-	)
-	(no_connect
-		(at 170.815 89.535)
-	)
 	(hierarchical_label "R1"
 		(shape input)
@@
 		)
 	)
+	(hierarchical_label "Q4"
+		(shape input)
+		(at 109.855 86.995 180)
+		(fields_autoplaced yes)
+		(effects
+			(font
+				(size 1.27 1.27)
+			)
+			(justify right)
+		)
+	)
 	(hierarchical_label "GND"
 		(shape input)
@@
 		(shape input)
 		(at 170.815 97.155 0)
+		(fields_autoplaced yes)
+		(effects
+			(font
+				(size 1.27 1.27)
+			)
+			(justify left)
+		)
+	)
+	(hierarchical_label "R4"
+		(shape input)
+		(at 170.815 92.075 0)
 		(fields_autoplaced yes)
 		(effects
@@
 		)
 	)
+	(hierarchical_label "S4"
+		(shape input)
+		(at 170.815 89.535 0)
+		(fields_autoplaced yes)
+		(effects
+			(font
+				(size 1.27 1.27)
+			)
+			(justify left)
+		)
+	)

Commit message: add 2V8 regulator and switch for SCI cameras, refactor switch/monitors with nonstandard voltage that require level shifting
Parts:
- renumbered C1 to C146, U64 to U68
Changed lines of the file:
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@@
 		(dnp no)
 		(fields_autoplaced yes)
-		(property "Reference" "U64"
+		(property "Reference" "U68"
 			(at 140.335 77.47 0)
 			(effects
@@
 			(project ""
 				(path "/05170af6-30ef-4c3a-b972-f098085da1bc/cb187d8a-b60d-4ae1-bb3e-5ed90a470051"
-					(reference "U64")
+					(reference "U68")
 					(unit 1)
 				)
@@
 		(dnp no)
 		(fields_autoplaced yes)
-		(property "Reference" "C1"
+		(property "Reference" "C146"
 			(at 166.37 73.0249 0)
 			(effects
@@
 			(project ""
 				(path "/05170af6-30ef-4c3a-b972-f098085da1bc/cb187d8a-b60d-4ae1-bb3e-5ed90a470051"
-					(reference "C1")
+					(reference "C146")
 					(unit 1)
 				)
