File: eps_board/boost_regulator_3v3.kicad_sch (KiCad schematic)
At the start: 2 parts

Commit message: add 2V8 regulator and switch for SCI cameras, refactor switch/monitors with nonstandard voltage that require level shifting
Parts:
- renumbered R32 to R147, R33 to R148
Changed lines of the file:
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@@
 		(on_board yes)
 		(dnp no)
-		(property "Reference" "R33"
+		(property "Reference" "R148"
 			(at 131.4449 81.28 90)
 			(effects
@@
 			(project "EPS"
 				(path "/05170af6-30ef-4c3a-b972-f098085da1bc/8033e540-d786-4a4d-a9f2-768a6d82be4a"
-					(reference "R33")
+					(reference "R148")
 					(unit 1)
 				)
 				(path "/05170af6-30ef-4c3a-b972-f098085da1bc/f32018c1-dd23-48ff-aa7d-92319aee7b65"
-					(reference "R118")
+					(reference "R150")
 					(unit 1)
 				)
@@
 		(on_board yes)
 		(dnp no)
-		(property "Reference" "R32"
+		(property "Reference" "R147"
 			(at 120.6499 81.28 90)
 			(effects
@@
 			(project "EPS"
 				(path "/05170af6-30ef-4c3a-b972-f098085da1bc/8033e540-d786-4a4d-a9f2-768a6d82be4a"
-					(reference "R32")
+					(reference "R147")
 					(unit 1)
 				)
 				(path "/05170af6-30ef-4c3a-b972-f098085da1bc/f32018c1-dd23-48ff-aa7d-92319aee7b65"
-					(reference "R117")
+					(reference "R149")
 					(unit 1)
 				)

Commit message: connect all parallel solar panels to mcu
Parts:
- renumbered R147 to R154, R148 to R155
Changed lines of the file:
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@@
 		(on_board yes)
 		(dnp no)
-		(property "Reference" "R148"
+		(property "Reference" "R155"
 			(at 131.4449 81.28 90)
 			(effects
@@
 			(project "EPS"
 				(path "/05170af6-30ef-4c3a-b972-f098085da1bc/8033e540-d786-4a4d-a9f2-768a6d82be4a"
-					(reference "R148")
+					(reference "R155")
 					(unit 1)
 				)
 				(path "/05170af6-30ef-4c3a-b972-f098085da1bc/f32018c1-dd23-48ff-aa7d-92319aee7b65"
-					(reference "R150")
+					(reference "R157")
 					(unit 1)
 				)
@@
 		(on_board yes)
 		(dnp no)
-		(property "Reference" "R147"
+		(property "Reference" "R154"
 			(at 120.6499 81.28 90)
 			(effects
@@
 			(project "EPS"
 				(path "/05170af6-30ef-4c3a-b972-f098085da1bc/8033e540-d786-4a4d-a9f2-768a6d82be4a"
-					(reference "R147")
+					(reference "R154")
 					(unit 1)
 				)
 				(path "/05170af6-30ef-4c3a-b972-f098085da1bc/f32018c1-dd23-48ff-aa7d-92319aee7b65"
-					(reference "R149")
+					(reference "R156")
 					(unit 1)
 				)

Commit message: flip CAN high low around to ease access from the front side
Parts:
- renumbered R154 to R157, R155 to R158
Changed lines of the file:
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@@
 		(on_board yes)
 		(dnp no)
-		(property "Reference" "R155"
+		(property "Reference" "R158"
 			(at 131.4449 81.28 90)
 			(effects
@@
 			(project "EPS"
 				(path "/05170af6-30ef-4c3a-b972-f098085da1bc/8033e540-d786-4a4d-a9f2-768a6d82be4a"
-					(reference "R155")
+					(reference "R158")
 					(unit 1)
 				)
 				(path "/05170af6-30ef-4c3a-b972-f098085da1bc/f32018c1-dd23-48ff-aa7d-92319aee7b65"
-					(reference "R157")
+					(reference "R160")
 					(unit 1)
 				)
@@
 		(on_board yes)
 		(dnp no)
-		(property "Reference" "R154"
+		(property "Reference" "R157"
 			(at 120.6499 81.28 90)
 			(effects
@@
 			(project "EPS"
 				(path "/05170af6-30ef-4c3a-b972-f098085da1bc/8033e540-d786-4a4d-a9f2-768a6d82be4a"
-					(reference "R154")
+					(reference "R157")
 					(unit 1)
 				)
 				(path "/05170af6-30ef-4c3a-b972-f098085da1bc/f32018c1-dd23-48ff-aa7d-92319aee7b65"
-					(reference "R156")
+					(reference "R159")
 					(unit 1)
 				)

Commit message: replace nearly all buck converters with boost buck (missing is 5raw
Parts:
- renumbered R157 to R158, R158 to R159
Changed lines of the file:
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@@
 		(on_board yes)
 		(dnp no)
-		(property "Reference" "R158"
+		(property "Reference" "R159"
 			(at 131.4449 81.28 90)
 			(effects
@@
 			(project "EPS"
 				(path "/05170af6-30ef-4c3a-b972-f098085da1bc/8033e540-d786-4a4d-a9f2-768a6d82be4a"
-					(reference "R158")
+					(reference "R159")
 					(unit 1)
 				)
 				(path "/05170af6-30ef-4c3a-b972-f098085da1bc/f32018c1-dd23-48ff-aa7d-92319aee7b65"
-					(reference "R160")
+					(reference "R161")
 					(unit 1)
 				)
@@
 		(on_board yes)
 		(dnp no)
-		(property "Reference" "R157"
+		(property "Reference" "R158"
 			(at 120.6499 81.28 90)
 			(effects
@@
 			(project "EPS"
 				(path "/05170af6-30ef-4c3a-b972-f098085da1bc/8033e540-d786-4a4d-a9f2-768a6d82be4a"
-					(reference "R157")
+					(reference "R158")
 					(unit 1)
 				)
 				(path "/05170af6-30ef-4c3a-b972-f098085da1bc/f32018c1-dd23-48ff-aa7d-92319aee7b65"
-					(reference "R159")
+					(reference "R160")
 					(unit 1)
 				)
