File: sci_board/cameras.kicad_sch (KiCad schematic)
At the start: 10 parts, among them J7 10051922-2410EHLF, X1 TG2520SMN 24.0000M-ECGNNM0

Commit message: SCI BOM updated
Parts:
- C54: renamed from C57; value 100n -> 100nF; Manufacturer (none) -> Murata; Mfr. # CL10B104KA8NNNC -> (none); Order https://www.digikey.com/product-detail/en/samsung-electro-m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 -> (none); Part Number (none) -> GRM155R61C104KA88D; Tolerance (none) -> 10; Voltage 25V -> 16
- J7: Description_1 0.50mm Flex Connector, VLL Series, 24 Position, Lower Side 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 -> (none); Height 1.5 -> (none); Manufacturer_Name Amphenol Communications Solutions -> (none); Manufacturer_Part_Number 10051922-2410EHLF -> (none)
- JP7, JP8, NT4: now not fitted
- L1, L2: value 1u -> 1uH; Amps (none) -> 3.2; Manufacturer (none) -> Murata; Part Number (none) -> DFE252012P-1R0M=P2
- R30: value 418K6 -> 422K; footprint Resistor_SMD:R_0603_1608Metric_Pad0.98x0.95mm_HandSolder -> Resistor_SMD:R_0402_1005Metric_Pad0.72x0.64mm_HandSolder; Manufacturer (none) -> YAGEO; Note (none) -> Regulator; Part Number (none) -> RC0402FR-07422KL; Tolerance (none) -> 1
- R31: footprint Resistor_SMD:R_0603_1608Metric_Pad0.98x0.95mm_HandSolder -> Resistor_SMD:R_0402_1005Metric_Pad0.72x0.64mm_HandSolder; Manufacturer (none) -> YAGEO; Note (none) -> Regulator; Part Number (none) -> RT0402BRD07182KL; Tolerance (none) -> 0.1
- X1: value TG2520SMN 24.0000M-ECGNNM0 -> 24MHz; footprint Project:TG2520_EPS -> Oscillator:Oscillator_SMD_ECS_2520MV-xxx-xx-4Pin_2.5x2.0mm; symbol Project:TG2520SMN_EPS -> Common:ECS-TXO-2016-33-100-TR; Manufacturer (none) -> ECS; Mfr. # TG-3541CE 32.7680KXA3 -> (none); Order https://www.digikey.com/product-detail/en/epson/TG-3541CE-3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 -> (none); Part Number (none) -> ECS-TXO-2520MV-240-AY-TR
Connections:
- net CLK_OE: now reaches X1.1 (TRI-STATE)
Other:
- moved on the sheet: C54
