File: sci_board/flash.kicad_sch (KiCad schematic)
At the start: 4 parts, among them IC2 MT29F4G01ABAFDWB-IT_F

Commit message: push PC104 bus reorder (no more 5V, 20 lines of 3V3 and 4 switched batt) to system components
Parts:
- IC2: footprint Project:SON127P800X600X65-8N -> SON127P800X600X65-8N
Changed lines of the file:
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@@
 			)
 		)
-		(property "Footprint" "Project:SON127P800X600X65-8N"
+		(property "Footprint" "SON127P800X600X65-8N"
 			(at 106.68 167.945 0)
 			(effects

Commit message: SCI BOM updated
Parts:
- C67: renamed from C70; value 100n -> 100nF; Manufacturer (none) -> Murata; Mfr. # CL10B104KA8NNNC -> (none); Order https://www.digikey.com/product-detail/en/samsung-electro-m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 -> (none); Part Number (none) -> GRM155R61C104KA88D; Tolerance (none) -> 10; Voltage 25V -> 16
- R47, R48: Manufacturer (none) -> YAGEO; Mfr. # RMCF0603FT100K -> (none); Note (none) -> generic pullup/down; Order https://www.digikey.com/en/products/detail/stackpole-electr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 -> (none); Part Number (none) -> RC0402FR-07100KL; Tolerance (none) -> 1
- U30: renamed from IC2; value MT29F4G01ABAFDWB-IT_F -> MT29F4G01ABAFDWB-IT:F TR; footprint SON127P800X600X65-8N -> Common:DFN800X600X65-8N; symbol Project:MT29F4G01ABAFDWB-IT_F -> Common:MT29F4G01ABAFDWB-IT{colon}F; Height 0.65 -> (none); Manufacturer (none) -> Mircon Technology; Manufacturer_Name Micron -> (none); Manufacturer_Part_Number MT29F4G01ABAFDWB-IT:F -> (none); Mouser Part Number 340-359563 -> (none); Mouser Price/Stock https://www.mouser.co.uk/ProductDetail/Micron/MT29F4G01ABAF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 -> (none); Note (none) -> 4Gbit; Part Number (none) -> MT29F4G01ABAFDWB-IT:F TR
Changed lines of the file:
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@@
 		(on_board yes)
 		(dnp no)
-		(property "Reference" "C70"
+		(property "Reference" "C67"
 			(at 143.891 70.5866 0)
 			(effects
@@
 			)
 		)
-		(property "Value" "100n"
+		(property "Value" "100nF"
 			(at 143.891 72.898 0)
 			(effects
@@
 			)
 		)
-		(property "Datasheet" "~"
+		(property "Datasheet" "https://search.murata.co.jp/Ceramy/image/img/A01X/G101/ENG/GRM155R61C104KA88-01.pdf"
 			(at 140.97 71.755 0)
 			(effects
@@
 			)
 		)
-		(property "Mfr. #" "CL10B104KA8NNNC"
-			(at 140.97 71.755 0)
-			(effects
-				(font
-					(size 1.27 1.27)
-				)
-				(hide yes)
-			)
-		)
-		(property "Order" "https://www.digikey.com/product-detail/en/samsung-electro-mechanics/CL10B104KA8NNNC/1276-1006-1-ND/3889092"
-			(at 140.97 71.755 0)
-			(effects
-				(font
-					(size 1.27 1.27)
-				)
-				(hide yes)
-			)
-		)
-		(property "Voltage" "25V"
+		(property "Voltage" "16"
+			(at 140.97 71.755 0)
+			(effects
+				(font
+					(size 1.27 1.27)
+				)
+				(hide yes)
+			)
+		)
+		(property "Manufacturer" "Murata"
+			(at 140.97 71.755 0)
+			(effects
+				(font
+					(size 1.27 1.27)
+				)
+				(hide yes)
+			)
+		)
+		(property "Part Number" "GRM155R61C104KA88D"
+			(at 140.97 71.755 0)
+			(effects
+				(font
+					(size 1.27 1.27)
+				)
+				(hide yes)
+			)
+		)
+		(property "Tolerance" "10"
+			(at 140.97 71.755 0)
+			(effects
+				(font
+					(size 1.27 1.27)
+				)
+				(hide yes)
+			)
+		)
+		(property "Note" ""
 			(at 140.97 71.755 0)
 			(effects
@@
 			(project "sci_board"
 				(path "/b4b2c88d-f6cd-4e60-862d-e21f68728580/1e53aba3-dd28-4d46-80f1-455dd7d8f930"
-					(reference "C70")
+					(reference "C67")
 					(unit 1)
 				)
 				(path "/b4b2c88d-f6cd-4e60-862d-e21f68728580/f6b358f0-c3e5-4f27-97bc-30bc2986accd"
-					(reference "C63")
+					(reference "C60")
 					(unit 1)
 				)
@@
 	)
 	(symbol
-		(lib_id "Project:MT29F4G01ABAFDWB-IT_F")
+		(lib_id "Common:MT29F4G01ABAFDWB-IT{colon}F")
 		(at 72.39 73.025 0)
 		(unit 1)
@@
 		(dnp no)
 		(fields_autoplaced yes)
-		(property "Reference" "IC2"
+		(property "Reference" "U30"
 			(at 91.44 66.04 0)
 			(effects
@@
 			)
 		)
-		(property "Value" "MT29F4G01ABAFDWB-IT_F"
+		(property "Value" "MT29F4G01ABAFDWB-IT:F TR"
 			(at 91.44 68.58 0)
 			(effects
@@
 			)
 		)
-		(property "Footprint" "SON127P800X600X65-8N"
+		(property "Footprint" "Common:DFN800X600X65-8N"
 			(at 106.68 167.945 0)
 			(effects
@@
 			)
 		)
-		(property "Height" "0.65"
-			(at 106.68 467.945 0)
-			(effects
-				(font
-					(size 1.27 1.27)
-				)
-				(justify left top)
-				(hide yes)
-			)
-		)
-		(property "Mouser Part Number" "340-359563"
-			(at 106.68 567.945 0)
-			(effects
-				(font
-					(size 1.27 1.27)
-				)
-				(justify left top)
-				(hide yes)
-			)
-		)
-		(property "Mouser Price/Stock" "https://www.mouser.co.uk/ProductDetail/Micron/MT29F4G01ABAFDWB-ITF?qs=wUXugUrL1qwrjb7To7JPbA%3D%3D"
-			(at 106.68 667.945 0)
-			(effects
-				(font
-					(size 1.27 1.27)
-				)
-				(justify left top)
-				(hide yes)
-			)
-		)
-		(property "Manufacturer_Name" "Micron"
-			(at 106.68 767.945 0)
-			(effects
-				(font
-					(size 1.27 1.27)
-				)
-				(justify left top)
-				(hide yes)
-			)
-		)
-		(property "Manufacturer_Part_Number" "MT29F4G01ABAFDWB-IT:F"
-			(at 106.68 867.945 0)
-			(effects
-				(font
-					(size 1.27 1.27)
-				)
-				(justify left top)
+		(property "Note" "4Gbit"
+			(at 72.39 73.025 0)
+			(effects
+				(font
+					(size 1.27 1.27)
+				)
+				(hide yes)
+			)
+		)
+		(property "Manufacturer" "Mircon Technology"
+			(at 72.39 73.025 0)
+			(effects
+				(font
+					(size 1.27 1.27)
+				)
+				(hide yes)
+			)
+		)
+		(property "Part Number" "MT29F4G01ABAFDWB-IT:F TR"
+			(at 72.39 73.025 0)
+			(effects
+				(font
+					(size 1.27 1.27)
+				)
 				(hide yes)
 			)
@@
 			(project "sci_board"
 				(path "/b4b2c88d-f6cd-4e60-862d-e21f68728580/1e53aba3-dd28-4d46-80f1-455dd7d8f930"
-					(reference "IC2")
+					(reference "U30")
 					(unit 1)
 				)
 				(path "/b4b2c88d-f6cd-4e60-862d-e21f68728580/f6b358f0-c3e5-4f27-97bc-30bc2986accd"
-					(reference "IC1")
+					(reference "U27")
 					(unit 1)
 				)
@@
 			)
 		)
-		(property "Datasheet" "~"
+		(property "Datasheet" "https://www.yageo.com/upload/media/product/products/datasheet/rchip/PYu-RC_Group_51_RoHS_L_12.pdf"
 			(at 53.975 71.755 0)
 			(effects
@@
 			)
 		)
-		(property "Mfr. #" "RMCF0603FT100K"
-			(at 53.975 71.755 0)
-			(effects
-				(font
-					(size 1.27 1.27)
-				)
-				(hide yes)
-			)
-		)
-		(property "Order" "https://www.digikey.com/en/products/detail/stackpole-electronics-inc/RMCF0603FT100K/1761112"
+		(property "Manufacturer" "YAGEO"
+			(at 53.975 71.755 0)
+			(effects
+				(font
+					(size 1.27 1.27)
+				)
+				(hide yes)
+			)
+		)
+		(property "Note" "generic pullup/down"
+			(at 53.975 71.755 0)
+			(effects
+				(font
+					(size 1.27 1.27)
+				)
+				(hide yes)
+			)
+		)
+		(property "Part Number" "RC0402FR-07100KL"
+			(at 53.975 71.755 0)
+			(effects
+				(font
+					(size 1.27 1.27)
+				)
+				(hide yes)
+			)
+		)
+		(property "Tolerance" "1"
 			(at 53.975 71.755 0)
 			(effects
@@
 			)
 		)
-		(property "Datasheet" "~"
+		(property "Datasheet" "https://www.yageo.com/upload/media/product/products/datasheet/rchip/PYu-RC_Group_51_RoHS_L_12.pdf"
 			(at 123.825 71.755 0)
 			(effects
@@
 			)
 		)
-		(property "Mfr. #" "RMCF0603FT100K"
-			(at 123.825 71.755 0)
-			(effects
-				(font
-					(size 1.27 1.27)
-				)
-				(hide yes)
-			)
-		)
-		(property "Order" "https://www.digikey.com/en/products/detail/stackpole-electronics-inc/RMCF0603FT100K/1761112"
-			(at 123.825 71.755 0)
-			(effects
+		(property "Manufacturer" "YAGEO"
+			(at 123.825 71.755 0)
+			(effects
+				(font
+					(size 1.27 1.27)
+				)
+				(hide yes)
+			)
+		)
+		(property "Note" "generic pullup/down"
+			(at 123.825 71.755 0)
+			(effects
+				(font
+					(size 1.27 1.27)
+				)
+				(hide yes)
+			)
+		)
+		(property "Part Number" "RC0402FR-07100KL"
+			(at 123.825 71.755 0)
+			(effects
+				(font
+					(size 1.27 1.27)
+				)
+				(hide yes)
+			)
+		)
+		(property "Tolerance" "1"
+			(at 123.825 71.755 0)
+			(effects

Commit message: reconcile BOMS for AVI. SCI and AUX
Parts:
- C67: Part Number GRM155R61C104KA88D -> GRM155R61E102KA01D; Voltage 16 -> 25
Changed lines of the file:
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@@
 			)
 		)
-		(property "Datasheet" "https://search.murata.co.jp/Ceramy/image/img/A01X/G101/ENG/GRM155R61C104KA88-01.pdf"
+		(property "Datasheet" "https://search.murata.co.jp/Ceramy/image/img/A01X/G101/ENG/GRM155R61E102KA01-01.pdf"
 			(at 140.97 71.755 0)
 			(effects
@@
 			)
 		)
-		(property "Voltage" "16"
+		(property "Voltage" "25"
 			(at 140.97 71.755 0)
 			(effects
@@
 			)
 		)
-		(property "Part Number" "GRM155R61C104KA88D"
+		(property "Part Number" "GRM155R61E102KA01D "
 			(at 140.97 71.755 0)
 			(effects

Commit message: consistency between the different boards
Parts:
- C67: Part Number GRM155R61E102KA01D -> GRM155R61E104KA87D
Changed lines of the file:
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@@
 			)
 		)
-		(property "Datasheet" "https://search.murata.co.jp/Ceramy/image/img/A01X/G101/ENG/GRM155R61E102KA01-01.pdf"
+		(property "Datasheet" "https://search.murata.co.jp/Ceramy/image/img/A01X/G101/ENG/GRM155R61E104KA87-01.pdf"
 			(at 140.97 71.755 0)
 			(effects
@@
 			)
 		)
-		(property "Part Number" "GRM155R61E102KA01D "
+		(property "Part Number" "GRM155R61E104KA87D"
 			(at 140.97 71.755 0)
 			(effects
@@
 			)
 		)
-		(property "Datasheet" ""
+		(property "Datasheet" "https://www.farnell.com/datasheets/3151403.pdf"
 			(at 106.68 267.945 0)
 			(effects

Commit message: add decorations and labels to PCBs
Parts:
- renumbered R47 to R50, R48 to R51
Changed lines of the file:
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@@
 		(on_board yes)
 		(dnp no)
-		(property "Reference" "R47"
+		(property "Reference" "R50"
 			(at 56.515 70.485 0)
 			(effects
@@
 			(project "sci_board"
 				(path "/b4b2c88d-f6cd-4e60-862d-e21f68728580/1e53aba3-dd28-4d46-80f1-455dd7d8f930"
-					(reference "R47")
+					(reference "R50")
 					(unit 1)
 				)
 				(path "/b4b2c88d-f6cd-4e60-862d-e21f68728580/f6b358f0-c3e5-4f27-97bc-30bc2986accd"
-					(reference "R38")
+					(reference "R41")
 					(unit 1)
 				)
@@
 		(on_board yes)
 		(dnp no)
-		(property "Reference" "R48"
+		(property "Reference" "R51"
 			(at 121.285 70.485 0)
 			(effects
@@
 			(project "sci_board"
 				(path "/b4b2c88d-f6cd-4e60-862d-e21f68728580/1e53aba3-dd28-4d46-80f1-455dd7d8f930"
-					(reference "R48")
+					(reference "R51")
 					(unit 1)
 				)
 				(path "/b4b2c88d-f6cd-4e60-862d-e21f68728580/f6b358f0-c3e5-4f27-97bc-30bc2986accd"
-					(reference "R39")
-					(unit 1)
-				)
+					(reference "R42")
+					(unit 1)
+				)

Commit message: use small connectors in corners and on sides for sun sensors and solar cells
Parts:
- added R59: 100K, Resistor_SMD:R_0402_1005Metric_Pad0.72x0.64mm_HandSolder, symbol Device:R
- added R61: 22R, Resistor_SMD:R_0402_1005Metric_Pad0.72x0.64mm_HandSolder, symbol Device:R
- renumbered R50 to R58, R51 to R60, U30 to U29
Connections:
- net SPI_CS: now also R59.2
- net SPI_MISO: now also R61.1; no longer U29.2 (SO/IO1)
- net VDD: now also R59.1
- new net: R61.2, U29.2 (SO/IO1)
Other:
- moved on the sheet: R58

Commit message: detailed power switches moved from EPS to invidual boards, each board only has core and aux bus (and batt if needed) which scales better. Reassign PC104 slots
Parts:
- renumbered C67 to C68, R58 to R65, R59 to R66, R60 to R67, R61 to R68, U29 to U30
Changed lines of the file:
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@@
 		(on_board yes)
 		(dnp no)
-		(property "Reference" "C67"
+		(property "Reference" "C68"
 			(at 143.891 70.5866 0)
 			(effects
@@
 			(project "sci_board"
 				(path "/b4b2c88d-f6cd-4e60-862d-e21f68728580/1e53aba3-dd28-4d46-80f1-455dd7d8f930"
-					(reference "C67")
+					(reference "C68")
 					(unit 1)
 				)
@@
 		(dnp no)
 		(fields_autoplaced yes)
-		(property "Reference" "U29"
+		(property "Reference" "U30"
 			(at 91.44 66.04 0)
 			(effects
@@
 			(project "sci_board"
 				(path "/b4b2c88d-f6cd-4e60-862d-e21f68728580/1e53aba3-dd28-4d46-80f1-455dd7d8f930"
-					(reference "U29")
+					(reference "U30")
 					(unit 1)
 				)
@@
 		(on_board yes)
 		(dnp no)
-		(property "Reference" "R59"
+		(property "Reference" "R66"
 			(at 64.135 63.5 0)
 			(effects
@@
 			(project "sci_board"
 				(path "/b4b2c88d-f6cd-4e60-862d-e21f68728580/1e53aba3-dd28-4d46-80f1-455dd7d8f930"
-					(reference "R59")
+					(reference "R66")
 					(unit 1)
 				)
 				(path "/b4b2c88d-f6cd-4e60-862d-e21f68728580/f6b358f0-c3e5-4f27-97bc-30bc2986accd"
-					(reference "R47")
+					(reference "R50")
 					(unit 1)
 				)
@@
 		(on_board yes)
 		(dnp no)
-		(property "Reference" "R58"
+		(property "Reference" "R65"
 			(at 46.355 63.5 0)
 			(effects
@@
 			(project "sci_board"
 				(path "/b4b2c88d-f6cd-4e60-862d-e21f68728580/1e53aba3-dd28-4d46-80f1-455dd7d8f930"
-					(reference "R58")
+					(reference "R65")
 					(unit 1)
 				)
 				(path "/b4b2c88d-f6cd-4e60-862d-e21f68728580/f6b358f0-c3e5-4f27-97bc-30bc2986accd"
-					(reference "R46")
+					(reference "R49")
 					(unit 1)
 				)
@@
 		(on_board yes)
 		(dnp no)
-		(property "Reference" "R60"
+		(property "Reference" "R67"
 			(at 121.285 70.485 0)
 			(effects
@@
 			(project "sci_board"
 				(path "/b4b2c88d-f6cd-4e60-862d-e21f68728580/1e53aba3-dd28-4d46-80f1-455dd7d8f930"
-					(reference "R60")
+					(reference "R67")
 					(unit 1)
 				)
 				(path "/b4b2c88d-f6cd-4e60-862d-e21f68728580/f6b358f0-c3e5-4f27-97bc-30bc2986accd"
-					(reference "R48")
+					(reference "R51")
 					(unit 1)
 				)
@@
 		(dnp no)
 		(fields_autoplaced yes)
-		(property "Reference" "R61"
+		(property "Reference" "R68"
 			(at 67.945 69.85 90)
 			(effects
@@
 			(project ""
 				(path "/b4b2c88d-f6cd-4e60-862d-e21f68728580/1e53aba3-dd28-4d46-80f1-455dd7d8f930"
-					(reference "R61")
+					(reference "R68")
 					(unit 1)
 				)
 				(path "/b4b2c88d-f6cd-4e60-862d-e21f68728580/f6b358f0-c3e5-4f27-97bc-30bc2986accd"
-					(reference "R49")
-					(unit 1)
-				)
+					(reference "R52")
+					(unit 1)
+				)

Commit message: AUX ready for build SCI: changed camera power switches because the original ones cannot handle voltage below 2.5, we have 1.8!
Parts:
- C66: renamed from C68; Color (none) -> https://search.murata.co.jp/Ceramy/image/img/A01X/G101/ENG/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
- renumbered R65 to R43, R66 to R44, R67 to R45, R68 to R46, U30 to U20
Changed lines of the file:
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@@
 		(on_board yes)
 		(dnp no)
-		(property "Reference" "C68"
+		(property "Reference" "C66"
 			(at 143.891 70.5866 0)
 			(effects
@@
 		)
 		(property "STANDARD" ""
+			(at 140.97 71.755 0)
+			(effects
+				(font
+					(size 1.27 1.27)
+				)
+				(hide yes)
+			)
+		)
+		(property "Color" "https://search.murata.co.jp/Ceramy/image/img/A01X/G101/ENG/GRM155R61E104KA87-01.pdf"
 			(at 140.97 71.755 0)
 			(effects
@@
 			(project "sci_board"
 				(path "/b4b2c88d-f6cd-4e60-862d-e21f68728580/1e53aba3-dd28-4d46-80f1-455dd7d8f930"
-					(reference "C68")
+					(reference "C66")
 					(unit 1)
 				)
 				(path "/b4b2c88d-f6cd-4e60-862d-e21f68728580/f6b358f0-c3e5-4f27-97bc-30bc2986accd"
-					(reference "C59")
+					(reference "C65")
 					(unit 1)
 				)
@@
 		(dnp no)
 		(fields_autoplaced yes)
-		(property "Reference" "U30"
+		(property "Reference" "U20"
 			(at 91.44 66.04 0)
 			(effects
@@
 			(project "sci_board"
 				(path "/b4b2c88d-f6cd-4e60-862d-e21f68728580/1e53aba3-dd28-4d46-80f1-455dd7d8f930"
-					(reference "U30")
+					(reference "U20")
 					(unit 1)
 				)
 				(path "/b4b2c88d-f6cd-4e60-862d-e21f68728580/f6b358f0-c3e5-4f27-97bc-30bc2986accd"
-					(reference "U26")
+					(reference "U19")
 					(unit 1)
 				)
@@
 		(on_board yes)
 		(dnp no)
-		(property "Reference" "R66"
+		(property "Reference" "R44"
 			(at 64.135 63.5 0)
 			(effects
@@
 			(project "sci_board"
 				(path "/b4b2c88d-f6cd-4e60-862d-e21f68728580/1e53aba3-dd28-4d46-80f1-455dd7d8f930"
-					(reference "R66")
+					(reference "R44")
 					(unit 1)
 				)
 				(path "/b4b2c88d-f6cd-4e60-862d-e21f68728580/f6b358f0-c3e5-4f27-97bc-30bc2986accd"
-					(reference "R50")
+					(reference "R40")
 					(unit 1)
 				)
@@
 		(on_board yes)
 		(dnp no)
-		(property "Reference" "R65"
+		(property "Reference" "R43"
 			(at 46.355 63.5 0)
 			(effects
@@
 			(project "sci_board"
 				(path "/b4b2c88d-f6cd-4e60-862d-e21f68728580/1e53aba3-dd28-4d46-80f1-455dd7d8f930"
-					(reference "R65")
+					(reference "R43")
 					(unit 1)
 				)
 				(path "/b4b2c88d-f6cd-4e60-862d-e21f68728580/f6b358f0-c3e5-4f27-97bc-30bc2986accd"
-					(reference "R49")
+					(reference "R39")
 					(unit 1)
 				)
@@
 		(on_board yes)
 		(dnp no)
-		(property "Reference" "R67"
+		(property "Reference" "R45"
 			(at 121.285 70.485 0)
 			(effects
@@
 			(project "sci_board"
 				(path "/b4b2c88d-f6cd-4e60-862d-e21f68728580/1e53aba3-dd28-4d46-80f1-455dd7d8f930"
-					(reference "R67")
+					(reference "R45")
 					(unit 1)
 				)
 				(path "/b4b2c88d-f6cd-4e60-862d-e21f68728580/f6b358f0-c3e5-4f27-97bc-30bc2986accd"
-					(reference "R51")
+					(reference "R41")
 					(unit 1)
 				)
@@
 		(dnp no)
 		(fields_autoplaced yes)
-		(property "Reference" "R68"
+		(property "Reference" "R46"
 			(at 67.945 69.85 90)
 			(effects
@@
 			(project ""
 				(path "/b4b2c88d-f6cd-4e60-862d-e21f68728580/1e53aba3-dd28-4d46-80f1-455dd7d8f930"
-					(reference "R68")
+					(reference "R46")
 					(unit 1)
 				)
 				(path "/b4b2c88d-f6cd-4e60-862d-e21f68728580/f6b358f0-c3e5-4f27-97bc-30bc2986accd"
-					(reference "R52")
-					(unit 1)
-				)
+					(reference "R42")
+					(unit 1)
+				)
