File: sci_board/simple_switch.kicad_sch (KiCad schematic)
At the start: 5 parts, among them U28 TPS22995HQDDCRQ1

Commit message: checking AUX and SCI, tweak BOM
Parts:
- C75: renamed from C87; MANUFACTURER (none) -> Murata; PARTREV (none) -> GRM155R61E104KA87D; Tolerance (none) -> 10
- C76: renamed from C88; MANUFACTURER (none) -> Murata; PARTREV (none) -> GRM188R61E106KA73D; Tolerance (none) -> 10
- C77: renamed from C89; MANUFACTURER (none) -> Murata; PARTREV (none) -> GRM188R61E106KA73D; Tolerance (none) -> 10
- R61: renamed from R63; value 5K1 -> 10K; MANUFACTURER (none) -> YAGEO; PARTREV (none) -> RC0402FR-0710KL; Tolerance (none) -> 1
- U24: renamed from U28; MANUFACTURER (none) -> TI; PARTREV (none) -> TPS22995HQDDCRQ1
Changed lines of the file:
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@@
 		(dnp no)
 		(fields_autoplaced yes)
-		(property "Reference" "C87"
+		(property "Reference" "C75"
 			(at 100.33 100.3299 0)
 			(effects
@@
 			)
 		)
-		(property "Datasheet" "~"
+		(property "Datasheet" "https://search.murata.co.jp/Ceramy/image/img/A01X/G101/ENG/GRM155R61E104KA87-01.pdf"
 			(at 97.155 101.6 0)
 			(effects
@@
 		)
 		(property "Description" "Unpolarized capacitor"
+			(at 97.155 101.6 0)
+			(effects
+				(font
+					(size 1.27 1.27)
+				)
+				(hide yes)
+			)
+		)
+		(property "Tolerance" "10"
+			(at 97.155 101.6 0)
+			(effects
+				(font
+					(size 1.27 1.27)
+				)
+				(hide yes)
+			)
+		)
+		(property "MANUFACTURER" "Murata"
+			(at 97.155 101.6 0)
+			(effects
+				(font
+					(size 1.27 1.27)
+				)
+				(hide yes)
+			)
+		)
+		(property "PARTREV" "GRM155R61E104KA87D"
 			(at 97.155 101.6 0)
 			(effects
@@
 		(dnp no)
 		(fields_autoplaced yes)
-		(property "Reference" "C88"
+		(property "Reference" "C76"
 			(at 115.57 105.4099 0)
 			(effects
@@
 			)
 		)
-		(property "Datasheet" "~"
+		(property "Datasheet" "https://search.murata.co.jp/Ceramy/image/img/A01X/G101/ENG/GRM188R61E106KA73-01.pdf"
 			(at 112.395 106.68 0)
 			(effects
@@
 		)
 		(property "Description" "Unpolarized capacitor"
+			(at 112.395 106.68 0)
+			(effects
+				(font
+					(size 1.27 1.27)
+				)
+				(hide yes)
+			)
+		)
+		(property "Tolerance" "10"
+			(at 112.395 106.68 0)
+			(effects
+				(font
+					(size 1.27 1.27)
+				)
+				(hide yes)
+			)
+		)
+		(property "MANUFACTURER" "Murata"
+			(at 112.395 106.68 0)
+			(effects
+				(font
+					(size 1.27 1.27)
+				)
+				(hide yes)
+			)
+		)
+		(property "PARTREV" "GRM188R61E106KA73D"
 			(at 112.395 106.68 0)
 			(effects
@@
 		(dnp no)
 		(fields_autoplaced yes)
-		(property "Reference" "C89"
+		(property "Reference" "C77"
 			(at 168.275 105.4099 0)
 			(effects
@@
 			)
 		)
-		(property "Datasheet" "~"
+		(property "Datasheet" "https://search.murata.co.jp/Ceramy/image/img/A01X/G101/ENG/GRM188R61E106KA73-01.pdf"
 			(at 165.1 106.68 0)
 			(effects
@@
 		)
 		(property "Description" "Unpolarized capacitor"
+			(at 165.1 106.68 0)
+			(effects
+				(font
+					(size 1.27 1.27)
+				)
+				(hide yes)
+			)
+		)
+		(property "Tolerance" "10"
+			(at 165.1 106.68 0)
+			(effects
+				(font
+					(size 1.27 1.27)
+				)
+				(hide yes)
+			)
+		)
+		(property "MANUFACTURER" "Murata"
+			(at 165.1 106.68 0)
+			(effects
+				(font
+					(size 1.27 1.27)
+				)
+				(hide yes)
+			)
+		)
+		(property "PARTREV" "GRM188R61E106KA73D"
 			(at 165.1 106.68 0)
 			(effects
@@
 		(dnp no)
 		(fields_autoplaced yes)
-		(property "Reference" "R63"
+		(property "Reference" "R61"
 			(at 159.385 91.44 90)
 			(effects
@@
 			)
 		)
-		(property "Value" "5K1"
+		(property "Value" "10K"
 			(at 159.385 93.98 90)
 			(effects
@@
 			)
 		)
-		(property "Datasheet" "~"
+		(property "Datasheet" "https://www.yageo.com/upload/media/product/products/datasheet/rchip/PYu-RC_Group_51_RoHS_L_12.pdf"
 			(at 159.385 97.79 0)
 			(effects
@@
 		)
 		(property "Description" "Resistor"
+			(at 159.385 97.79 0)
+			(effects
+				(font
+					(size 1.27 1.27)
+				)
+				(hide yes)
+			)
+		)
+		(property "Tolerance" "1"
+			(at 159.385 97.79 0)
+			(effects
+				(font
+					(size 1.27 1.27)
+				)
+				(hide yes)
+			)
+		)
+		(property "MANUFACTURER" "YAGEO"
+			(at 159.385 97.79 0)
+			(effects
+				(font
+					(size 1.27 1.27)
+				)
+				(hide yes)
+			)
+		)
+		(property "PARTREV" "RC0402FR-0710KL"
 			(at 159.385 97.79 0)
 			(effects
@@
 			(project "sci_board"
 				(path "/b4b2c88d-f6cd-4e60-862d-e21f68728580/5e5b27f8-7a4c-45d0-95f8-aff71797fcd3/09c52fbd-a66a-456f-a3b3-a583ddfe7084/03862b24-5072-4f26-9a88-8ef091cc932e"
-					(reference "R59")
+					(reference "R61")
 					(unit 1)
 				)
 				(path "/b4b2c88d-f6cd-4e60-862d-e21f68728580/5e5b27f8-7a4c-45d0-95f8-aff71797fcd3/09c52fbd-a66a-456f-a3b3-a583ddfe7084/98fe85ae-88e3-40b1-83ee-8d89343e2a54"
+					(reference "R64")
+					(unit 1)
+				)
+				(path "/b4b2c88d-f6cd-4e60-862d-e21f68728580/5e5b27f8-7a4c-45d0-95f8-aff71797fcd3/09c52fbd-a66a-456f-a3b3-a583ddfe7084/b68dd023-ac10-4845-8ce1-1e6a3ce1aca0"
+					(reference "R74")
+					(unit 1)
+				)
+				(path "/b4b2c88d-f6cd-4e60-862d-e21f68728580/5e5b27f8-7a4c-45d0-95f8-aff71797fcd3/3113fc14-4b9f-4852-8ddb-4c564d791d7f/03862b24-5072-4f26-9a88-8ef091cc932e"
+					(reference "R31")
+					(unit 1)
+				)
+				(path "/b4b2c88d-f6cd-4e60-862d-e21f68728580/5e5b27f8-7a4c-45d0-95f8-aff71797fcd3/3113fc14-4b9f-4852-8ddb-4c564d791d7f/98fe85ae-88e3-40b1-83ee-8d89343e2a54"
 					(reference "R62")
 					(unit 1)
 				)
-				(path "/b4b2c88d-f6cd-4e60-862d-e21f68728580/5e5b27f8-7a4c-45d0-95f8-aff71797fcd3/09c52fbd-a66a-456f-a3b3-a583ddfe7084/b68dd023-ac10-4845-8ce1-1e6a3ce1aca0"
-					(reference "R72")
-					(unit 1)
-				)
-				(path "/b4b2c88d-f6cd-4e60-862d-e21f68728580/5e5b27f8-7a4c-45d0-95f8-aff71797fcd3/3113fc14-4b9f-4852-8ddb-4c564d791d7f/03862b24-5072-4f26-9a88-8ef091cc932e"
-					(reference "R29")
-					(unit 1)
-				)
-				(path "/b4b2c88d-f6cd-4e60-862d-e21f68728580/5e5b27f8-7a4c-45d0-95f8-aff71797fcd3/3113fc14-4b9f-4852-8ddb-4c564d791d7f/98fe85ae-88e3-40b1-83ee-8d89343e2a54"
-					(reference "R60")
-					(unit 1)
-				)
 				(path "/b4b2c88d-f6cd-4e60-862d-e21f68728580/5e5b27f8-7a4c-45d0-95f8-aff71797fcd3/3113fc14-4b9f-4852-8ddb-4c564d791d7f/b68dd023-ac10-4845-8ce1-1e6a3ce1aca0"
+					(reference "R65")
+					(unit 1)
+				)
+				(path "/b4b2c88d-f6cd-4e60-862d-e21f68728580/5e5b27f8-7a4c-45d0-95f8-aff71797fcd3/df99859d-8e37-4f21-a1c5-637d9e74b907/03862b24-5072-4f26-9a88-8ef091cc932e"
+					(reference "R34")
+					(unit 1)
+				)
+				(path "/b4b2c88d-f6cd-4e60-862d-e21f68728580/5e5b27f8-7a4c-45d0-95f8-aff71797fcd3/df99859d-8e37-4f21-a1c5-637d9e74b907/98fe85ae-88e3-40b1-83ee-8d89343e2a54"
 					(reference "R63")
 					(unit 1)
 				)
-				(path "/b4b2c88d-f6cd-4e60-862d-e21f68728580/5e5b27f8-7a4c-45d0-95f8-aff71797fcd3/df99859d-8e37-4f21-a1c5-637d9e74b907/03862b24-5072-4f26-9a88-8ef091cc932e"
-					(reference "R32")
-					(unit 1)
-				)
-				(path "/b4b2c88d-f6cd-4e60-862d-e21f68728580/5e5b27f8-7a4c-45d0-95f8-aff71797fcd3/df99859d-8e37-4f21-a1c5-637d9e74b907/98fe85ae-88e3-40b1-83ee-8d89343e2a54"
-					(reference "R61")
-					(unit 1)
-				)
 				(path "/b4b2c88d-f6cd-4e60-862d-e21f68728580/5e5b27f8-7a4c-45d0-95f8-aff71797fcd3/df99859d-8e37-4f21-a1c5-637d9e74b907/b68dd023-ac10-4845-8ce1-1e6a3ce1aca0"
-					(reference "R73")
+					(reference "R75")
 					(unit 1)
 				)
@@
 		(dnp no)
 		(fields_autoplaced yes)
-		(property "Reference" "U28"
+		(property "Reference" "U24"
 			(at 141.605 90.17 0)
 			(effects
@@
 			)
 		)
-		(property "Description" ""
+		(property "Description" "Load Switch"
 			(at 141.605 99.06 0)
 			(effects
+				(font
+					(size 1.27 1.27)
+				)
+				(hide yes)
+			)
+		)
+		(property "MANUFACTURER" "TI"
+			(at 141.605 99.06 0)
+			(effects
+				(font
+					(size 1.27 1.27)
+				)
+				(hide yes)
+			)
+		)
+		(property "PARTREV" "TPS22995HQDDCRQ1"
+			(at 141.605 99.06 0)
+			(effects

Commit message: check BOM and footprints for SCI and AUX
Parts:
- R61: Note (none) -> slew rate
- U24: footprint Common:SOT-23-6 -> Common:TSOT-23-6
Changed lines of the file:
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@@
+			)
+		)
+		(property "Note" "slew rate"
+			(at 159.385 97.79 0)
+			(effects
+				(font
+					(size 1.27 1.27)
+				)
+				(hide yes)
 			)
 		)
@@
 			)
 		)
-		(property "Footprint" "Common:SOT-23-6"
+		(property "Footprint" "Common:TSOT-23-6"
 			(at 141.605 99.06 0)
 			(effects
