File: sci_board/power_regulator_mp3416.kicad_sch (KiCad schematic)
At the start: 5 parts, among them U54 TPS631000DRLR

Commit message: AUX ready for build SCI: changed camera power switches because the original ones cannot handle voltage below 2.5, we have 1.8!
Parts:
- C112, C113: Temperture Coefficient (none) -> X5R
- C114: Color (none) -> https://mm.digikey.com/Volume0/opasdata/d220001/medias/docu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; Temperture Coefficient (none) -> X5R
Changed lines of the file:
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@@
+			)
+		)
+		(property "Temperture Coefficient" ""
+			(at 72.39 132.08 0)
+			(effects
+				(font
+					(size 1.27 1.27)
+				)
+				(hide yes)
 			)
 		)
@@
 		(property "STANDARD" ""
 			(at 72.39 132.08 0)
-			(effects
-				(font
-					(size 1.27 1.27)
-				)
-				(hide yes)
-			)
-		)
-		(property "Manufactorer" ""
-			(at 0 264.16 0)
 			(effects
 				(font
@@
 			(project "sci_board"
 				(path "/b4b2c88d-f6cd-4e60-862d-e21f68728580/5e5b27f8-7a4c-45d0-95f8-aff71797fcd3/2f5a2990-2dc0-472a-952a-1bfd830a3aba"
-					(reference "U28")
+					(reference "U22")
 					(unit 1)
 				)
 				(path "/b4b2c88d-f6cd-4e60-862d-e21f68728580/5e5b27f8-7a4c-45d0-95f8-aff71797fcd3/7fde3d19-3e51-4869-ba44-af6d0a67b762"
-					(reference "U27")
+					(reference "U21")
 					(unit 1)
 				)
@@
 			)
 		)
+		(property "Temperture Coefficient" ""
+			(at 128.905 135.89 0)
+			(effects
+				(font
+					(size 1.27 1.27)
+				)
+				(hide yes)
+			)
+		)
 		(property "MANUFACTURER" ""
 			(at 128.905 135.89 0)
@@
 		(property "STANDARD" ""
 			(at 128.905 135.89 0)
-			(effects
-				(font
-					(size 1.27 1.27)
-				)
-				(hide yes)
-			)
-		)
-		(property "Manufactorer" ""
-			(at 0 271.78 0)
 			(effects
 				(font
@@
 			(project "sci_board"
 				(path "/b4b2c88d-f6cd-4e60-862d-e21f68728580/5e5b27f8-7a4c-45d0-95f8-aff71797fcd3/2f5a2990-2dc0-472a-952a-1bfd830a3aba"
-					(reference "R55")
+					(reference "R49")
 					(unit 1)
 				)
 				(path "/b4b2c88d-f6cd-4e60-862d-e21f68728580/5e5b27f8-7a4c-45d0-95f8-aff71797fcd3/7fde3d19-3e51-4869-ba44-af6d0a67b762"
-					(reference "R53")
+					(reference "R47")
 					(unit 1)
 				)
@@
 			)
 		)
+		(property "Temperture Coefficient" "X5R"
+			(at 72.39 143.51 0)
+			(effects
+				(font
+					(size 1.27 1.27)
+				)
+				(hide yes)
+			)
+		)
 		(property "MANUFACTURER" ""
 			(at 72.39 143.51 0)
@@
 			)
 		)
-		(property "Manufactorer" ""
-			(at 0 287.02 0)
+		(property "Color" "https://mm.digikey.com/Volume0/opasdata/d220001/medias/docus/6223/Chip_Multilayer_CC_CAT_Rev21.pdf"
+			(at 72.39 143.51 0)
 			(effects
 				(font
@@
 			(project "sci_board"
 				(path "/b4b2c88d-f6cd-4e60-862d-e21f68728580/5e5b27f8-7a4c-45d0-95f8-aff71797fcd3/2f5a2990-2dc0-472a-952a-1bfd830a3aba"
-					(reference "C66")
+					(reference "C73")
 					(unit 1)
 				)
 				(path "/b4b2c88d-f6cd-4e60-862d-e21f68728580/5e5b27f8-7a4c-45d0-95f8-aff71797fcd3/7fde3d19-3e51-4869-ba44-af6d0a67b762"
-					(reference "C62")
+					(reference "C69")
 					(unit 1)
 				)
@@
 			)
 		)
+		(property "Temperture Coefficient" "X5R"
+			(at 49.53 139.7 0)
+			(effects
+				(font
+					(size 1.27 1.27)
+				)
+				(hide yes)
+			)
+		)
 		(property "MANUFACTURER" ""
 			(at 49.53 139.7 0)
@@
 		(property "STANDARD" ""
 			(at 49.53 139.7 0)
-			(effects
-				(font
-					(size 1.27 1.27)
-				)
-				(hide yes)
-			)
-		)
-		(property "Manufactorer" ""
-			(at 99.06 279.4 0)
 			(effects
 				(font
@@
 			(project "sci_board"
 				(path "/b4b2c88d-f6cd-4e60-862d-e21f68728580/5e5b27f8-7a4c-45d0-95f8-aff71797fcd3/2f5a2990-2dc0-472a-952a-1bfd830a3aba"
-					(reference "C64")
+					(reference "C71")
 					(unit 1)
 				)
 				(path "/b4b2c88d-f6cd-4e60-862d-e21f68728580/5e5b27f8-7a4c-45d0-95f8-aff71797fcd3/7fde3d19-3e51-4869-ba44-af6d0a67b762"
-					(reference "C60")
+					(reference "C67")
 					(unit 1)
 				)
@@
 			)
 		)
+		(property "Temperture Coefficient" "X5R"
+			(at 59.69 139.7 0)
+			(effects
+				(font
+					(size 1.27 1.27)
+				)
+				(hide yes)
+			)
+		)
 		(property "MANUFACTURER" ""
 			(at 59.69 139.7 0)
@@
 		(property "STANDARD" ""
 			(at 59.69 139.7 0)
-			(effects
-				(font
-					(size 1.27 1.27)
-				)
-				(hide yes)
-			)
-		)
-		(property "Manufactorer" ""
-			(at 119.38 279.4 0)
 			(effects
 				(font
@@
 			(project "sci_board"
 				(path "/b4b2c88d-f6cd-4e60-862d-e21f68728580/5e5b27f8-7a4c-45d0-95f8-aff71797fcd3/2f5a2990-2dc0-472a-952a-1bfd830a3aba"
-					(reference "C65")
+					(reference "C72")
 					(unit 1)
 				)
 				(path "/b4b2c88d-f6cd-4e60-862d-e21f68728580/5e5b27f8-7a4c-45d0-95f8-aff71797fcd3/7fde3d19-3e51-4869-ba44-af6d0a67b762"
-					(reference "C61")
-					(unit 1)
-				)
+					(reference "C68")
+					(unit 1)
+				)

Commit message: checking AUX and SCI, tweak BOM
Parts:
- C112, C113: MANUFACTURER (none) -> Murata; Manufacturer Murata -> (none); PARTREV (none) -> GRM21BR61A476ME15K; Part Number GRM21BR61A476ME15K -> (none)
- C114: Color https://mm.digikey.com/Volume0/opasdata/d220001/medias/docu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 -> (none); MANUFACTURER (none) -> Murata; Manufacturer Murata -> (none); PARTREV (none) -> GRM188R61A226ME15D; Part Number GRM188R61A226ME15D -> (none)
- R143: MANUFACTURER (none) -> YAGEO; Manufacturer YAGEO -> (none); PARTREV (none) -> RC0402FR-0791KL; Part Number RC0402FR-0791KL -> (none)
- U54: MANUFACTURER (none) -> TI; Manufacturer TI -> (none); PARTREV (none) -> TPS631000DRLR; Part Number TPS631000DRLR -> (none)
Changed lines of the file:
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@@
-			)
-		)
-		(property "Manufacturer" "TI"
-			(at 72.39 132.08 0)
-			(effects
-				(font
-					(size 1.27 1.27)
-				)
-				(hide yes)
-			)
-		)
-		(property "Part Number" "TPS631000DRLR"
-			(at 72.39 132.08 0)
-			(effects
-				(font
-					(size 1.27 1.27)
-				)
-				(hide yes)
 			)
 		)
@@
 			)
 		)
-		(property "MANUFACTURER" ""
+		(property "MANUFACTURER" "TI"
 			(at 72.39 132.08 0)
 			(effects
@@
 			)
 		)
-		(property "PARTREV" ""
+		(property "PARTREV" "TPS631000DRLR"
 			(at 72.39 132.08 0)
 			(effects
@@
 			)
 		)
-		(property "Datasheet" "https://www.yageo.com/upload/media/product/app/datasheet/rchip/pyu-rt_1-to-0.01_rohs_l.pdf"
+		(property "Datasheet" "https://www.yageo.com/upload/media/product/products/datasheet/rchip/PYu-RC_Group_51_RoHS_L_12.pdf"
 			(at 128.905 135.89 0)
 			(effects
@@
 			)
 		)
-		(property "Manufacturer" "YAGEO"
-			(at 128.905 135.89 0)
-			(effects
-				(font
-					(size 1.27 1.27)
-				)
-				(hide yes)
-			)
-		)
-		(property "Part Number" "RC0402FR-0791KL "
-			(at 128.905 135.89 0)
-			(effects
-				(font
-					(size 1.27 1.27)
-				)
-				(hide yes)
-			)
-		)
 		(property "Tolerance" "1"
 			(at 128.905 135.89 0)
@@
 			)
 		)
-		(property "MANUFACTURER" ""
+		(property "MANUFACTURER" "YAGEO"
 			(at 128.905 135.89 0)
 			(effects
@@
 			)
 		)
-		(property "PARTREV" ""
+		(property "PARTREV" "RC0402FR-0791KL "
 			(at 128.905 135.89 0)
 			(effects
@@
 			(project "sci_board"
 				(path "/b4b2c88d-f6cd-4e60-862d-e21f68728580/5e5b27f8-7a4c-45d0-95f8-aff71797fcd3/2f5a2990-2dc0-472a-952a-1bfd830a3aba"
+					(reference "R51")
+					(unit 1)
+				)
+				(path "/b4b2c88d-f6cd-4e60-862d-e21f68728580/5e5b27f8-7a4c-45d0-95f8-aff71797fcd3/7fde3d19-3e51-4869-ba44-af6d0a67b762"
 					(reference "R49")
-					(unit 1)
-				)
-				(path "/b4b2c88d-f6cd-4e60-862d-e21f68728580/5e5b27f8-7a4c-45d0-95f8-aff71797fcd3/7fde3d19-3e51-4869-ba44-af6d0a67b762"
-					(reference "R47")
 					(unit 1)
 				)
@@
 			)
 		)
-		(property "Manufacturer" "Murata"
-			(at 72.39 143.51 0)
-			(effects
-				(font
-					(size 1.27 1.27)
-				)
-				(hide yes)
-			)
-		)
-		(property "Part Number" "GRM188R61A226ME15D"
-			(at 72.39 143.51 0)
-			(effects
-				(font
-					(size 1.27 1.27)
-				)
-				(hide yes)
-			)
-		)
 		(property "Tolerance" "20"
 			(at 72.39 143.51 0)
@@
 			)
 		)
-		(property "MANUFACTURER" ""
+		(property "MANUFACTURER" "Murata"
 			(at 72.39 143.51 0)
 			(effects
@@
 			)
 		)
-		(property "PARTREV" ""
+		(property "PARTREV" "GRM188R61A226ME15D"
 			(at 72.39 143.51 0)
 			(effects
@@
 			)
 		)
-		(property "Color" "https://mm.digikey.com/Volume0/opasdata/d220001/medias/docus/6223/Chip_Multilayer_CC_CAT_Rev21.pdf"
+		(property "Color" ""
 			(at 72.39 143.51 0)
 			(effects
@@
 			(project "aux_board"
 				(path "/85134265-2435-454a-99c4-e49d8e69c5c2/180ab09f-8202-4a23-a970-ad767a3abcbf"
-					(reference "C40")
+					(reference "C41")
 					(unit 1)
 				)
 				(path "/85134265-2435-454a-99c4-e49d8e69c5c2/21705b31-e71e-4020-a43e-3303465bf5fd"
-					(reference "C34")
+					(reference "C35")
 					(unit 1)
 				)
 				(path "/85134265-2435-454a-99c4-e49d8e69c5c2/89862a4b-05be-454b-946e-6c4f5a4f01a7"
-					(reference "C43")
+					(reference "C44")
 					(unit 1)
 				)
 				(path "/85134265-2435-454a-99c4-e49d8e69c5c2/c6f75225-fda9-49b7-af41-6a3b5c80f9a2"
-					(reference "C37")
+					(reference "C38")
 					(unit 1)
 				)
@@
 			)
 		)
-		(property "Manufacturer" "Murata"
-			(at 49.53 139.7 0)
-			(effects
-				(font
-					(size 1.27 1.27)
-				)
-				(hide yes)
-			)
-		)
-		(property "Part Number" "GRM21BR61A476ME15K"
-			(at 49.53 139.7 0)
-			(effects
-				(font
-					(size 1.27 1.27)
-				)
-				(hide yes)
-			)
-		)
 		(property "Tolerance" "20"
 			(at 49.53 139.7 0)
@@
 			)
 		)
-		(property "MANUFACTURER" ""
+		(property "MANUFACTURER" "Murata"
 			(at 49.53 139.7 0)
 			(effects
@@
 			)
 		)
-		(property "PARTREV" ""
+		(property "PARTREV" "GRM21BR61A476ME15K"
 			(at 49.53 139.7 0)
 			(effects
@@
 			(project "aux_board"
 				(path "/85134265-2435-454a-99c4-e49d8e69c5c2/180ab09f-8202-4a23-a970-ad767a3abcbf"
-					(reference "C38")
+					(reference "C39")
 					(unit 1)
 				)
 				(path "/85134265-2435-454a-99c4-e49d8e69c5c2/21705b31-e71e-4020-a43e-3303465bf5fd"
-					(reference "C32")
+					(reference "C33")
 					(unit 1)
 				)
 				(path "/85134265-2435-454a-99c4-e49d8e69c5c2/89862a4b-05be-454b-946e-6c4f5a4f01a7"
-					(reference "C41")
+					(reference "C42")
 					(unit 1)
 				)
 				(path "/85134265-2435-454a-99c4-e49d8e69c5c2/c6f75225-fda9-49b7-af41-6a3b5c80f9a2"
-					(reference "C35")
+					(reference "C36")
 					(unit 1)
 				)
@@
 			)
 		)
-		(property "Manufacturer" "Murata"
-			(at 59.69 139.7 0)
-			(effects
-				(font
-					(size 1.27 1.27)
-				)
-				(hide yes)
-			)
-		)
-		(property "Part Number" "GRM21BR61A476ME15K"
-			(at 59.69 139.7 0)
-			(effects
-				(font
-					(size 1.27 1.27)
-				)
-				(hide yes)
-			)
-		)
 		(property "Tolerance" "20"
 			(at 59.69 139.7 0)
@@
 			)
 		)
-		(property "MANUFACTURER" ""
+		(property "MANUFACTURER" "Murata"
 			(at 59.69 139.7 0)
 			(effects
@@
 			)
 		)
-		(property "PARTREV" ""
+		(property "PARTREV" "GRM21BR61A476ME15K"
 			(at 59.69 139.7 0)
 			(effects
@@
 			(project "aux_board"
 				(path "/85134265-2435-454a-99c4-e49d8e69c5c2/180ab09f-8202-4a23-a970-ad767a3abcbf"
-					(reference "C39")
+					(reference "C40")
 					(unit 1)
 				)
 				(path "/85134265-2435-454a-99c4-e49d8e69c5c2/21705b31-e71e-4020-a43e-3303465bf5fd"
-					(reference "C33")
+					(reference "C34")
 					(unit 1)
 				)
 				(path "/85134265-2435-454a-99c4-e49d8e69c5c2/89862a4b-05be-454b-946e-6c4f5a4f01a7"
-					(reference "C42")
+					(reference "C43")
 					(unit 1)
 				)
 				(path "/85134265-2435-454a-99c4-e49d8e69c5c2/c6f75225-fda9-49b7-af41-6a3b5c80f9a2"
-					(reference "C36")
-					(unit 1)
-				)
+					(reference "C37")
+					(unit 1)
+				)

Commit message: check BOM and footprints for SCI and AUX
Parts:
- R143: Note regulator -> Regulator
Changed lines of the file:
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@@
 			)
 		)
-		(property "Note" "regulator"
+		(property "Note" "Regulator"
 			(at 128.905 135.89 0)
 			(effects

Commit message: SCI power switch: change I2C expander to manufacturer recommended footprint to enable production with PCBWAY
Parts:
- renumbered R143 to R141
Changed lines of the file:
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@@
 		(on_board yes)
 		(dnp no)
-		(property "Reference" "R143"
+		(property "Reference" "R141"
 			(at 130.81 134.62 0)
 			(effects
@@
 			(project "EPS"
 				(path "/05170af6-30ef-4c3a-b972-f098085da1bc/87930429-600a-4d20-9691-47e157ed6d1e"
-					(reference "R143")
+					(reference "R141")
 					(unit 1)
 				)
 				(path "/05170af6-30ef-4c3a-b972-f098085da1bc/e1d2fe3b-9ba5-4366-9cc3-67e5d340cfc0/4b0ead8a-9397-4a83-9955-863b935c5b9c"
-					(reference "R39")
+					(reference "R37")
 					(unit 1)
 				)
 				(path "/05170af6-30ef-4c3a-b972-f098085da1bc/e1d2fe3b-9ba5-4366-9cc3-67e5d340cfc0/744250af-b7e3-4edd-bc04-e013bd519440"
-					(reference "R45")
+					(reference "R43")
 					(unit 1)
 				)
 				(path "/05170af6-30ef-4c3a-b972-f098085da1bc/e1d2fe3b-9ba5-4366-9cc3-67e5d340cfc0/772eb76d-f57b-4f14-8409-6548bfc340ef"
-					(reference "R44")
+					(reference "R42")
 					(unit 1)
 				)

Commit message: full science board with camera switches
Parts:
- renumbered C112 to C82, C113 to C83, C114 to C84, R141 to R52, U54 to U23
Changed lines of the file:
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@@
 (kicad_sch
-	(version 20231120)
+	(version 20250114)
 	(generator "eeschema")
-	(generator_version "8.0")
+	(generator_version "9.0")
 	(paper "A4")
 	(junction
@@
 		(shape input)
 		(at 128.905 139.7 0)
-		(fields_autoplaced yes)
 		(effects
 			(font
@@
 		(shape input)
 		(at 49.53 144.78 180)
-		(fields_autoplaced yes)
 		(effects
 			(font
@@
 		(shape input)
 		(at 113.03 137.16 0)
-		(fields_autoplaced yes)
 		(effects
 			(font
@@
 		(shape input)
 		(at 128.905 132.08 0)
-		(fields_autoplaced yes)
 		(effects
 			(font
@@
 		(shape input)
 		(at 72.39 147.32 180)
-		(fields_autoplaced yes)
 		(effects
 			(font
@@
 		(shape input)
 		(at 72.39 139.7 180)
-		(fields_autoplaced yes)
 		(effects
 			(font
@@
 		(shape output)
 		(at 49.53 132.08 180)
-		(fields_autoplaced yes)
 		(effects
 			(font
@@
 		(shape input)
 		(at 128.905 127 0)
-		(fields_autoplaced yes)
 		(effects
 			(font
@@
 		(shape input)
 		(at 72.39 137.16 180)
-		(fields_autoplaced yes)
 		(effects
 			(font
@@
 		(shape input)
 		(at 113.03 134.62 0)
-		(fields_autoplaced yes)
 		(effects
 			(font
@@
 		(shape input)
 		(at 113.03 139.7 0)
-		(fields_autoplaced yes)
 		(effects
 			(font
@@
 		(shape input)
 		(at 72.39 134.62 180)
-		(fields_autoplaced yes)
 		(effects
 			(font
@@
 		(shape output)
 		(at 128.905 127 180)
-		(fields_autoplaced yes)
 		(effects
 			(font
@@
 		(dnp no)
 		(fields_autoplaced yes)
-		(property "Reference" "U54"
+		(property "Reference" "U23"
 			(at 92.71 121.92 0)
 			(effects
@@
 			(project "sci_board"
 				(path "/b4b2c88d-f6cd-4e60-862d-e21f68728580/5e5b27f8-7a4c-45d0-95f8-aff71797fcd3/2f5a2990-2dc0-472a-952a-1bfd830a3aba"
-					(reference "U22")
+					(reference "U24")
 					(unit 1)
 				)
 				(path "/b4b2c88d-f6cd-4e60-862d-e21f68728580/5e5b27f8-7a4c-45d0-95f8-aff71797fcd3/7fde3d19-3e51-4869-ba44-af6d0a67b762"
-					(reference "U21")
+					(reference "U23")
 					(unit 1)
 				)
@@
 		(on_board yes)
 		(dnp no)
-		(property "Reference" "R141"
+		(property "Reference" "R52"
 			(at 130.81 134.62 0)
 			(effects
@@
 			)
 		)
-		(property "Datasheet" "https://www.yageo.com/upload/media/product/products/datasheet/rchip/PYu-RC_Group_51_RoHS_L_12.pdf"
+		(property "Datasheet" "~"
 			(at 128.905 135.89 0)
 			(effects
@@
 			)
 		)
-		(property "Description" "Resistor"
+		(property "Description" "Resistor, small symbol"
 			(at 128.905 135.89 0)
 			(effects
@@
 			(project "sci_board"
 				(path "/b4b2c88d-f6cd-4e60-862d-e21f68728580/5e5b27f8-7a4c-45d0-95f8-aff71797fcd3/2f5a2990-2dc0-472a-952a-1bfd830a3aba"
-					(reference "R51")
+					(reference "R54")
 					(unit 1)
 				)
 				(path "/b4b2c88d-f6cd-4e60-862d-e21f68728580/5e5b27f8-7a4c-45d0-95f8-aff71797fcd3/7fde3d19-3e51-4869-ba44-af6d0a67b762"
-					(reference "R49")
+					(reference "R52")
 					(unit 1)
 				)
@@
 		(on_board yes)
 		(dnp no)
-		(property "Reference" "C114"
+		(property "Reference" "C84"
 			(at 74.93 142.24 0)
 			(effects
@@
 			(project "sci_board"
 				(path "/b4b2c88d-f6cd-4e60-862d-e21f68728580/5e5b27f8-7a4c-45d0-95f8-aff71797fcd3/2f5a2990-2dc0-472a-952a-1bfd830a3aba"
-					(reference "C73")
+					(reference "C88")
 					(unit 1)
 				)
 				(path "/b4b2c88d-f6cd-4e60-862d-e21f68728580/5e5b27f8-7a4c-45d0-95f8-aff71797fcd3/7fde3d19-3e51-4869-ba44-af6d0a67b762"
-					(reference "C69")
+					(reference "C84")
 					(unit 1)
 				)
@@
 		(on_board yes)
 		(dnp no)
-		(property "Reference" "C112"
+		(property "Reference" "C82"
 			(at 53.34 138.4299 0)
 			(effects
@@
 			(project "sci_board"
 				(path "/b4b2c88d-f6cd-4e60-862d-e21f68728580/5e5b27f8-7a4c-45d0-95f8-aff71797fcd3/2f5a2990-2dc0-472a-952a-1bfd830a3aba"
-					(reference "C71")
+					(reference "C86")
 					(unit 1)
 				)
 				(path "/b4b2c88d-f6cd-4e60-862d-e21f68728580/5e5b27f8-7a4c-45d0-95f8-aff71797fcd3/7fde3d19-3e51-4869-ba44-af6d0a67b762"
-					(reference "C67")
+					(reference "C82")
 					(unit 1)
 				)
@@
 		(on_board yes)
 		(dnp no)
-		(property "Reference" "C113"
+		(property "Reference" "C83"
 			(at 46.355 138.43 0)
 			(effects
@@
 			(project "sci_board"
 				(path "/b4b2c88d-f6cd-4e60-862d-e21f68728580/5e5b27f8-7a4c-45d0-95f8-aff71797fcd3/2f5a2990-2dc0-472a-952a-1bfd830a3aba"
-					(reference "C72")
+					(reference "C87")
 					(unit 1)
 				)
 				(path "/b4b2c88d-f6cd-4e60-862d-e21f68728580/5e5b27f8-7a4c-45d0-95f8-aff71797fcd3/7fde3d19-3e51-4869-ba44-af6d0a67b762"
-					(reference "C68")
-					(unit 1)
-				)
+					(reference "C83")
+					(unit 1)
+				)

Commit message: cleanup and bom
Parts:
- renumbered R52 to R50
Changed lines of the file:
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@@
 		(on_board yes)
 		(dnp no)
-		(property "Reference" "R52"
+		(property "Reference" "R50"
 			(at 130.81 134.62 0)
 			(effects
@@
 			)
 		)
-		(property "Datasheet" "~"
+		(property "Datasheet" "https://www.yageo.com/upload/media/product/app/datasheet/rchip/pyu-rt_1-to-0.01_rohs_l.pdf"
 			(at 128.905 135.89 0)
 			(effects
@@
 			(project "sci_board"
 				(path "/b4b2c88d-f6cd-4e60-862d-e21f68728580/5e5b27f8-7a4c-45d0-95f8-aff71797fcd3/2f5a2990-2dc0-472a-952a-1bfd830a3aba"
-					(reference "R54")
+					(reference "R52")
 					(unit 1)
 				)
 				(path "/b4b2c88d-f6cd-4e60-862d-e21f68728580/5e5b27f8-7a4c-45d0-95f8-aff71797fcd3/7fde3d19-3e51-4869-ba44-af6d0a67b762"
-					(reference "R52")
+					(reference "R50")
 					(unit 1)
 				)

Commit message: update aux board to kicad 9: fix USB UART 2 TWO pin switches
Parts:
- renumbered C82 to C33, C83 to C34, C84 to C35, R50 to R27, U23 to U6
Changed lines of the file:
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@@
 		(dnp no)
 		(fields_autoplaced yes)
-		(property "Reference" "U23"
+		(property "Reference" "U6"
 			(at 92.71 121.92 0)
 			(effects
@@
 		(on_board yes)
 		(dnp no)
-		(property "Reference" "R50"
+		(property "Reference" "R27"
 			(at 130.81 134.62 0)
 			(effects
@@
 			(project "aux_board"
 				(path "/85134265-2435-454a-99c4-e49d8e69c5c2/180ab09f-8202-4a23-a970-ad767a3abcbf"
-					(reference "R33")
+					(reference "R29")
 					(unit 1)
 				)
 				(path "/85134265-2435-454a-99c4-e49d8e69c5c2/21705b31-e71e-4020-a43e-3303465bf5fd"
-					(reference "R31")
+					(reference "R27")
 					(unit 1)
 				)
 				(path "/85134265-2435-454a-99c4-e49d8e69c5c2/89862a4b-05be-454b-946e-6c4f5a4f01a7"
-					(reference "R34")
+					(reference "R30")
 					(unit 1)
 				)
 				(path "/85134265-2435-454a-99c4-e49d8e69c5c2/c6f75225-fda9-49b7-af41-6a3b5c80f9a2"
-					(reference "R32")
+					(reference "R28")
 					(unit 1)
 				)
@@
 		(on_board yes)
 		(dnp no)
-		(property "Reference" "C84"
+		(property "Reference" "C35"
 			(at 74.93 142.24 0)
 			(effects
@@
 			)
 		)
-		(property "Datasheet" "https://mm.digikey.com/Volume0/opasdata/d220001/medias/docus/6223/Chip_Multilayer_CC_CAT_Rev21.pdf"
+		(property "Datasheet" "https://search.murata.co.jp/Ceramy/image/img/A01X/G101/ENG/GRM188R61A226ME15-01.pdf"
 			(at 72.39 143.51 0)
 			(effects
@@
 			(project "sci_board"
 				(path "/b4b2c88d-f6cd-4e60-862d-e21f68728580/5e5b27f8-7a4c-45d0-95f8-aff71797fcd3/2f5a2990-2dc0-472a-952a-1bfd830a3aba"
-					(reference "C88")
+					(reference "C89")
 					(unit 1)
 				)
 				(path "/b4b2c88d-f6cd-4e60-862d-e21f68728580/5e5b27f8-7a4c-45d0-95f8-aff71797fcd3/7fde3d19-3e51-4869-ba44-af6d0a67b762"
-					(reference "C84")
+					(reference "C85")
 					(unit 1)
 				)
@@
 		(on_board yes)
 		(dnp no)
-		(property "Reference" "C82"
+		(property "Reference" "C33"
 			(at 53.34 138.4299 0)
 			(effects
@@
 			(project "sci_board"
 				(path "/b4b2c88d-f6cd-4e60-862d-e21f68728580/5e5b27f8-7a4c-45d0-95f8-aff71797fcd3/2f5a2990-2dc0-472a-952a-1bfd830a3aba"
-					(reference "C86")
+					(reference "C87")
 					(unit 1)
 				)
 				(path "/b4b2c88d-f6cd-4e60-862d-e21f68728580/5e5b27f8-7a4c-45d0-95f8-aff71797fcd3/7fde3d19-3e51-4869-ba44-af6d0a67b762"
-					(reference "C82")
+					(reference "C83")
 					(unit 1)
 				)
@@
 		(on_board yes)
 		(dnp no)
-		(property "Reference" "C83"
+		(property "Reference" "C34"
 			(at 46.355 138.43 0)
 			(effects
@@
 			(project "sci_board"
 				(path "/b4b2c88d-f6cd-4e60-862d-e21f68728580/5e5b27f8-7a4c-45d0-95f8-aff71797fcd3/2f5a2990-2dc0-472a-952a-1bfd830a3aba"
-					(reference "C87")
+					(reference "C88")
 					(unit 1)
 				)
 				(path "/b4b2c88d-f6cd-4e60-862d-e21f68728580/5e5b27f8-7a4c-45d0-95f8-aff71797fcd3/7fde3d19-3e51-4869-ba44-af6d0a67b762"
-					(reference "C83")
-					(unit 1)
-				)
+					(reference "C84")
+					(unit 1)
+				)

Commit message: via - pad distance rules for SCI and AVI
Parts:
- renumbered C33 to C83, C34 to C84, C35 to C85, R27 to R50, U6 to U23
Changed lines of the file:
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@@
 		(dnp no)
 		(fields_autoplaced yes)
-		(property "Reference" "U6"
+		(property "Reference" "U23"
 			(at 92.71 121.92 0)
 			(effects
@@
 		(on_board yes)
 		(dnp no)
-		(property "Reference" "R27"
+		(property "Reference" "R50"
 			(at 130.81 134.62 0)
 			(effects
@@
 		(on_board yes)
 		(dnp no)
-		(property "Reference" "C35"
+		(property "Reference" "C85"
 			(at 74.93 142.24 0)
 			(effects
@@
 		(on_board yes)
 		(dnp no)
-		(property "Reference" "C33"
+		(property "Reference" "C83"
 			(at 53.34 138.4299 0)
 			(effects
@@
 		(on_board yes)
 		(dnp no)
-		(property "Reference" "C34"
+		(property "Reference" "C84"
 			(at 46.355 138.43 0)
 			(effects
