File: sci_board/camera.kicad_sch (KiCad schematic)
At the start: 7 parts, among them J3 10051922-2410EHLF

Commit message: bom for SCI
Parts:
- C24, C25: MANUFACTURER Murata -> (none); Manufacturer (none) -> Murata; PARTREV GRM155R61E104KA87D -> (none); Part Number (none) -> GRM155R61E104KA87D
- J3: MANUFACTURER Amphenol -> (none); Manufacturer (none) -> Amphenol; PARTREV 10051922-2410EHLF -> (none); Part Number (none) -> 10051922-2410EHLF
- RN4: Manufacturer (none) -> Panasonic; Part Number (none) -> EXB-24V562JX; Tolerance (none) -> 5
Changed lines of the file:
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@@
 			)
 		)
-		(property "MANUFACTURER" "Amphenol"
+		(property "Manufacturer" "Amphenol"
 			(at 149.225 99.06 0)
 			(effects
@@
 			)
 		)
-		(property "MAXIMUM_PACKAGE_HEIGHT" ""
-			(at 149.225 99.06 0)
-			(effects
-				(font
-					(size 1.27 1.27)
-				)
-				(hide yes)
-			)
-		)
-		(property "PARTREV" "10051922-2410EHLF"
-			(at 149.225 99.06 0)
-			(effects
-				(font
-					(size 1.27 1.27)
-				)
-				(hide yes)
-			)
-		)
-		(property "STANDARD" ""
+		(property "Part Number" "10051922-2410EHLF"
 			(at 149.225 99.06 0)
 			(effects
@@
 			)
 		)
-		(property "MANUFACTURER" "Murata"
-			(at 57.785 51.435 0)
-			(effects
-				(font
-					(size 1.27 1.27)
-				)
-				(hide yes)
-			)
-		)
-		(property "MAXIMUM_PACKAGE_HEIGHT" ""
-			(at 57.785 51.435 0)
-			(effects
-				(font
-					(size 1.27 1.27)
-				)
-				(hide yes)
-			)
-		)
-		(property "PARTREV" "GRM155R61E104KA87D"
-			(at 57.785 51.435 0)
-			(effects
-				(font
-					(size 1.27 1.27)
-				)
-				(hide yes)
-			)
-		)
-		(property "STANDARD" ""
-			(at 57.785 51.435 0)
-			(effects
-				(font
-					(size 1.27 1.27)
-				)
-				(hide yes)
-			)
-		)
 		(property "Color" ""
 			(at 57.785 51.435 0)
@@
 		)
 		(property "Temperture Coefficient" "X5R"
+			(at 57.785 51.435 0)
+			(effects
+				(font
+					(size 1.27 1.27)
+				)
+				(hide yes)
+			)
+		)
+		(property "Manufacturer" "Murata"
+			(at 57.785 51.435 0)
+			(effects
+				(font
+					(size 1.27 1.27)
+				)
+				(hide yes)
+			)
+		)
+		(property "Part Number" "GRM155R61E104KA87D"
 			(at 57.785 51.435 0)
 			(effects
@@
 			)
 		)
-		(property "MANUFACTURER" ""
-			(at 89.535 29.845 0)
-			(effects
-				(font
-					(size 1.27 1.27)
-				)
-				(hide yes)
-			)
-		)
-		(property "MAXIMUM_PACKAGE_HEIGHT" ""
-			(at 89.535 29.845 0)
-			(effects
-				(font
-					(size 1.27 1.27)
-				)
-				(hide yes)
-			)
-		)
-		(property "PARTREV" ""
-			(at 89.535 29.845 0)
-			(effects
-				(font
-					(size 1.27 1.27)
-				)
-				(hide yes)
-			)
-		)
-		(property "STANDARD" ""
-			(at 89.535 29.845 0)
-			(effects
-				(font
-					(size 1.27 1.27)
-				)
-				(hide yes)
-			)
-		)
 		(pin "1"
 		)
@@
 			)
 		)
-		(property "Datasheet" "~"
+		(property "Datasheet" "https://industrial.panasonic.com/cdbs/www-data/pdf/AOC0000/AOC0000C14.pdf"
 			(at 45.085 106.045 0)
 			(effects
@@
 		)
 		(property "Description" "2 resistor network, parallel topology"
+			(at 45.085 106.045 0)
+			(effects
+				(font
+					(size 1.27 1.27)
+				)
+				(hide yes)
+			)
+		)
+		(property "Manufacturer" "Panasonic"
+			(at 45.085 106.045 0)
+			(effects
+				(font
+					(size 1.27 1.27)
+				)
+				(hide yes)
+			)
+		)
+		(property "Part Number" "EXB-24V562JX"
+			(at 45.085 106.045 0)
+			(effects
+				(font
+					(size 1.27 1.27)
+				)
+				(hide yes)
+			)
+		)
+		(property "Tolerance" "5"
 			(at 45.085 106.045 0)
 			(effects
@@
 			)
 		)
-		(property "MANUFACTURER" ""
-			(at 22.86 50.165 0)
-			(effects
-				(font
-					(size 1.27 1.27)
-				)
-				(hide yes)
-			)
-		)
-		(property "MAXIMUM_PACKAGE_HEIGHT" ""
-			(at 22.86 50.165 0)
-			(effects
-				(font
-					(size 1.27 1.27)
-				)
-				(hide yes)
-			)
-		)
-		(property "PARTREV" ""
-			(at 22.86 50.165 0)
-			(effects
-				(font
-					(size 1.27 1.27)
-				)
-				(hide yes)
-			)
-		)
-		(property "STANDARD" ""
-			(at 22.86 50.165 0)
-			(effects
-				(font
-					(size 1.27 1.27)
-				)
-				(hide yes)
-			)
-		)
 		(pin "1"
 		)
@@
 			)
 		)
-		(property "MANUFACTURER" ""
-			(at 113.03 30.48 0)
-			(effects
-				(font
-					(size 1.27 1.27)
-				)
-				(hide yes)
-			)
-		)
-		(property "MAXIMUM_PACKAGE_HEIGHT" ""
-			(at 113.03 30.48 0)
-			(effects
-				(font
-					(size 1.27 1.27)
-				)
-				(hide yes)
-			)
-		)
-		(property "PARTREV" ""
-			(at 113.03 30.48 0)
-			(effects
-				(font
-					(size 1.27 1.27)
-				)
-				(hide yes)
-			)
-		)
-		(property "STANDARD" ""
-			(at 113.03 30.48 0)
-			(effects
-				(font
-					(size 1.27 1.27)
-				)
-				(hide yes)
-			)
-		)
 		(pin "1"
 		)
@@
 			)
 		)
-		(property "MANUFACTURER" "Murata"
-			(at 43.18 51.435 0)
-			(effects
-				(font
-					(size 1.27 1.27)
-				)
-				(hide yes)
-			)
-		)
-		(property "MAXIMUM_PACKAGE_HEIGHT" ""
-			(at 43.18 51.435 0)
-			(effects
-				(font
-					(size 1.27 1.27)
-				)
-				(hide yes)
-			)
-		)
-		(property "PARTREV" "GRM155R61E104KA87D"
-			(at 43.18 51.435 0)
-			(effects
-				(font
-					(size 1.27 1.27)
-				)
-				(hide yes)
-			)
-		)
-		(property "STANDARD" ""
-			(at 43.18 51.435 0)
-			(effects
-				(font
-					(size 1.27 1.27)
-				)
-				(hide yes)
-			)
-		)
 		(property "Color" ""
 			(at 43.18 51.435 0)
@@
 			(at 43.18 51.435 0)
 			(effects
+				(font
+					(size 1.27 1.27)
+				)
+				(hide yes)
+			)
+		)
+		(property "Manufacturer" "Murata"
+			(at 43.18 51.435 0)
+			(effects
+				(font
+					(size 1.27 1.27)
+				)
+				(hide yes)
+			)
+		)
+		(property "Part Number" "GRM155R61E104KA87D"
+			(at 43.18 51.435 0)
+			(effects

Commit message: sorting out pullups on resets and attention. replace reset with RN where possible. Introduce CN to save some parts
Parts:
- renumbered RN4 to RN6
Changed lines of the file:
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@@
 				)
 				(path "/b4b2c88d-f6cd-4e60-862d-e21f68728580/5e5b27f8-7a4c-45d0-95f8-aff71797fcd3/3e22df28-91f0-4c0f-b958-7bfd7fe99c70"
+					(reference "C27")
+					(unit 1)
+				)
+				(path "/b4b2c88d-f6cd-4e60-862d-e21f68728580/5e5b27f8-7a4c-45d0-95f8-aff71797fcd3/87e2c931-24b0-464d-a54c-5e253d37e662"
 					(reference "C29")
-					(unit 1)
-				)
-				(path "/b4b2c88d-f6cd-4e60-862d-e21f68728580/5e5b27f8-7a4c-45d0-95f8-aff71797fcd3/87e2c931-24b0-464d-a54c-5e253d37e662"
-					(reference "C33")
 					(unit 1)
 				)
@@
 		(dnp no)
 		(fields_autoplaced yes)
-		(property "Reference" "RN4"
+		(property "Reference" "RN6"
 			(at 48.26 104.7749 0)
 			(effects
@@
 			(project "sci_board_wo_switches"
 				(path "/b4b2c88d-f6cd-4e60-862d-e21f68728580/5e5b27f8-7a4c-45d0-95f8-aff71797fcd3/21d0e59e-a5df-4633-9634-c7d789255f22"
-					(reference "RN4")
+					(reference "RN6")
 					(unit 1)
 				)
 				(path "/b4b2c88d-f6cd-4e60-862d-e21f68728580/5e5b27f8-7a4c-45d0-95f8-aff71797fcd3/3e22df28-91f0-4c0f-b958-7bfd7fe99c70"
-					(reference "RN5")
+					(reference "RN7")
 					(unit 1)
 				)
 				(path "/b4b2c88d-f6cd-4e60-862d-e21f68728580/5e5b27f8-7a4c-45d0-95f8-aff71797fcd3/87e2c931-24b0-464d-a54c-5e253d37e662"
-					(reference "RN6")
+					(reference "RN8")
 					(unit 1)
 				)
@@
 				)
 				(path "/b4b2c88d-f6cd-4e60-862d-e21f68728580/5e5b27f8-7a4c-45d0-95f8-aff71797fcd3/3e22df28-91f0-4c0f-b958-7bfd7fe99c70"
+					(reference "C26")
+					(unit 1)
+				)
+				(path "/b4b2c88d-f6cd-4e60-862d-e21f68728580/5e5b27f8-7a4c-45d0-95f8-aff71797fcd3/87e2c931-24b0-464d-a54c-5e253d37e662"
 					(reference "C28")
 					(unit 1)
 				)
-				(path "/b4b2c88d-f6cd-4e60-862d-e21f68728580/5e5b27f8-7a4c-45d0-95f8-aff71797fcd3/87e2c931-24b0-464d-a54c-5e253d37e662"
-					(reference "C32")
-					(unit 1)
-				)

Commit message: cleanup pullups for reset and schmitt trigger for reset; select available thermal NTCs for avi board and use chip for voltage dividers
Parts:
- RN6: footprint Resistor_SMD:R_Array_Convex_2x0402 -> Common:R_Array_Convex_2x0402_widepads
Changed lines of the file:
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@@
 			)
 		)
-		(property "Footprint" "Resistor_SMD:R_Array_Convex_2x0402"
+		(property "Footprint" "Common:R_Array_Convex_2x0402_widepads"
 			(at 49.53 106.045 90)
 			(effects

Commit message: power traces and vias of AUX and SCIlite are 0,5mm and 0.5/1.0mm
Parts:
- renumbered RN6 to RN7
Changed lines of the file:
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@@
 		(dnp no)
 		(fields_autoplaced yes)
-		(property "Reference" "RN6"
+		(property "Reference" "RN7"
 			(at 48.26 104.7749 0)
 			(effects
@@
 			(project "sci_board_wo_switches"
 				(path "/b4b2c88d-f6cd-4e60-862d-e21f68728580/5e5b27f8-7a4c-45d0-95f8-aff71797fcd3/21d0e59e-a5df-4633-9634-c7d789255f22"
-					(reference "RN6")
+					(reference "RN7")
 					(unit 1)
 				)
 				(path "/b4b2c88d-f6cd-4e60-862d-e21f68728580/5e5b27f8-7a4c-45d0-95f8-aff71797fcd3/3e22df28-91f0-4c0f-b958-7bfd7fe99c70"
-					(reference "RN7")
+					(reference "RN8")
 					(unit 1)
 				)
 				(path "/b4b2c88d-f6cd-4e60-862d-e21f68728580/5e5b27f8-7a4c-45d0-95f8-aff71797fcd3/87e2c931-24b0-464d-a54c-5e253d37e662"
-					(reference "RN8")
+					(reference "RN9")
 					(unit 1)
 				)

Commit message: EPS needs flash to self update with bootloader
Parts:
- renumbered RN7 to RN6
Changed lines of the file:
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@@
 		(dnp no)
 		(fields_autoplaced yes)
-		(property "Reference" "RN7"
+		(property "Reference" "RN6"
 			(at 48.26 104.7749 0)
 			(effects
@@
 			(project "sci_board_wo_switches"
 				(path "/b4b2c88d-f6cd-4e60-862d-e21f68728580/5e5b27f8-7a4c-45d0-95f8-aff71797fcd3/21d0e59e-a5df-4633-9634-c7d789255f22"
+					(reference "RN6")
+					(unit 1)
+				)
+				(path "/b4b2c88d-f6cd-4e60-862d-e21f68728580/5e5b27f8-7a4c-45d0-95f8-aff71797fcd3/3e22df28-91f0-4c0f-b958-7bfd7fe99c70"
 					(reference "RN7")
 					(unit 1)
 				)
-				(path "/b4b2c88d-f6cd-4e60-862d-e21f68728580/5e5b27f8-7a4c-45d0-95f8-aff71797fcd3/3e22df28-91f0-4c0f-b958-7bfd7fe99c70"
+				(path "/b4b2c88d-f6cd-4e60-862d-e21f68728580/5e5b27f8-7a4c-45d0-95f8-aff71797fcd3/87e2c931-24b0-464d-a54c-5e253d37e662"
 					(reference "RN8")
 					(unit 1)
 				)
-				(path "/b4b2c88d-f6cd-4e60-862d-e21f68728580/5e5b27f8-7a4c-45d0-95f8-aff71797fcd3/87e2c931-24b0-464d-a54c-5e253d37e662"
-					(reference "RN9")
-					(unit 1)
-				)

Commit message: move project to new location, update sympbol, footprint and step paths
Parts:
- renumbered RN6 to RN8
Changed lines of the file:
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@@
 		(dnp no)
 		(fields_autoplaced yes)
-		(property "Reference" "RN6"
+		(property "Reference" "RN8"
 			(at 48.26 104.7749 0)
 			(effects
@@
 			(project "sci_board_wo_switches"
 				(path "/b4b2c88d-f6cd-4e60-862d-e21f68728580/5e5b27f8-7a4c-45d0-95f8-aff71797fcd3/21d0e59e-a5df-4633-9634-c7d789255f22"
-					(reference "RN6")
+					(reference "RN8")
 					(unit 1)
 				)
 				(path "/b4b2c88d-f6cd-4e60-862d-e21f68728580/5e5b27f8-7a4c-45d0-95f8-aff71797fcd3/3e22df28-91f0-4c0f-b958-7bfd7fe99c70"
-					(reference "RN7")
+					(reference "RN9")
 					(unit 1)
 				)
 				(path "/b4b2c88d-f6cd-4e60-862d-e21f68728580/5e5b27f8-7a4c-45d0-95f8-aff71797fcd3/87e2c931-24b0-464d-a54c-5e253d37e662"
-					(reference "RN8")
+					(reference "RN10")
 					(unit 1)
 				)

Commit message: VRef+ meeds to be connected to VDDA, should not be left floating
Parts:
- renumbered RN8 to RN6
Changed lines of the file:
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@@
 		(dnp no)
 		(fields_autoplaced yes)
-		(property "Reference" "RN8"
+		(property "Reference" "RN6"
 			(at 48.26 104.7749 0)
 			(effects
@@
 			(project "sci_board_wo_switches"
 				(path "/b4b2c88d-f6cd-4e60-862d-e21f68728580/5e5b27f8-7a4c-45d0-95f8-aff71797fcd3/21d0e59e-a5df-4633-9634-c7d789255f22"
+					(reference "RN6")
+					(unit 1)
+				)
+				(path "/b4b2c88d-f6cd-4e60-862d-e21f68728580/5e5b27f8-7a4c-45d0-95f8-aff71797fcd3/3e22df28-91f0-4c0f-b958-7bfd7fe99c70"
+					(reference "RN7")
+					(unit 1)
+				)
+				(path "/b4b2c88d-f6cd-4e60-862d-e21f68728580/5e5b27f8-7a4c-45d0-95f8-aff71797fcd3/87e2c931-24b0-464d-a54c-5e253d37e662"
 					(reference "RN8")
 					(unit 1)
 				)
-				(path "/b4b2c88d-f6cd-4e60-862d-e21f68728580/5e5b27f8-7a4c-45d0-95f8-aff71797fcd3/3e22df28-91f0-4c0f-b958-7bfd7fe99c70"
-					(reference "RN9")
-					(unit 1)
-				)
-				(path "/b4b2c88d-f6cd-4e60-862d-e21f68728580/5e5b27f8-7a4c-45d0-95f8-aff71797fcd3/87e2c931-24b0-464d-a54c-5e253d37e662"
-					(reference "RN10")
-					(unit 1)
-				)
