File: avionics_board/acs_directional_unit.kicad_sch (KiCad schematic)
At the start: 7 parts, among them J4 Conn_01x04, U7 INA226, U8 DRV8838

Commit message: interim checkin before streamlining AVI
Parts:
- U8: Mfr. # DRV8838DSGR -> (none); Part Number (none) -> DRV8838DSGR
Changed lines of the file:
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@@
-			)
-		)
-		(property "Mfr. #" "DRV8838DSGR"
-			(at 160.02 105.41 0)
-			(effects
-				(font
-					(size 1.27 1.27)
-				)
-				(hide yes)
 			)
 		)
@@
 			(at 160.02 105.41 0)
 			(effects
+				(font
+					(size 1.27 1.27)
+				)
+				(hide yes)
+			)
+		)
+		(property "Part Number" "DRV8838DSGR"
+			(at 160.02 105.41 0)
+			(effects

Commit message: refactor AVI into nicer hierarchical components
Parts:
- renumbered C36 to C31, C37 to C32, C38 to C33, J4 to J1, R31 to R22, U7 to U4, U8 to U5
Changed lines of the file:
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@@
 		(on_board yes)
 		(dnp no)
-		(property "Reference" "U8"
+		(property "Reference" "U5"
 			(at 164.465 88.265 0)
 			(effects
@@
 		(instances
 			(project "AVIONICS_BOARD"
-				(path "/f6cc00ab-17f1-4973-862f-7ac95fe70668/00000000-0000-0000-0000-00005ea31c93/00000000-0000-0000-0000-00005eb482dd/4e2a47c2-c2ed-4db2-bf85-7030d7458163"
+				(path "/f6cc00ab-17f1-4973-862f-7ac95fe70668/1f9ae17d-3f3e-4633-9b01-30c344473415/4e2a47c2-c2ed-4db2-bf85-7030d7458163"
 					(reference "U8")
 					(unit 1)
 				)
-				(path "/f6cc00ab-17f1-4973-862f-7ac95fe70668/00000000-0000-0000-0000-00005ea31c93/00000000-0000-0000-0000-00005eb482dd/7d3e76d7-4668-440d-8487-c4215eabf8a2"
+				(path "/f6cc00ab-17f1-4973-862f-7ac95fe70668/1f9ae17d-3f3e-4633-9b01-30c344473415/7d3e76d7-4668-440d-8487-c4215eabf8a2"
 					(reference "U15")
 					(unit 1)
 				)
-				(path "/f6cc00ab-17f1-4973-862f-7ac95fe70668/00000000-0000-0000-0000-00005ea31c93/00000000-0000-0000-0000-00005eb482dd/a0859814-3829-45a9-a25d-0db563664eca"
+				(path "/f6cc00ab-17f1-4973-862f-7ac95fe70668/1f9ae17d-3f3e-4633-9b01-30c344473415/a0859814-3829-45a9-a25d-0db563664eca"
 					(reference "U5")
 					(unit 1)
@@
 		(dnp no)
 		(fields_autoplaced yes)
-		(property "Reference" "C36"
+		(property "Reference" "C31"
 			(at 129.54 58.4262 0)
 			(effects
@@
 		(instances
 			(project "AVIONICS_BOARD"
-				(path "/f6cc00ab-17f1-4973-862f-7ac95fe70668/00000000-0000-0000-0000-00005ea31c93/00000000-0000-0000-0000-00005eb482dd/4e2a47c2-c2ed-4db2-bf85-7030d7458163"
+				(path "/f6cc00ab-17f1-4973-862f-7ac95fe70668/1f9ae17d-3f3e-4633-9b01-30c344473415/4e2a47c2-c2ed-4db2-bf85-7030d7458163"
 					(reference "C36")
 					(unit 1)
 				)
-				(path "/f6cc00ab-17f1-4973-862f-7ac95fe70668/00000000-0000-0000-0000-00005ea31c93/00000000-0000-0000-0000-00005eb482dd/7d3e76d7-4668-440d-8487-c4215eabf8a2"
+				(path "/f6cc00ab-17f1-4973-862f-7ac95fe70668/1f9ae17d-3f3e-4633-9b01-30c344473415/7d3e76d7-4668-440d-8487-c4215eabf8a2"
 					(reference "C55")
 					(unit 1)
 				)
-				(path "/f6cc00ab-17f1-4973-862f-7ac95fe70668/00000000-0000-0000-0000-00005ea31c93/00000000-0000-0000-0000-00005eb482dd/a0859814-3829-45a9-a25d-0db563664eca"
+				(path "/f6cc00ab-17f1-4973-862f-7ac95fe70668/1f9ae17d-3f3e-4633-9b01-30c344473415/a0859814-3829-45a9-a25d-0db563664eca"
 					(reference "C31")
 					(unit 1)
@@
 		(on_board yes)
 		(dnp no)
-		(property "Reference" "U7"
+		(property "Reference" "U4"
 			(at 120.9959 60.325 0)
 			(effects
@@
 		(instances
 			(project "AVIONICS_BOARD"
-				(path "/f6cc00ab-17f1-4973-862f-7ac95fe70668/00000000-0000-0000-0000-00005ea31c93/00000000-0000-0000-0000-00005eb482dd/4e2a47c2-c2ed-4db2-bf85-7030d7458163"
+				(path "/f6cc00ab-17f1-4973-862f-7ac95fe70668/1f9ae17d-3f3e-4633-9b01-30c344473415/4e2a47c2-c2ed-4db2-bf85-7030d7458163"
 					(reference "U7")
 					(unit 1)
 				)
-				(path "/f6cc00ab-17f1-4973-862f-7ac95fe70668/00000000-0000-0000-0000-00005ea31c93/00000000-0000-0000-0000-00005eb482dd/7d3e76d7-4668-440d-8487-c4215eabf8a2"
+				(path "/f6cc00ab-17f1-4973-862f-7ac95fe70668/1f9ae17d-3f3e-4633-9b01-30c344473415/7d3e76d7-4668-440d-8487-c4215eabf8a2"
 					(reference "U14")
 					(unit 1)
 				)
-				(path "/f6cc00ab-17f1-4973-862f-7ac95fe70668/00000000-0000-0000-0000-00005ea31c93/00000000-0000-0000-0000-00005eb482dd/a0859814-3829-45a9-a25d-0db563664eca"
+				(path "/f6cc00ab-17f1-4973-862f-7ac95fe70668/1f9ae17d-3f3e-4633-9b01-30c344473415/a0859814-3829-45a9-a25d-0db563664eca"
 					(reference "U4")
 					(unit 1)
@@
 		(dnp no)
 		(fields_autoplaced yes)
-		(property "Reference" "#FLG015"
+		(property "Reference" "#FLG013"
 			(at 160.02 81.915 0)
 			(effects
@@
 		)
 		(instances
-			(project ""
-				(path "/f6cc00ab-17f1-4973-862f-7ac95fe70668/00000000-0000-0000-0000-00005ea31c93/00000000-0000-0000-0000-00005eb482dd/4e2a47c2-c2ed-4db2-bf85-7030d7458163"
+			(project "AVIONICS_BOARD"
+				(path "/f6cc00ab-17f1-4973-862f-7ac95fe70668/1f9ae17d-3f3e-4633-9b01-30c344473415/4e2a47c2-c2ed-4db2-bf85-7030d7458163"
 					(reference "#FLG015")
 					(unit 1)
 				)
-				(path "/f6cc00ab-17f1-4973-862f-7ac95fe70668/00000000-0000-0000-0000-00005ea31c93/00000000-0000-0000-0000-00005eb482dd/7d3e76d7-4668-440d-8487-c4215eabf8a2"
-					(reference "#FLG016")
-					(unit 1)
-				)
-				(path "/f6cc00ab-17f1-4973-862f-7ac95fe70668/00000000-0000-0000-0000-00005ea31c93/00000000-0000-0000-0000-00005eb482dd/a0859814-3829-45a9-a25d-0db563664eca"
+				(path "/f6cc00ab-17f1-4973-862f-7ac95fe70668/1f9ae17d-3f3e-4633-9b01-30c344473415/7d3e76d7-4668-440d-8487-c4215eabf8a2"
 					(reference "#FLG014")
+					(unit 1)
+				)
+				(path "/f6cc00ab-17f1-4973-862f-7ac95fe70668/1f9ae17d-3f3e-4633-9b01-30c344473415/a0859814-3829-45a9-a25d-0db563664eca"
+					(reference "#FLG013")
 					(unit 1)
 				)
@@
 		(on_board yes)
 		(dnp no)
-		(property "Reference" "C38"
+		(property "Reference" "C33"
 			(at 140.97 93.98 0)
 			(effects
@@
 		(instances
 			(project "AVIONICS_BOARD"
-				(path "/f6cc00ab-17f1-4973-862f-7ac95fe70668/00000000-0000-0000-0000-00005ea31c93/00000000-0000-0000-0000-00005eb482dd/4e2a47c2-c2ed-4db2-bf85-7030d7458163"
+				(path "/f6cc00ab-17f1-4973-862f-7ac95fe70668/1f9ae17d-3f3e-4633-9b01-30c344473415/4e2a47c2-c2ed-4db2-bf85-7030d7458163"
 					(reference "C38")
 					(unit 1)
 				)
-				(path "/f6cc00ab-17f1-4973-862f-7ac95fe70668/00000000-0000-0000-0000-00005ea31c93/00000000-0000-0000-0000-00005eb482dd/7d3e76d7-4668-440d-8487-c4215eabf8a2"
+				(path "/f6cc00ab-17f1-4973-862f-7ac95fe70668/1f9ae17d-3f3e-4633-9b01-30c344473415/7d3e76d7-4668-440d-8487-c4215eabf8a2"
 					(reference "C57")
 					(unit 1)
 				)
-				(path "/f6cc00ab-17f1-4973-862f-7ac95fe70668/00000000-0000-0000-0000-00005ea31c93/00000000-0000-0000-0000-00005eb482dd/a0859814-3829-45a9-a25d-0db563664eca"
+				(path "/f6cc00ab-17f1-4973-862f-7ac95fe70668/1f9ae17d-3f3e-4633-9b01-30c344473415/a0859814-3829-45a9-a25d-0db563664eca"
 					(reference "C33")
 					(unit 1)
@@
 		(on_board yes)
 		(dnp no)
-		(property "Reference" "R31"
+		(property "Reference" "R22"
 			(at 139.065 79.3749 0)
 			(effects
@@
 		(instances
 			(project "AVIONICS_BOARD"
-				(path "/f6cc00ab-17f1-4973-862f-7ac95fe70668/00000000-0000-0000-0000-00005ea31c93/00000000-0000-0000-0000-00005eb482dd/4e2a47c2-c2ed-4db2-bf85-7030d7458163"
+				(path "/f6cc00ab-17f1-4973-862f-7ac95fe70668/1f9ae17d-3f3e-4633-9b01-30c344473415/4e2a47c2-c2ed-4db2-bf85-7030d7458163"
 					(reference "R31")
 					(unit 1)
 				)
-				(path "/f6cc00ab-17f1-4973-862f-7ac95fe70668/00000000-0000-0000-0000-00005ea31c93/00000000-0000-0000-0000-00005eb482dd/7d3e76d7-4668-440d-8487-c4215eabf8a2"
+				(path "/f6cc00ab-17f1-4973-862f-7ac95fe70668/1f9ae17d-3f3e-4633-9b01-30c344473415/7d3e76d7-4668-440d-8487-c4215eabf8a2"
 					(reference "R42")
 					(unit 1)
 				)
-				(path "/f6cc00ab-17f1-4973-862f-7ac95fe70668/00000000-0000-0000-0000-00005ea31c93/00000000-0000-0000-0000-00005eb482dd/a0859814-3829-45a9-a25d-0db563664eca"
+				(path "/f6cc00ab-17f1-4973-862f-7ac95fe70668/1f9ae17d-3f3e-4633-9b01-30c344473415/a0859814-3829-45a9-a25d-0db563664eca"
 					(reference "R22")
 					(unit 1)
@@
 		(on_board yes)
 		(dnp no)
-		(property "Reference" "C37"
+		(property "Reference" "C32"
 			(at 148.59 85.0962 0)
 			(effects
@@
 		(instances
 			(project "AVIONICS_BOARD"
-				(path "/f6cc00ab-17f1-4973-862f-7ac95fe70668/00000000-0000-0000-0000-00005ea31c93/00000000-0000-0000-0000-00005eb482dd/4e2a47c2-c2ed-4db2-bf85-7030d7458163"
+				(path "/f6cc00ab-17f1-4973-862f-7ac95fe70668/1f9ae17d-3f3e-4633-9b01-30c344473415/4e2a47c2-c2ed-4db2-bf85-7030d7458163"
 					(reference "C37")
 					(unit 1)
 				)
-				(path "/f6cc00ab-17f1-4973-862f-7ac95fe70668/00000000-0000-0000-0000-00005ea31c93/00000000-0000-0000-0000-00005eb482dd/7d3e76d7-4668-440d-8487-c4215eabf8a2"
+				(path "/f6cc00ab-17f1-4973-862f-7ac95fe70668/1f9ae17d-3f3e-4633-9b01-30c344473415/7d3e76d7-4668-440d-8487-c4215eabf8a2"
 					(reference "C56")
 					(unit 1)
 				)
-				(path "/f6cc00ab-17f1-4973-862f-7ac95fe70668/00000000-0000-0000-0000-00005ea31c93/00000000-0000-0000-0000-00005eb482dd/a0859814-3829-45a9-a25d-0db563664eca"
+				(path "/f6cc00ab-17f1-4973-862f-7ac95fe70668/1f9ae17d-3f3e-4633-9b01-30c344473415/a0859814-3829-45a9-a25d-0db563664eca"
 					(reference "C32")
 					(unit 1)
@@
 		(on_board yes)
 		(dnp no)
-		(property "Reference" "J4"
+		(property "Reference" "J1"
 			(at 196.85 96.52 0)
 			(effects
@@
 		(instances
 			(project "AVIONICS_BOARD"
-				(path "/f6cc00ab-17f1-4973-862f-7ac95fe70668/00000000-0000-0000-0000-00005ea31c93/00000000-0000-0000-0000-00005eb482dd/4e2a47c2-c2ed-4db2-bf85-7030d7458163"
+				(path "/f6cc00ab-17f1-4973-862f-7ac95fe70668/1f9ae17d-3f3e-4633-9b01-30c344473415/4e2a47c2-c2ed-4db2-bf85-7030d7458163"
 					(reference "J4")
 					(unit 1)
 				)
-				(path "/f6cc00ab-17f1-4973-862f-7ac95fe70668/00000000-0000-0000-0000-00005ea31c93/00000000-0000-0000-0000-00005eb482dd/7d3e76d7-4668-440d-8487-c4215eabf8a2"
+				(path "/f6cc00ab-17f1-4973-862f-7ac95fe70668/1f9ae17d-3f3e-4633-9b01-30c344473415/7d3e76d7-4668-440d-8487-c4215eabf8a2"
 					(reference "J9")
 					(unit 1)
 				)
-				(path "/f6cc00ab-17f1-4973-862f-7ac95fe70668/00000000-0000-0000-0000-00005ea31c93/00000000-0000-0000-0000-00005eb482dd/a0859814-3829-45a9-a25d-0db563664eca"
+				(path "/f6cc00ab-17f1-4973-862f-7ac95fe70668/1f9ae17d-3f3e-4633-9b01-30c344473415/a0859814-3829-45a9-a25d-0db563664eca"
 					(reference "J1")
 					(unit 1)

Commit message: AVI assigning interrupts
Parts:
- renumbered C31 to C36, C32 to C37, C33 to C38, J1 to J4, R22 to R31, U4 to U7, U5 to U8
Changed lines of the file:
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@@
 		(on_board yes)
 		(dnp no)
-		(property "Reference" "U5"
+		(property "Reference" "U8"
 			(at 164.465 88.265 0)
 			(effects
@@
 		(dnp no)
 		(fields_autoplaced yes)
-		(property "Reference" "C31"
+		(property "Reference" "C36"
 			(at 129.54 58.4262 0)
 			(effects
@@
 		(on_board yes)
 		(dnp no)
-		(property "Reference" "U4"
+		(property "Reference" "U7"
 			(at 120.9959 60.325 0)
 			(effects
@@
 		(dnp no)
 		(fields_autoplaced yes)
-		(property "Reference" "#FLG013"
+		(property "Reference" "#FLG015"
 			(at 160.02 81.915 0)
 			(effects
@@
 		(on_board yes)
 		(dnp no)
-		(property "Reference" "C33"
+		(property "Reference" "C38"
 			(at 140.97 93.98 0)
 			(effects
@@
 		(on_board yes)
 		(dnp no)
-		(property "Reference" "R22"
+		(property "Reference" "R31"
 			(at 139.065 79.3749 0)
 			(effects
@@
 		(on_board yes)
 		(dnp no)
-		(property "Reference" "C32"
+		(property "Reference" "C37"
 			(at 148.59 85.0962 0)
 			(effects
@@
 		(on_board yes)
 		(dnp no)
-		(property "Reference" "J1"
+		(property "Reference" "J4"
 			(at 196.85 96.52 0)
 			(effects

Commit message: reconcile BOMS for AVI. SCI and AUX
Parts:
- C36, C37, C38: value 100n -> 100nF; Manufacturer (none) -> Murata; Part Number (none) -> GRM155R61E102KA01D; Tolerance (none) -> 10; Voltage (none) -> 25
- J4: now not fitted
- R31: Manufacturer (none) -> YAGEO; Part Number (none) -> PE0805FRE470R01Z; Tolerance (none) -> 1
- U7: Manufacturer (none) -> TI; Part Number (none) -> INA226
- U8: Manufacturer (none) -> TI
Changed lines of the file:
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@@
+			)
+		)
+		(property "Manufacturer" "TI"
+			(at 160.02 105.41 0)
+			(effects
+				(font
+					(size 1.27 1.27)
+				)
+				(hide yes)
 			)
 		)
@@
 			)
 		)
-		(property "Value" "100n"
+		(property "Value" "100nF"
 			(at 129.54 60.9662 0)
 			(effects
@@
 			)
 		)
-		(property "Datasheet" "~"
+		(property "Datasheet" "https://search.murata.co.jp/Ceramy/image/img/A01X/G101/ENG/GRM155R61E102KA01-01.pdf"
 			(at 126.365 59.69 0)
 			(effects
@@
 		)
 		(property "Alt" ""
+			(at 126.365 59.69 0)
+			(effects
+				(font
+					(size 1.27 1.27)
+				)
+				(hide yes)
+			)
+		)
+		(property "Manufacturer" "Murata"
+			(at 126.365 59.69 0)
+			(effects
+				(font
+					(size 1.27 1.27)
+				)
+				(hide yes)
+			)
+		)
+		(property "Part Number" "GRM155R61E102KA01D "
+			(at 126.365 59.69 0)
+			(effects
+				(font
+					(size 1.27 1.27)
+				)
+				(hide yes)
+			)
+		)
+		(property "Tolerance" "10"
+			(at 126.365 59.69 0)
+			(effects
+				(font
+					(size 1.27 1.27)
+				)
+				(hide yes)
+			)
+		)
+		(property "Voltage" "25"
 			(at 126.365 59.69 0)
 			(effects
@@
 			)
 		)
+		(property "Manufacturer" "TI"
+			(at 123.19 74.93 0)
+			(effects
+				(font
+					(size 1.27 1.27)
+				)
+				(hide yes)
+			)
+		)
+		(property "Part Number" "INA226"
+			(at 123.19 74.93 0)
+			(effects
+				(font
+					(size 1.27 1.27)
+				)
+				(hide yes)
+			)
+		)
 		(pin "5"
 		)
@@
 			)
 		)
-		(property "Value" "100n"
+		(property "Value" "100nF"
 			(at 140.97 96.52 0)
 			(effects
@@
 			)
 		)
-		(property "Datasheet" "~"
+		(property "Datasheet" "https://search.murata.co.jp/Ceramy/image/img/A01X/G101/ENG/GRM155R61E102KA01-01.pdf"
 			(at 146.685 94.615 0)
 			(effects
@@
 		)
 		(property "Alt" ""
+			(at 146.685 94.615 0)
+			(effects
+				(font
+					(size 1.27 1.27)
+				)
+				(hide yes)
+			)
+		)
+		(property "Manufacturer" "Murata"
+			(at 146.685 94.615 0)
+			(effects
+				(font
+					(size 1.27 1.27)
+				)
+				(hide yes)
+			)
+		)
+		(property "Part Number" "GRM155R61E102KA01D "
+			(at 146.685 94.615 0)
+			(effects
+				(font
+					(size 1.27 1.27)
+				)
+				(hide yes)
+			)
+		)
+		(property "Tolerance" "10"
+			(at 146.685 94.615 0)
+			(effects
+				(font
+					(size 1.27 1.27)
+				)
+				(hide yes)
+			)
+		)
+		(property "Voltage" "25"
 			(at 146.685 94.615 0)
 			(effects
@@
 			)
 		)
-		(property "Datasheet" "~"
+		(property "Datasheet" "https://mm.digikey.com/Volume0/opasdata/d220001/medias/docus/5343/PE_Series_DS.pdf"
 			(at 137.16 80.645 0)
 			(effects
@@
 		)
 		(property "Alt" ""
+			(at 137.16 80.645 0)
+			(effects
+				(font
+					(size 1.27 1.27)
+				)
+				(hide yes)
+			)
+		)
+		(property "Manufacturer" "YAGEO"
+			(at 137.16 80.645 0)
+			(effects
+				(font
+					(size 1.27 1.27)
+				)
+				(hide yes)
+			)
+		)
+		(property "Part Number" "PE0805FRE470R01Z"
+			(at 137.16 80.645 0)
+			(effects
+				(font
+					(size 1.27 1.27)
+				)
+				(hide yes)
+			)
+		)
+		(property "Tolerance" "1"
 			(at 137.16 80.645 0)
 			(effects
@@
 			)
 		)
-		(property "Value" "100n"
+		(property "Value" "100nF"
 			(at 148.59 86.36 0)
 			(effects
@@
 			)
 		)
-		(property "Datasheet" "~"
+		(property "Datasheet" "https://search.murata.co.jp/Ceramy/image/img/A01X/G101/ENG/GRM155R61E102KA01-01.pdf"
 			(at 145.415 86.36 0)
 			(effects
@@
 		)
 		(property "Alt" ""
+			(at 145.415 86.36 0)
+			(effects
+				(font
+					(size 1.27 1.27)
+				)
+				(hide yes)
+			)
+		)
+		(property "Manufacturer" "Murata"
+			(at 145.415 86.36 0)
+			(effects
+				(font
+					(size 1.27 1.27)
+				)
+				(hide yes)
+			)
+		)
+		(property "Part Number" "GRM155R61E102KA01D "
+			(at 145.415 86.36 0)
+			(effects
+				(font
+					(size 1.27 1.27)
+				)
+				(hide yes)
+			)
+		)
+		(property "Tolerance" "10"
+			(at 145.415 86.36 0)
+			(effects
+				(font
+					(size 1.27 1.27)
+				)
+				(hide yes)
+			)
+		)
+		(property "Voltage" "25"
 			(at 145.415 86.36 0)
 			(effects
@@
 		(in_bom yes)
 		(on_board yes)
-		(dnp no)
+		(dnp yes)
 		(property "Reference" "J4"
 			(at 196.85 96.52 0)

Commit message: interim checkin for EPS BOM
Parts:
- C36, C37, C38: Part Number GRM155R61E102KA01D -> GRM155R61E104KA87D
Changed lines of the file:
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@@
 			)
 		)
-		(property "Datasheet" "https://search.murata.co.jp/Ceramy/image/img/A01X/G101/ENG/GRM155R61E102KA01-01.pdf"
+		(property "Datasheet" "https://search.murata.co.jp/Ceramy/image/img/A01X/G101/ENG/GRM155R61E104KA87-01.pdf"
 			(at 126.365 59.69 0)
 			(effects
@@
 			)
 		)
-		(property "Part Number" "GRM155R61E102KA01D "
+		(property "Part Number" "GRM155R61E104KA87D"
 			(at 126.365 59.69 0)
 			(effects
@@
 			)
 		)
-		(property "Datasheet" "https://search.murata.co.jp/Ceramy/image/img/A01X/G101/ENG/GRM155R61E102KA01-01.pdf"
+		(property "Datasheet" "https://search.murata.co.jp/Ceramy/image/img/A01X/G101/ENG/GRM155R61E104KA87-01.pdf"
 			(at 146.685 94.615 0)
 			(effects
@@
 			)
 		)
-		(property "Part Number" "GRM155R61E102KA01D "
+		(property "Part Number" "GRM155R61E104KA87D"
 			(at 146.685 94.615 0)
 			(effects
@@
 			)
 		)
-		(property "Datasheet" "https://search.murata.co.jp/Ceramy/image/img/A01X/G101/ENG/GRM155R61E102KA01-01.pdf"
+		(property "Datasheet" "https://search.murata.co.jp/Ceramy/image/img/A01X/G101/ENG/GRM155R61E104KA87-01.pdf"
 			(at 145.415 86.36 0)
 			(effects
@@
 			)
 		)
-		(property "Part Number" "GRM155R61E102KA01D "
+		(property "Part Number" "GRM155R61E104KA87D"
 			(at 145.415 86.36 0)
 			(effects

Commit message: reenumerate AVI board
Parts:
- renumbered C36 to C50, C37 to C51, C38 to C52, J4 to J8, R31 to R40, U7 to U13, U8 to U14
Changed lines of the file:
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@@
 		(on_board yes)
 		(dnp no)
-		(property "Reference" "U8"
+		(property "Reference" "U14"
 			(at 164.465 88.265 0)
 			(effects
@@
 			(project "AVIONICS_BOARD"
 				(path "/f6cc00ab-17f1-4973-862f-7ac95fe70668/1f9ae17d-3f3e-4633-9b01-30c344473415/4e2a47c2-c2ed-4db2-bf85-7030d7458163"
+					(reference "U14")
+					(unit 1)
+				)
+				(path "/f6cc00ab-17f1-4973-862f-7ac95fe70668/1f9ae17d-3f3e-4633-9b01-30c344473415/7d3e76d7-4668-440d-8487-c4215eabf8a2"
 					(reference "U8")
-					(unit 1)
-				)
-				(path "/f6cc00ab-17f1-4973-862f-7ac95fe70668/1f9ae17d-3f3e-4633-9b01-30c344473415/7d3e76d7-4668-440d-8487-c4215eabf8a2"
-					(reference "U15")
 					(unit 1)
 				)
@@
 		(dnp no)
 		(fields_autoplaced yes)
-		(property "Reference" "C36"
+		(property "Reference" "C50"
 			(at 129.54 58.4262 0)
 			(effects
@@
 			(project "AVIONICS_BOARD"
 				(path "/f6cc00ab-17f1-4973-862f-7ac95fe70668/1f9ae17d-3f3e-4633-9b01-30c344473415/4e2a47c2-c2ed-4db2-bf85-7030d7458163"
+					(reference "C50")
+					(unit 1)
+				)
+				(path "/f6cc00ab-17f1-4973-862f-7ac95fe70668/1f9ae17d-3f3e-4633-9b01-30c344473415/7d3e76d7-4668-440d-8487-c4215eabf8a2"
 					(reference "C36")
-					(unit 1)
-				)
-				(path "/f6cc00ab-17f1-4973-862f-7ac95fe70668/1f9ae17d-3f3e-4633-9b01-30c344473415/7d3e76d7-4668-440d-8487-c4215eabf8a2"
-					(reference "C55")
 					(unit 1)
 				)
@@
 		(on_board yes)
 		(dnp no)
-		(property "Reference" "U7"
+		(property "Reference" "U13"
 			(at 120.9959 60.325 0)
 			(effects
@@
 			(project "AVIONICS_BOARD"
 				(path "/f6cc00ab-17f1-4973-862f-7ac95fe70668/1f9ae17d-3f3e-4633-9b01-30c344473415/4e2a47c2-c2ed-4db2-bf85-7030d7458163"
+					(reference "U13")
+					(unit 1)
+				)
+				(path "/f6cc00ab-17f1-4973-862f-7ac95fe70668/1f9ae17d-3f3e-4633-9b01-30c344473415/7d3e76d7-4668-440d-8487-c4215eabf8a2"
 					(reference "U7")
-					(unit 1)
-				)
-				(path "/f6cc00ab-17f1-4973-862f-7ac95fe70668/1f9ae17d-3f3e-4633-9b01-30c344473415/7d3e76d7-4668-440d-8487-c4215eabf8a2"
-					(reference "U14")
 					(unit 1)
 				)
@@
 		(on_board yes)
 		(dnp no)
-		(property "Reference" "C38"
+		(property "Reference" "C52"
 			(at 140.97 93.98 0)
 			(effects
@@
 			(project "AVIONICS_BOARD"
 				(path "/f6cc00ab-17f1-4973-862f-7ac95fe70668/1f9ae17d-3f3e-4633-9b01-30c344473415/4e2a47c2-c2ed-4db2-bf85-7030d7458163"
+					(reference "C52")
+					(unit 1)
+				)
+				(path "/f6cc00ab-17f1-4973-862f-7ac95fe70668/1f9ae17d-3f3e-4633-9b01-30c344473415/7d3e76d7-4668-440d-8487-c4215eabf8a2"
 					(reference "C38")
-					(unit 1)
-				)
-				(path "/f6cc00ab-17f1-4973-862f-7ac95fe70668/1f9ae17d-3f3e-4633-9b01-30c344473415/7d3e76d7-4668-440d-8487-c4215eabf8a2"
-					(reference "C57")
 					(unit 1)
 				)
@@
 		(on_board yes)
 		(dnp no)
-		(property "Reference" "R31"
+		(property "Reference" "R40"
 			(at 139.065 79.3749 0)
 			(effects
@@
 			(project "AVIONICS_BOARD"
 				(path "/f6cc00ab-17f1-4973-862f-7ac95fe70668/1f9ae17d-3f3e-4633-9b01-30c344473415/4e2a47c2-c2ed-4db2-bf85-7030d7458163"
-					(reference "R31")
+					(reference "R40")
 					(unit 1)
 				)
 				(path "/f6cc00ab-17f1-4973-862f-7ac95fe70668/1f9ae17d-3f3e-4633-9b01-30c344473415/7d3e76d7-4668-440d-8487-c4215eabf8a2"
-					(reference "R42")
+					(reference "R28")
 					(unit 1)
 				)
 				(path "/f6cc00ab-17f1-4973-862f-7ac95fe70668/1f9ae17d-3f3e-4633-9b01-30c344473415/a0859814-3829-45a9-a25d-0db563664eca"
-					(reference "R22")
+					(reference "R20")
 					(unit 1)
 				)
@@
 		(on_board yes)
 		(dnp no)
-		(property "Reference" "C37"
+		(property "Reference" "C51"
 			(at 148.59 85.0962 0)
 			(effects
@@
 			(project "AVIONICS_BOARD"
 				(path "/f6cc00ab-17f1-4973-862f-7ac95fe70668/1f9ae17d-3f3e-4633-9b01-30c344473415/4e2a47c2-c2ed-4db2-bf85-7030d7458163"
+					(reference "C51")
+					(unit 1)
+				)
+				(path "/f6cc00ab-17f1-4973-862f-7ac95fe70668/1f9ae17d-3f3e-4633-9b01-30c344473415/7d3e76d7-4668-440d-8487-c4215eabf8a2"
 					(reference "C37")
-					(unit 1)
-				)
-				(path "/f6cc00ab-17f1-4973-862f-7ac95fe70668/1f9ae17d-3f3e-4633-9b01-30c344473415/7d3e76d7-4668-440d-8487-c4215eabf8a2"
-					(reference "C56")
 					(unit 1)
 				)
@@
 		(on_board yes)
 		(dnp yes)
-		(property "Reference" "J4"
+		(property "Reference" "J8"
 			(at 196.85 96.52 0)
 			(effects
@@
 			(project "AVIONICS_BOARD"
 				(path "/f6cc00ab-17f1-4973-862f-7ac95fe70668/1f9ae17d-3f3e-4633-9b01-30c344473415/4e2a47c2-c2ed-4db2-bf85-7030d7458163"
+					(reference "J8")
+					(unit 1)
+				)
+				(path "/f6cc00ab-17f1-4973-862f-7ac95fe70668/1f9ae17d-3f3e-4633-9b01-30c344473415/7d3e76d7-4668-440d-8487-c4215eabf8a2"
 					(reference "J4")
 					(unit 1)
 				)
-				(path "/f6cc00ab-17f1-4973-862f-7ac95fe70668/1f9ae17d-3f3e-4633-9b01-30c344473415/7d3e76d7-4668-440d-8487-c4215eabf8a2"
-					(reference "J9")
-					(unit 1)
-				)
