File: avionics_board/TEMPERATURE_ADC.kicad_sch (KiCad schematic)
At the start: 1 part

Commit message: change form factor to 80x80 and cleanup pcb
Parts:
- renumbered R8 to R9
Changed lines of the file:
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@@
 		(on_board yes)
 		(dnp no)
-		(property "Reference" "R8"
+		(property "Reference" "R9"
 			(at 48.26 26.4922 90)
 			(effects
@@
 			(project ""
 				(path "/f6cc00ab-17f1-4973-862f-7ac95fe70668/00000000-0000-0000-0000-00005ea31c93/00000000-0000-0000-0000-00005eab0b79"
-					(reference "R8")
+					(reference "R9")
 					(unit 1)
 				)

Commit message: AV: small cleanup, USB, and CAN power
Parts:
- renumbered R9 to R18
Changed lines of the file:
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@@
 		(on_board yes)
 		(dnp no)
-		(property "Reference" "R9"
+		(property "Reference" "R18"
 			(at 48.26 26.4922 90)
 			(effects
@@
 			(project ""
 				(path "/f6cc00ab-17f1-4973-862f-7ac95fe70668/00000000-0000-0000-0000-00005ea31c93/00000000-0000-0000-0000-00005eab0b79"
-					(reference "R9")
+					(reference "R18")
 					(unit 1)
 				)

Commit message: replace nearly all buck converters with boost buck (missing is 5raw
Parts:
- renumbered R18 to R11
Changed lines of the file:
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@@
 		(on_board yes)
 		(dnp no)
-		(property "Reference" "R18"
+		(property "Reference" "R11"
 			(at 48.26 26.4922 90)
 			(effects
@@
 			(project ""
 				(path "/f6cc00ab-17f1-4973-862f-7ac95fe70668/00000000-0000-0000-0000-00005ea31c93/00000000-0000-0000-0000-00005eab0b79"
-					(reference "R18")
+					(reference "R11")
 					(unit 1)
 				)

Commit message: interim checkin before streamlining AVI
Parts:
- R11: Mfr. # RK73Z1JTTD -> (none)
Changed lines of the file:
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@@
-			)
-		)
-		(property "Mfr. #" "RK73Z1JTTD"
-			(at 48.26 31.75 0)
-			(effects
-				(font
-					(size 1.27 1.27)
-				)
-				(hide yes)
 			)
 		)

Commit message: reconcile BOMS for AVI. SCI and AUX
Parts:
- removed R11: 0, Resistor_SMD:R_0603_1608Metric_Pad0.98x0.95mm_HandSolder, symbol Device:R
Changed lines of the file:
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@@
 	(wire
 		(pts
-			(xy 167.64 77.47) (xy 156.21 77.47)
-		)
-		(stroke
-			(width 0)
-			(type default)
-		)
-	)
-	(wire
-		(pts
-			(xy 40.64 31.75) (xy 44.45 31.75)
+			(xy 167.64 77.47) (xy 163.83 77.47)
 		)
 		(stroke
@@
 	(wire
 		(pts
-			(xy 167.64 54.61) (xy 156.21 54.61)
+			(xy 167.64 54.61) (xy 163.83 54.61)
 		)
 		(stroke
@@
 	(wire
 		(pts
-			(xy 106.68 124.46) (xy 95.25 124.46)
+			(xy 106.68 124.46) (xy 100.965 124.46)
 		)
 		(stroke
@@
 	(wire
 		(pts
-			(xy 52.07 31.75) (xy 63.5 31.75)
-		)
-		(stroke
-			(width 0)
-			(type default)
-		)
-	)
-	(wire
-		(pts
 			(xy 163.83 57.15) (xy 167.64 57.15)
 		)
@@
 	(wire
 		(pts
-			(xy 106.68 77.47) (xy 95.25 77.47)
-		)
-		(stroke
-			(width 0)
-			(type default)
-		)
-	)
-	(wire
-		(pts
-			(xy 167.64 124.46) (xy 156.21 124.46)
+			(xy 106.68 77.47) (xy 101.6 77.47)
+		)
+		(stroke
+			(width 0)
+			(type default)
+		)
+	)
+	(wire
+		(pts
+			(xy 167.64 124.46) (xy 163.83 124.46)
 		)
 		(stroke
@@
 	(wire
 		(pts
-			(xy 106.68 53.34) (xy 95.25 53.34)
+			(xy 106.68 53.34) (xy 101.6 53.34)
 		)
 		(stroke
@@
 	(wire
 		(pts
-			(xy 167.64 101.6) (xy 156.21 101.6)
+			(xy 167.64 101.6) (xy 163.83 101.6)
 		)
 		(stroke
@@
 	(wire
 		(pts
-			(xy 106.68 100.33) (xy 95.25 100.33)
+			(xy 106.68 100.33) (xy 101.6 100.33)
 		)
 		(stroke
@@
 		)
 	)
-	(label "INTRNL_VDD"
-		(at 95.25 53.34 0)
-		(fields_autoplaced yes)
-		(effects
-			(font
-				(size 1.27 1.27)
-			)
-			(justify left bottom)
-		)
-	)
-	(label "INTRNL_VDD"
-		(at 156.21 54.61 0)
-		(fields_autoplaced yes)
-		(effects
-			(font
-				(size 1.27 1.27)
-			)
-			(justify left bottom)
-		)
-	)
-	(label "INTRNL_VDD"
-		(at 95.25 77.47 0)
-		(fields_autoplaced yes)
-		(effects
-			(font
-				(size 1.27 1.27)
-			)
-			(justify left bottom)
-		)
-	)
-	(label "INTRNL_VDD"
-		(at 63.5 31.75 180)
-		(fields_autoplaced yes)
-		(effects
-			(font
-				(size 1.27 1.27)
-			)
-			(justify right bottom)
-		)
-	)
-	(label "INTRNL_VDD"
-		(at 156.21 77.47 0)
-		(fields_autoplaced yes)
-		(effects
-			(font
-				(size 1.27 1.27)
-			)
-			(justify left bottom)
-		)
-	)
-	(label "INTRNL_VDD"
-		(at 95.25 100.33 0)
-		(fields_autoplaced yes)
-		(effects
-			(font
-				(size 1.27 1.27)
-			)
-			(justify left bottom)
-		)
-	)
-	(label "INTRNL_VDD"
-		(at 95.25 124.46 0)
-		(fields_autoplaced yes)
-		(effects
-			(font
-				(size 1.27 1.27)
-			)
-			(justify left bottom)
-		)
-	)
-	(label "INTRNL_VDD"
-		(at 156.21 101.6 0)
-		(fields_autoplaced yes)
-		(effects
-			(font
-				(size 1.27 1.27)
-			)
-			(justify left bottom)
-		)
-	)
-	(label "INTRNL_VDD"
-		(at 156.21 124.46 0)
-		(fields_autoplaced yes)
-		(effects
-			(font
-				(size 1.27 1.27)
-			)
-			(justify left bottom)
+	(hierarchical_label "VDD"
+		(shape input)
+		(at 163.83 124.46 180)
+		(fields_autoplaced yes)
+		(effects
+			(font
+				(size 1.27 1.27)
+			)
+			(justify right)
 		)
 	)
@@
 		)
 	)
+	(hierarchical_label "VDD"
+		(shape input)
+		(at 163.83 101.6 180)
+		(fields_autoplaced yes)
+		(effects
+			(font
+				(size 1.27 1.27)
+			)
+			(justify right)
+		)
+	)
 	(hierarchical_label "GND"
 		(shape input)
@@
 		)
 	)
+	(hierarchical_label "VDD"
+		(shape input)
+		(at 163.83 54.61 180)
+		(fields_autoplaced yes)
+		(effects
+			(font
+				(size 1.27 1.27)
+			)
+			(justify right)
+		)
+	)
+	(hierarchical_label "VDD"
+		(shape input)
+		(at 163.83 77.47 180)
+		(fields_autoplaced yes)
+		(effects
+			(font
+				(size 1.27 1.27)
+			)
+			(justify right)
+		)
+	)
 	(hierarchical_label "OUT8"
 		(shape output)
@@
 		)
 	)
+	(hierarchical_label "VDD"
+		(shape input)
+		(at 100.965 124.46 180)
+		(fields_autoplaced yes)
+		(effects
+			(font
+				(size 1.27 1.27)
+			)
+			(justify right)
+		)
+	)
 	(hierarchical_label "GND"
 		(shape input)
@@
 		)
 	)
+	(hierarchical_label "VDD"
+		(shape input)
+		(at 101.6 100.33 180)
+		(fields_autoplaced yes)
+		(effects
+			(font
+				(size 1.27 1.27)
+			)
+			(justify right)
+		)
+	)
+	(hierarchical_label "VDD"
+		(shape input)
+		(at 101.6 53.34 180)
+		(fields_autoplaced yes)
+		(effects
+			(font
+				(size 1.27 1.27)
+			)
+			(justify right)
+		)
+	)
 	(hierarchical_label "OUT6"
 		(shape output)
@@
 	(hierarchical_label "VDD"
 		(shape input)
-		(at 40.64 31.75 180)
+		(at 101.6 77.47 180)
 		(fields_autoplaced yes)
 		(effects
@@
 		)
 	)
-	(symbol
-		(lib_id "Device:R")
-		(at 48.26 31.75 270)
-		(unit 1)
-		(exclude_from_sim no)
-		(in_bom yes)
-		(on_board yes)
-		(dnp no)
-		(property "Reference" "R11"
-			(at 48.26 26.4922 90)
-			(effects
-				(font
-					(size 1.27 1.27)
-				)
-			)
-		)
-		(property "Value" "0"
-			(at 48.26 28.8036 90)
-			(effects
-				(font
-					(size 1.27 1.27)
-				)
-			)
-		)
-		(property "Footprint" "Resistor_SMD:R_0603_1608Metric_Pad0.98x0.95mm_HandSolder"
-			(at 48.26 29.972 90)
-			(effects
-				(font
-					(size 1.27 1.27)
-				)
-				(hide yes)
-			)
-		)
-		(property "Datasheet" "~"
-			(at 48.26 31.75 0)
-			(effects
-				(font
-					(size 1.27 1.27)
-				)
-				(hide yes)
-			)
-		)
-		(property "Description" ""
-			(at 48.26 31.75 0)
-			(effects
-				(font
-					(size 1.27 1.27)
-				)
-				(hide yes)
-			)
-		)
-		(property "Order" "https://www.digikey.com/product-detail/en/koa-speer-electronics-inc/RK73Z1JTTD/2019-RK73Z1JTTDCT-ND/9847522"
-			(at 48.26 31.75 0)
-			(effects
-				(font
-					(size 1.27 1.27)
-				)
-				(hide yes)
-			)
-		)
-		(property "Alt" ""
-			(at 48.26 31.75 0)
-			(effects
-				(font
-					(size 1.27 1.27)
-				)
-				(hide yes)
-			)
-		)
-		(pin "1"
-		)
-		(pin "2"
-		)
-		(instances
-			(project "AVIONICS_BOARD"
-				(path "/f6cc00ab-17f1-4973-862f-7ac95fe70668/4b32b6cb-e4ab-41a8-b61c-93e0ce1b94ae"
-					(reference "R11")
-					(unit 1)
-				)
-			)
-		)
-	)
