File: avionics_board/WATCHDOG.kicad_sch (KiCad schematic)
At the start: 5 parts, among them SW1 EVP-AA602W, SW2 SW_DIP_x01, U6 TPL5010

Commit message: sorting out pullups on resets and attention. replace reset with RN where possible. Introduce CN to save some parts
Parts:
- renumbered C34 to C25, R20 to R5, U6 to U4
Changed lines of the file:
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@@
 		(dnp no)
 		(fields_autoplaced yes)
-		(property "Reference" "U6"
+		(property "Reference" "U4"
 			(at 158.75 82.5814 0)
 			(effects
@@
 		(on_board yes)
 		(dnp no)
-		(property "Reference" "C34"
+		(property "Reference" "C25"
 			(at 123.571 77.5716 0)
 			(effects
@@
 			(project "EPS"
 				(path "/05170af6-30ef-4c3a-b972-f098085da1bc/099fb907-8e0d-460a-bca0-f0390fc6b64a"
-					(reference "C29")
+					(reference "C25")
 					(unit 1)
 				)
@@
 		(on_board yes)
 		(dnp no)
-		(property "Reference" "R20"
+		(property "Reference" "R5"
 			(at 177.038 97.8916 0)
 			(effects
@@
 			(project "EPS"
 				(path "/05170af6-30ef-4c3a-b972-f098085da1bc/099fb907-8e0d-460a-bca0-f0390fc6b64a"
-					(reference "R4")
-					(unit 1)
-				)
+					(reference "R5")
+					(unit 1)
+				)

Commit message: cleanup pullups for reset and schmitt trigger for reset; select available thermal NTCs for avi board and use chip for voltage dividers
Parts:
- renumbered C25 to C34, R5 to R20, U4 to U6
Changed lines of the file:
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@@
 		(dnp no)
 		(fields_autoplaced yes)
-		(property "Reference" "U4"
+		(property "Reference" "U6"
 			(at 158.75 82.5814 0)
 			(effects
@@
 		(on_board yes)
 		(dnp no)
-		(property "Reference" "C25"
+		(property "Reference" "C34"
 			(at 123.571 77.5716 0)
 			(effects
@@
 		(on_board yes)
 		(dnp no)
-		(property "Reference" "R5"
+		(property "Reference" "R20"
 			(at 177.038 97.8916 0)
 			(effects

Commit message: checked BOM for sci wo switches
Parts:
- R11: renamed from R20; value 8K87 -> 22K; Part Number RC0402FR-078K87L -> RC0402FR-078K22KL
- renumbered C34 to C40, U6 to U7
Other:
- note added: "1 min"
- note added: "First 9 Time Intervals tIP (ms) Resistance (Ω) Closest Real Value (Ω) 100 500 500 200 1000 1000 300 1500 1500 400 2000 2000 500 2500 2500 600 3000 3000 700 3500 3500 800 4000 4000 900 4500 4501 Most Common Time Intervals Between 1s to 1min tIP Calculated Resistance (kΩ) Closest Real Value (kΩ) 1s 5.20 5.202 2s 6.79 6.788 3s 7.64 7.628 4s 8.30 8.306 5s 8.85 8.852 6s 9.27 9.223 7s 9.71 9.673 8s 10.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"
- note removed: "5 seconds"
- note removed: "Use 1% Resistors 100 ms == 500 ohm 200 ms == 1000 ohm 300 ms == 1500 ohm 400 ms == 2000 ohm 500 ms == 2500 ohm 1 s == 5.2 Kohm 2 s == 6.79 Kohm 5 s == 8.85 Kohm 10 s == 11.20 Kohm"
Changed lines of the file:
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@@
 		)
 	)
-	(text "5 seconds"
+	(text "First 9 Time Intervals\ntIP (ms) Resistance (Ω) Closest Real Value (Ω)\n100 500 500\n200 1000 1000\n300 1500 1500\n400 2000 2000\n500 2500 2500\n600 3000 3000\n700 3500 3500\n800 4000 4000\n900 4500 4501\n\nMost Common Time Intervals Between 1s to 1min\ntIP Calculated Resistance (kΩ) Closest Real Value (kΩ)\n1s 5.20 5.202\n2s 6.79 6.788\n3s 7.64 7.628\n4s 8.30 8.306\n5s 8.85 8.852\n6s 9.27 9.223\n7s 9.71 9.673\n8s 10.18 10.180\n9s 10.68 10.68\n10s 11.20 11.199\n20s 14.41 14.405\n30s 16.78 16.778\n40s 18.75 18.748\n50s 20.047 20.047\n\nMost Common Time Intervals Between 1min to 2h\ntIP Calculated Resistance (kΩ) Closest Real Value (kΩ)\n1min 22.02 22.021\n2min 29.35 29.349\n3min 34.73 34.729\n4min 39.11 39.097\n5min 42.90 42.887\n6min 46.29 46.301\n7min 49.38 49.392\n8min 52.24 52.224\n9min 54.92 54.902\n10min 57.44 57.437\n20min 77.57 77.579\n30min 92.43 92.233\n40min 104.67 104.625\n50min 115.33 115.331\n1h 124.91 124.856\n1h30min 149.39 149.398\n2h 170.00 170.00"
+		(exclude_from_sim no)
+		(at 46.99 97.79 0)
+		(effects
+			(font
+				(size 1.27 1.27)
+			)
+		)
+	)
+	(text "1 min"
 		(exclude_from_sim no)
 		(at 172.72 99.06 0)
@@
 			)
 			(justify right bottom)
-		)
-	)
-	(text "Use 1% Resistors\n\n100 ms == 500 ohm\n200 ms == 1000 ohm\n300 ms == 1500 ohm\n400 ms == 2000 ohm\n500 ms == 2500 ohm\n1 s     ==  5.2 Kohm\n2 s     == 6.79 Kohm\n5 s     == 8.85 Kohm\n10 s    == 11.20 Kohm"
-		(exclude_from_sim no)
-		(at 195.58 118.11 0)
-		(effects
-			(font
-				(size 1.27 1.27)
-			)
-			(justify left bottom)
 		)
 	)
@@
 		(dnp no)
 		(fields_autoplaced yes)
-		(property "Reference" "U6"
+		(property "Reference" "U7"
 			(at 158.75 82.5814 0)
 			(effects
@@
 			(project ""
 				(path "/f6cc00ab-17f1-4973-862f-7ac95fe70668/00000000-0000-0000-0000-00005ea31c93/00000000-0000-0000-0000-00005eab0a1f"
-					(reference "U6")
+					(reference "U7")
 					(unit 1)
 				)
@@
 		(on_board yes)
 		(dnp no)
-		(property "Reference" "C34"
+		(property "Reference" "C40"
 			(at 123.571 77.5716 0)
 			(effects
@@
 			(project ""
 				(path "/f6cc00ab-17f1-4973-862f-7ac95fe70668/00000000-0000-0000-0000-00005ea31c93/00000000-0000-0000-0000-00005eab0a1f"
-					(reference "C34")
+					(reference "C40")
 					(unit 1)
 				)
@@
 		(on_board yes)
 		(dnp no)
-		(property "Reference" "R20"
+		(property "Reference" "R11"
 			(at 177.038 97.8916 0)
 			(effects
@@
 			)
 		)
-		(property "Value" "8K87"
+		(property "Value" "22K"
 			(at 177.038 100.203 0)
 			(effects
@@
 			)
 		)
-		(property "Part Number" "RC0402FR-078K87L"
+		(property "Part Number" "RC0402FR-078K22KL"
 			(at 175.26 99.06 0)
 			(effects
@@
 			(project ""
 				(path "/f6cc00ab-17f1-4973-862f-7ac95fe70668/00000000-0000-0000-0000-00005ea31c93/00000000-0000-0000-0000-00005eab0a1f"
-					(reference "R20")
-					(unit 1)
-				)
+					(reference "R11")
+					(unit 1)
+				)

Commit message: BOM avi checked
Parts:
- R11: Part Number RC0402FR-078K22KL -> RC0402FR-0722KL
- SW2: value SW_DIP_x01 -> Conn_01x02_Pin Vertical
Changed lines of the file:
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@@
 			)
 		)
-		(property "Description" "Timer, Nano Power, Watchdog, 35 nA, 100 ms to 7200 s, VDD 1.8V to 5.5V, Iout max 1mA"
+		(property "Description" "IC OSC PROG TIMER TSOT23-6"
 			(at 140.97 88.9 0)
 			(effects
@@
 			)
 		)
-		(property "Value" "SW_DIP_x01"
+		(property "Value" "Conn_01x02_Pin Vertical"
 			(at 104.14 81.8896 0)
 			(effects
@@
 			)
 		)
-		(property "Description" ""
+		(property "Description" "Conn_01x02_Pin Vertical"
 			(at 104.14 86.36 0)
 			(effects
@@
 			)
 		)
-		(property "Part Number" "RC0402FR-078K22KL"
+		(property "Part Number" "RC0402FR-0722KL"
 			(at 175.26 99.06 0)
 			(effects
@@
 			)
 		)
-		(property "Description" ""
+		(property "Description" "SPST"
 			(at 175.26 73.66 0)
 			(effects

Commit message: EPS needs flash to self update with bootloader
Parts:
- renumbered C40 to C25, R11 to R5, U7 to U4
Changed lines of the file:
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@@
 		(dnp no)
 		(fields_autoplaced yes)
-		(property "Reference" "U7"
+		(property "Reference" "U4"
 			(at 158.75 82.5814 0)
 			(effects
@@
 		(on_board yes)
 		(dnp no)
-		(property "Reference" "C40"
+		(property "Reference" "C25"
 			(at 123.571 77.5716 0)
 			(effects
@@
 		(on_board yes)
 		(dnp no)
-		(property "Reference" "R11"
+		(property "Reference" "R5"
 			(at 177.038 97.8916 0)
 			(effects

Commit message: power traces and vias of AUX and SCIlite are 0,5mm and 0.5/1.0mm
Parts:
- renumbered C25 to C40, R5 to R11, U4 to U7
Changed lines of the file:
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@@
 		(dnp no)
 		(fields_autoplaced yes)
-		(property "Reference" "U4"
+		(property "Reference" "U7"
 			(at 158.75 82.5814 0)
 			(effects
@@
 		(on_board yes)
 		(dnp no)
-		(property "Reference" "C25"
+		(property "Reference" "C40"
 			(at 123.571 77.5716 0)
 			(effects
@@
 		(on_board yes)
 		(dnp no)
-		(property "Reference" "R5"
+		(property "Reference" "R11"
 			(at 177.038 97.8916 0)
 			(effects
@@
 			)
 		)
-		(property "Description" "SPST"
+		(property "Description" "SWITCH TACTILE SPST-NO 0.02A 15V"
 			(at 175.26 73.66 0)
 			(effects

Commit message: reconcile suite
Parts:
- renumbered C40 to C25, R11 to R5, U7 to U4
Changed lines of the file:
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@@
 		(dnp no)
 		(fields_autoplaced yes)
-		(property "Reference" "U7"
+		(property "Reference" "U4"
 			(at 158.75 82.5814 0)
 			(effects
@@
 		(on_board yes)
 		(dnp no)
-		(property "Reference" "C40"
+		(property "Reference" "C25"
 			(at 123.571 77.5716 0)
 			(effects
@@
 		(on_board yes)
 		(dnp no)
-		(property "Reference" "R11"
+		(property "Reference" "R5"
 			(at 177.038 97.8916 0)
 			(effects

Commit message: move SPI CS pullups to outer schema to combine multiple with RNs
Parts:
- renumbered C25 to C40, R5 to R12, U4 to U7
Changed lines of the file:
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@@
 		(dnp no)
 		(fields_autoplaced yes)
-		(property "Reference" "U4"
+		(property "Reference" "U7"
 			(at 158.75 82.5814 0)
 			(effects
@@
 		(on_board yes)
 		(dnp no)
-		(property "Reference" "C25"
+		(property "Reference" "C40"
 			(at 123.571 77.5716 0)
 			(effects
@@
 		(on_board yes)
 		(dnp no)
-		(property "Reference" "R5"
+		(property "Reference" "R12"
 			(at 177.038 97.8916 0)
 			(effects
@@
 			(project ""
 				(path "/f6cc00ab-17f1-4973-862f-7ac95fe70668/00000000-0000-0000-0000-00005ea31c93/00000000-0000-0000-0000-00005eab0a1f"
-					(reference "R11")
-					(unit 1)
-				)
+					(reference "R12")
+					(unit 1)
+				)
