File: avionics_board/CAN_TRANSCEIVER.kicad_sch (KiCad schematic)
At the start: 8 parts, among them U10 TCAN3414

Commit message: EPS needs flash to self update with bootloader
Parts:
- renumbered C46 to C31, C47 to C32, C48 to C33, C49 to C34, R13 to R8, R14 to R9, U10 to U7
Changed lines of the file:
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@@
 		(on_board yes)
 		(dnp no)
-		(property "Reference" "R13"
+		(property "Reference" "R8"
 			(at 166.878 86.4616 0)
 			(effects
@@
 			(project "sci_board"
 				(path "/b4b2c88d-f6cd-4e60-862d-e21f68728580/1a2691c5-5723-4a0d-b1a6-0fb5069c9e03"
+					(reference "R9")
+					(unit 1)
+				)
+				(path "/b4b2c88d-f6cd-4e60-862d-e21f68728580/5e856d8a-328e-413a-92b7-9cd181b0cc6b"
 					(reference "R7")
-					(unit 1)
-				)
-				(path "/b4b2c88d-f6cd-4e60-862d-e21f68728580/5e856d8a-328e-413a-92b7-9cd181b0cc6b"
-					(reference "R5")
 					(unit 1)
 				)
@@
 		(on_board yes)
 		(dnp no)
-		(property "Reference" "R14"
+		(property "Reference" "R9"
 			(at 166.878 94.0816 0)
 			(effects
@@
 			(project "sci_board"
 				(path "/b4b2c88d-f6cd-4e60-862d-e21f68728580/1a2691c5-5723-4a0d-b1a6-0fb5069c9e03"
+					(reference "R10")
+					(unit 1)
+				)
+				(path "/b4b2c88d-f6cd-4e60-862d-e21f68728580/5e856d8a-328e-413a-92b7-9cd181b0cc6b"
 					(reference "R8")
-					(unit 1)
-				)
-				(path "/b4b2c88d-f6cd-4e60-862d-e21f68728580/5e856d8a-328e-413a-92b7-9cd181b0cc6b"
-					(reference "R6")
 					(unit 1)
 				)
@@
 		(on_board yes)
 		(dnp no)
-		(property "Reference" "C47"
+		(property "Reference" "C32"
 			(at 177.165 88.265 90)
 			(effects
@@
 		(on_board yes)
 		(dnp no)
-		(property "Reference" "C49"
+		(property "Reference" "C34"
 			(at 108.331 124.5616 0)
 			(effects
@@
 		(dnp no)
 		(fields_autoplaced yes)
-		(property "Reference" "C46"
+		(property "Reference" "C31"
 			(at 153.035 85.0962 0)
 			(effects
@@
 		(dnp no)
 		(fields_autoplaced yes)
-		(property "Reference" "C48"
+		(property "Reference" "C33"
 			(at 153.035 95.2562 0)
 			(effects
@@
 		(dnp no)
 		(fields_autoplaced yes)
-		(property "Reference" "U10"
+		(property "Reference" "U7"
 			(at 122.8441 78.74 0)
 			(effects

Commit message: power traces and vias of AUX and SCIlite are 0,5mm and 0.5/1.0mm
Parts:
- C17: renamed from C32; value 4.7nF -> 4nF7
- renumbered C31 to C16, C33 to C18, C34 to C19, D6 to D1, R8 to R5, R9 to R6, U7 to U2
Changed lines of the file:
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@@
 		(on_board yes)
 		(dnp no)
-		(property "Reference" "R8"
+		(property "Reference" "R5"
 			(at 166.878 86.4616 0)
 			(effects
@@
 			(project "sci_board"
 				(path "/b4b2c88d-f6cd-4e60-862d-e21f68728580/1a2691c5-5723-4a0d-b1a6-0fb5069c9e03"
-					(reference "R9")
+					(reference "R7")
 					(unit 1)
 				)
 				(path "/b4b2c88d-f6cd-4e60-862d-e21f68728580/5e856d8a-328e-413a-92b7-9cd181b0cc6b"
-					(reference "R7")
+					(reference "R5")
 					(unit 1)
 				)
@@
 		(on_board yes)
 		(dnp no)
-		(property "Reference" "R9"
+		(property "Reference" "R6"
 			(at 166.878 94.0816 0)
 			(effects
@@
 			(project "sci_board"
 				(path "/b4b2c88d-f6cd-4e60-862d-e21f68728580/1a2691c5-5723-4a0d-b1a6-0fb5069c9e03"
-					(reference "R10")
+					(reference "R8")
 					(unit 1)
 				)
 				(path "/b4b2c88d-f6cd-4e60-862d-e21f68728580/5e856d8a-328e-413a-92b7-9cd181b0cc6b"
-					(reference "R8")
+					(reference "R6")
 					(unit 1)
 				)
@@
 		(on_board yes)
 		(dnp yes)
-		(property "Reference" "D6"
+		(property "Reference" "D1"
 			(at 193.04 85.725 90)
 			(effects
@@
 		(on_board yes)
 		(dnp no)
-		(property "Reference" "C32"
+		(property "Reference" "C17"
 			(at 177.165 88.265 90)
 			(effects
@@
 			)
 		)
-		(property "Value" "4.7nF"
+		(property "Value" "4nF7"
 			(at 177.8 95.25 90)
 			(effects
@@
 		(on_board yes)
 		(dnp no)
-		(property "Reference" "C34"
+		(property "Reference" "C19"
 			(at 108.331 124.5616 0)
 			(effects
@@
 		(dnp no)
 		(fields_autoplaced yes)
-		(property "Reference" "C31"
+		(property "Reference" "C16"
 			(at 153.035 85.0962 0)
 			(effects
@@
 		(dnp no)
 		(fields_autoplaced yes)
-		(property "Reference" "C33"
+		(property "Reference" "C18"
 			(at 153.035 95.2562 0)
 			(effects
@@
 		(dnp no)
 		(fields_autoplaced yes)
-		(property "Reference" "U7"
+		(property "Reference" "U2"
 			(at 122.8441 78.74 0)
 			(effects

Commit message: reconcile suite
Parts:
- renumbered C16 to C31, C17 to C32, C18 to C33, C19 to C34, D1 to D6, R5 to R8, R6 to R9, U2 to U7
Changed lines of the file:
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@@
 		(on_board yes)
 		(dnp no)
-		(property "Reference" "R5"
+		(property "Reference" "R8"
 			(at 166.878 86.4616 0)
 			(effects
@@
 			(project "sci_board"
 				(path "/b4b2c88d-f6cd-4e60-862d-e21f68728580/1a2691c5-5723-4a0d-b1a6-0fb5069c9e03"
+					(reference "R9")
+					(unit 1)
+				)
+				(path "/b4b2c88d-f6cd-4e60-862d-e21f68728580/5e856d8a-328e-413a-92b7-9cd181b0cc6b"
 					(reference "R7")
-					(unit 1)
-				)
-				(path "/b4b2c88d-f6cd-4e60-862d-e21f68728580/5e856d8a-328e-413a-92b7-9cd181b0cc6b"
-					(reference "R5")
 					(unit 1)
 				)
@@
 		(on_board yes)
 		(dnp no)
-		(property "Reference" "R6"
+		(property "Reference" "R9"
 			(at 166.878 94.0816 0)
 			(effects
@@
 			(project "sci_board"
 				(path "/b4b2c88d-f6cd-4e60-862d-e21f68728580/1a2691c5-5723-4a0d-b1a6-0fb5069c9e03"
+					(reference "R10")
+					(unit 1)
+				)
+				(path "/b4b2c88d-f6cd-4e60-862d-e21f68728580/5e856d8a-328e-413a-92b7-9cd181b0cc6b"
 					(reference "R8")
-					(unit 1)
-				)
-				(path "/b4b2c88d-f6cd-4e60-862d-e21f68728580/5e856d8a-328e-413a-92b7-9cd181b0cc6b"
-					(reference "R6")
 					(unit 1)
 				)
@@
 		(on_board yes)
 		(dnp yes)
-		(property "Reference" "D1"
+		(property "Reference" "D6"
 			(at 193.04 85.725 90)
 			(effects
@@
 		(on_board yes)
 		(dnp no)
-		(property "Reference" "C17"
+		(property "Reference" "C32"
 			(at 177.165 88.265 90)
 			(effects
@@
 		(on_board yes)
 		(dnp no)
-		(property "Reference" "C19"
+		(property "Reference" "C34"
 			(at 108.331 124.5616 0)
 			(effects
@@
 		(dnp no)
 		(fields_autoplaced yes)
-		(property "Reference" "C16"
+		(property "Reference" "C31"
 			(at 153.035 85.0962 0)
 			(effects
@@
 		(dnp no)
 		(fields_autoplaced yes)
-		(property "Reference" "C18"
+		(property "Reference" "C33"
 			(at 153.035 95.2562 0)
 			(effects
@@
 		(dnp no)
 		(fields_autoplaced yes)
-		(property "Reference" "U2"
+		(property "Reference" "U7"
 			(at 122.8441 78.74 0)
 			(effects

Commit message: move SPI CS pullups to outer schema to combine multiple with RNs
Parts:
- renumbered C31 to C16, C32 to C17, C33 to C18, C34 to C19, D6 to D1, R8 to R6, R9 to R7, U7 to U2
Changed lines of the file:
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@@
 		(on_board yes)
 		(dnp no)
-		(property "Reference" "R8"
+		(property "Reference" "R6"
 			(at 166.878 86.4616 0)
 			(effects
@@
 			(project "EPS"
 				(path "/05170af6-30ef-4c3a-b972-f098085da1bc/00000000-0000-0000-0000-00005fbffcb6/00000000-0000-0000-0000-0000602b3abb"
-					(reference "R8")
+					(reference "R7")
 					(unit 1)
 				)
 				(path "/05170af6-30ef-4c3a-b972-f098085da1bc/00000000-0000-0000-0000-00005fbffcb6/17eaa29e-6d79-4e5a-8640-52ffcb1a20e4"
-					(reference "R10")
+					(reference "R9")
 					(unit 1)
 				)
@@
 			(project ""
 				(path "/a863a5ec-a5d4-4f54-be53-e8c01d5e3ac4/53f12969-e593-459a-9671-cc23a5a9aea0/505d7be7-0770-45bf-bc6f-d3bee2934d1d"
-					(reference "R18")
+					(reference "R20")
 					(unit 1)
 				)
@@
 			(project "sci_board"
 				(path "/b4b2c88d-f6cd-4e60-862d-e21f68728580/1a2691c5-5723-4a0d-b1a6-0fb5069c9e03"
-					(reference "R9")
+					(reference "R8")
 					(unit 1)
 				)
 				(path "/b4b2c88d-f6cd-4e60-862d-e21f68728580/5e856d8a-328e-413a-92b7-9cd181b0cc6b"
-					(reference "R7")
+					(reference "R6")
 					(unit 1)
 				)
@@
 		(on_board yes)
 		(dnp no)
-		(property "Reference" "R9"
+		(property "Reference" "R7"
 			(at 166.878 94.0816 0)
 			(effects
@@
 			(project "EPS"
 				(path "/05170af6-30ef-4c3a-b972-f098085da1bc/00000000-0000-0000-0000-00005fbffcb6/00000000-0000-0000-0000-0000602b3abb"
-					(reference "R9")
+					(reference "R8")
 					(unit 1)
 				)
 				(path "/05170af6-30ef-4c3a-b972-f098085da1bc/00000000-0000-0000-0000-00005fbffcb6/17eaa29e-6d79-4e5a-8640-52ffcb1a20e4"
-					(reference "R11")
+					(reference "R10")
 					(unit 1)
 				)
@@
 			(project ""
 				(path "/a863a5ec-a5d4-4f54-be53-e8c01d5e3ac4/53f12969-e593-459a-9671-cc23a5a9aea0/505d7be7-0770-45bf-bc6f-d3bee2934d1d"
-					(reference "R19")
+					(reference "R21")
 					(unit 1)
 				)
@@
 			(project "sci_board"
 				(path "/b4b2c88d-f6cd-4e60-862d-e21f68728580/1a2691c5-5723-4a0d-b1a6-0fb5069c9e03"
-					(reference "R10")
+					(reference "R9")
 					(unit 1)
 				)
 				(path "/b4b2c88d-f6cd-4e60-862d-e21f68728580/5e856d8a-328e-413a-92b7-9cd181b0cc6b"
-					(reference "R8")
+					(reference "R7")
 					(unit 1)
 				)
@@
 		(on_board yes)
 		(dnp yes)
-		(property "Reference" "D6"
+		(property "Reference" "D1"
 			(at 193.04 85.725 90)
 			(effects
@@
 		(on_board yes)
 		(dnp no)
-		(property "Reference" "C32"
+		(property "Reference" "C17"
 			(at 177.165 88.265 90)
 			(effects
@@
 		(on_board yes)
 		(dnp no)
-		(property "Reference" "C34"
+		(property "Reference" "C19"
 			(at 108.331 124.5616 0)
 			(effects
@@
 		(dnp no)
 		(fields_autoplaced yes)
-		(property "Reference" "C31"
+		(property "Reference" "C16"
 			(at 153.035 85.0962 0)
 			(effects
@@
 		(dnp no)
 		(fields_autoplaced yes)
-		(property "Reference" "C33"
+		(property "Reference" "C18"
 			(at 153.035 95.2562 0)
 			(effects
@@
 		(dnp no)
 		(fields_autoplaced yes)
-		(property "Reference" "U7"
+		(property "Reference" "U2"
 			(at 122.8441 78.74 0)
 			(effects

Commit message: 06102025 SCI lite and AVI
Parts:
- C46: renamed from C16; Temperature Coefficient (none) -> C0G/NP0; Temperture Coefficient C0G/NP0 -> (none)
- C47: renamed from C17; Temperature Coefficient (none) -> X5R; Temperture Coefficient X5R -> (none)
- C48: renamed from C18; Temperature Coefficient (none) -> C0G/NP0; Temperture Coefficient C0G/NP0 -> (none)
- C49: renamed from C19; Temperature Coefficient (none) -> X5R; Temperture Coefficient X5R -> (none)
- renumbered D1 to D6, R6 to R13, R7 to R14, U2 to U10
Changed lines of the file:
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@@
 		(on_board yes)
 		(dnp no)
-		(property "Reference" "R6"
+		(property "Reference" "R13"
 			(at 166.878 86.4616 0)
 			(effects
@@
 		)
 		(property "Color" ""
-			(at 165.1 87.63 0)
-			(effects
-				(font
-					(size 1.27 1.27)
-				)
-				(hide yes)
-			)
-		)
-		(property "Temperture Coefficient" ""
 			(at 165.1 87.63 0)
 			(effects
@@
 		(on_board yes)
 		(dnp no)
-		(property "Reference" "R7"
+		(property "Reference" "R14"
 			(at 166.878 94.0816 0)
 			(effects
@@
 		)
 		(property "Color" ""
-			(at 165.1 95.25 0)
-			(effects
-				(font
-					(size 1.27 1.27)
-				)
-				(hide yes)
-			)
-		)
-		(property "Temperture Coefficient" ""
 			(at 165.1 95.25 0)
 			(effects
@@
 		(on_board yes)
 		(dnp yes)
-		(property "Reference" "D1"
+		(property "Reference" "D6"
 			(at 193.04 85.725 90)
 			(effects
@@
 		)
 		(property "Color" ""
-			(at 193.04 91.44 0)
-			(effects
-				(font
-					(size 1.27 1.27)
-				)
-				(hide yes)
-			)
-		)
-		(property "Temperture Coefficient" ""
 			(at 193.04 91.44 0)
 			(effects
@@
 		(on_board yes)
 		(dnp no)
-		(property "Reference" "C17"
+		(property "Reference" "C47"
 			(at 177.165 88.265 90)
 			(effects
@@
 			)
 		)
-		(property "Temperture Coefficient" "X5R"
-			(at 175.26 91.44 0)
-			(effects
-				(font
-					(size 1.27 1.27)
-				)
-				(hide yes)
-			)
-		)
 		(property "Manufacturer" "Murata"
 			(at 175.26 91.44 0)
@@
 		)
 		(property "Alt" ""
+			(at 175.26 91.44 90)
+			(effects
+				(font
+					(size 1.27 1.27)
+				)
+				(hide yes)
+			)
+		)
+		(property "Temperature Coefficient" "X5R"
 			(at 175.26 91.44 90)
 			(effects
@@
 		(on_board yes)
 		(dnp no)
-		(property "Reference" "C19"
+		(property "Reference" "C49"
 			(at 108.331 124.5616 0)
 			(effects
@@
 			)
 		)
-		(property "Temperture Coefficient" "X5R"
-			(at 105.41 125.73 0)
-			(effects
-				(font
-					(size 1.27 1.27)
-				)
-				(hide yes)
-			)
-		)
 		(property "Manufacturer" "Murata"
 			(at 105.41 125.73 0)
@@
 		)
 		(property "Alt" ""
+			(at 105.41 125.73 0)
+			(effects
+				(font
+					(size 1.27 1.27)
+				)
+				(hide yes)
+			)
+		)
+		(property "Temperature Coefficient" "X5R"
 			(at 105.41 125.73 0)
 			(effects
@@
 		(dnp no)
 		(fields_autoplaced yes)
-		(property "Reference" "C16"
+		(property "Reference" "C46"
 			(at 153.035 85.0962 0)
 			(effects
@@
 			)
 		)
-		(property "Temperture Coefficient" "C0G/NP0"
-			(at 149.86 86.36 0)
-			(effects
-				(font
-					(size 1.27 1.27)
-				)
-				(hide yes)
-			)
-		)
 		(property "Manufacturer" "Murata"
 			(at 149.86 86.36 0)
@@
 		)
 		(property "Alt" ""
+			(at 149.86 86.36 0)
+			(effects
+				(font
+					(size 1.27 1.27)
+				)
+				(hide yes)
+			)
+		)
+		(property "Temperature Coefficient" "C0G/NP0"
 			(at 149.86 86.36 0)
 			(effects
@@
 		(dnp no)
 		(fields_autoplaced yes)
-		(property "Reference" "C18"
+		(property "Reference" "C48"
 			(at 153.035 95.2562 0)
 			(effects
@@
 			)
 		)
-		(property "Temperture Coefficient" "C0G/NP0"
-			(at 149.86 96.52 0)
-			(effects
-				(font
-					(size 1.27 1.27)
-				)
-				(hide yes)
-			)
-		)
 		(property "Manufacturer" "Murata"
 			(at 149.86 96.52 0)
@@
 		)
 		(property "Alt" ""
+			(at 149.86 96.52 0)
+			(effects
+				(font
+					(size 1.27 1.27)
+				)
+				(hide yes)
+			)
+		)
+		(property "Temperature Coefficient" "C0G/NP0"
 			(at 149.86 96.52 0)
 			(effects
@@
 		(dnp no)
 		(fields_autoplaced yes)
-		(property "Reference" "U2"
+		(property "Reference" "U10"
 			(at 122.8441 78.74 0)
 			(effects
@@
 			(at 120.65 91.44 0)
 			(effects
-				(font
-					(size 1.27 1.27)
-				)
-				(hide yes)
-			)
-		)
-		(property "Temperture Coefficient" ""
-			(at 120.65 91.44 0)
-			(effects

Commit message: all projects satisfy custom rule of min pad spacing 0.2mm to satisfy pcbway constraints
Parts:
- renumbered C46 to C16, C47 to C17, C48 to C18, C49 to C19, D6 to D1, R13 to R10, R14 to R11, U10 to U2
Changed lines of the file:
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@@
 		(on_board yes)
 		(dnp no)
-		(property "Reference" "R13"
+		(property "Reference" "R10"
 			(at 166.878 86.4616 0)
 			(effects
@@
 			(project "sci_board"
 				(path "/b4b2c88d-f6cd-4e60-862d-e21f68728580/1a2691c5-5723-4a0d-b1a6-0fb5069c9e03"
-					(reference "R8")
+					(reference "R12")
 					(unit 1)
 				)
 				(path "/b4b2c88d-f6cd-4e60-862d-e21f68728580/5e856d8a-328e-413a-92b7-9cd181b0cc6b"
-					(reference "R6")
+					(reference "R10")
 					(unit 1)
 				)
@@
 		(on_board yes)
 		(dnp no)
-		(property "Reference" "R14"
+		(property "Reference" "R11"
 			(at 166.878 94.0816 0)
 			(effects
@@
 			(project "sci_board"
 				(path "/b4b2c88d-f6cd-4e60-862d-e21f68728580/1a2691c5-5723-4a0d-b1a6-0fb5069c9e03"
-					(reference "R9")
+					(reference "R13")
 					(unit 1)
 				)
 				(path "/b4b2c88d-f6cd-4e60-862d-e21f68728580/5e856d8a-328e-413a-92b7-9cd181b0cc6b"
-					(reference "R7")
+					(reference "R11")
 					(unit 1)
 				)
@@
 		(on_board yes)
 		(dnp yes)
-		(property "Reference" "D6"
+		(property "Reference" "D1"
 			(at 193.04 85.725 90)
 			(effects
@@
 		(on_board yes)
 		(dnp no)
-		(property "Reference" "C47"
+		(property "Reference" "C17"
 			(at 177.165 88.265 90)
 			(effects
@@
 		(on_board yes)
 		(dnp no)
-		(property "Reference" "C49"
+		(property "Reference" "C19"
 			(at 108.331 124.5616 0)
 			(effects
@@
 		(dnp no)
 		(fields_autoplaced yes)
-		(property "Reference" "C46"
+		(property "Reference" "C16"
 			(at 153.035 85.0962 0)
 			(effects
@@
 		(dnp no)
 		(fields_autoplaced yes)
-		(property "Reference" "C48"
+		(property "Reference" "C18"
 			(at 153.035 95.2562 0)
 			(effects
@@
 		(dnp no)
 		(fields_autoplaced yes)
-		(property "Reference" "U10"
+		(property "Reference" "U2"
 			(at 122.8441 78.74 0)
 			(effects

Commit message: EPS board add RTC battery
Parts:
- renumbered C16 to C32, C17 to C33, C18 to C34, C19 to C35, D1 to D6, R10 to R7, R11 to R8, U2 to U7
Changed lines of the file:
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@@
 		(on_board yes)
 		(dnp no)
-		(property "Reference" "R10"
+		(property "Reference" "R7"
 			(at 166.878 86.4616 0)
 			(effects
@@
 		(on_board yes)
 		(dnp no)
-		(property "Reference" "R11"
+		(property "Reference" "R8"
 			(at 166.878 94.0816 0)
 			(effects
@@
 		(on_board yes)
 		(dnp yes)
-		(property "Reference" "D1"
+		(property "Reference" "D6"
 			(at 193.04 85.725 90)
 			(effects
@@
 		(on_board yes)
 		(dnp no)
-		(property "Reference" "C17"
+		(property "Reference" "C33"
 			(at 177.165 88.265 90)
 			(effects
@@
 			(project "EPS"
 				(path "/05170af6-30ef-4c3a-b972-f098085da1bc/00000000-0000-0000-0000-00005fbffcb6/00000000-0000-0000-0000-0000602b3abb"
-					(reference "C32")
+					(reference "C33")
 					(unit 1)
 				)
 				(path "/05170af6-30ef-4c3a-b972-f098085da1bc/00000000-0000-0000-0000-00005fbffcb6/17eaa29e-6d79-4e5a-8640-52ffcb1a20e4"
-					(reference "C36")
+					(reference "C37")
 					(unit 1)
 				)
@@
 		(on_board yes)
 		(dnp no)
-		(property "Reference" "C19"
+		(property "Reference" "C35"
 			(at 108.331 124.5616 0)
 			(effects
@@
 			(project "EPS"
 				(path "/05170af6-30ef-4c3a-b972-f098085da1bc/00000000-0000-0000-0000-00005fbffcb6/00000000-0000-0000-0000-0000602b3abb"
-					(reference "C34")
+					(reference "C35")
 					(unit 1)
 				)
 				(path "/05170af6-30ef-4c3a-b972-f098085da1bc/00000000-0000-0000-0000-00005fbffcb6/17eaa29e-6d79-4e5a-8640-52ffcb1a20e4"
-					(reference "C38")
+					(reference "C39")
 					(unit 1)
 				)
@@
 		(dnp no)
 		(fields_autoplaced yes)
-		(property "Reference" "C16"
+		(property "Reference" "C32"
 			(at 153.035 85.0962 0)
 			(effects
@@
 			(project "EPS"
 				(path "/05170af6-30ef-4c3a-b972-f098085da1bc/00000000-0000-0000-0000-00005fbffcb6/00000000-0000-0000-0000-0000602b3abb"
-					(reference "C31")
+					(reference "C32")
 					(unit 1)
 				)
 				(path "/05170af6-30ef-4c3a-b972-f098085da1bc/00000000-0000-0000-0000-00005fbffcb6/17eaa29e-6d79-4e5a-8640-52ffcb1a20e4"
-					(reference "C35")
+					(reference "C36")
 					(unit 1)
 				)
@@
 		(dnp no)
 		(fields_autoplaced yes)
-		(property "Reference" "C18"
+		(property "Reference" "C34"
 			(at 153.035 95.2562 0)
 			(effects
@@
 			(project "EPS"
 				(path "/05170af6-30ef-4c3a-b972-f098085da1bc/00000000-0000-0000-0000-00005fbffcb6/00000000-0000-0000-0000-0000602b3abb"
-					(reference "C33")
+					(reference "C34")
 					(unit 1)
 				)
 				(path "/05170af6-30ef-4c3a-b972-f098085da1bc/00000000-0000-0000-0000-00005fbffcb6/17eaa29e-6d79-4e5a-8640-52ffcb1a20e4"
-					(reference "C37")
+					(reference "C38")
 					(unit 1)
 				)
@@
 		(dnp no)
 		(fields_autoplaced yes)
-		(property "Reference" "U2"
+		(property "Reference" "U7"
 			(at 122.8441 78.74 0)
 			(effects
