File: avionics_board/DEBUG_INTERFACE.kicad_sch (KiCad schematic)
At the start: 8 parts, among them J5 Conn_01x05_Pin Vertical, J6 Conn_01x04_Pin Vertical

Commit message: power traces and vias of AUX and SCIlite are 0,5mm and 0.5/1.0mm
Parts:
- renumbered D1 to D3, D2 to D4, D3 to D5, D4 to D6, D5 to D7, J5 to J8, J6 to J9, RN11 to RN10
Changed lines of the file:
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@@
 		(on_board yes)
 		(dnp yes)
-		(property "Reference" "J6"
+		(property "Reference" "J9"
 			(at 214.0712 103.6828 0)
 			(effects
@@
 		(on_board yes)
 		(dnp no)
-		(property "Reference" "D1"
+		(property "Reference" "D3"
 			(at 219.71 45.9486 0)
 			(effects
@@
 		(on_board yes)
 		(dnp no)
-		(property "Reference" "D4"
+		(property "Reference" "D6"
 			(at 219.71 60.96 0)
 			(effects
@@
 		(on_board yes)
 		(dnp no)
-		(property "Reference" "D2"
+		(property "Reference" "D4"
 			(at 219.71 51.0286 0)
 			(effects
@@
 		(on_board yes)
 		(dnp no)
-		(property "Reference" "D3"
+		(property "Reference" "D5"
 			(at 219.71 56.1086 0)
 			(effects
@@
 		(on_board yes)
 		(dnp no)
-		(property "Reference" "D5"
+		(property "Reference" "D7"
 			(at 219.71 66.2686 0)
 			(effects
@@
 		(on_board yes)
 		(dnp yes)
-		(property "Reference" "J5"
+		(property "Reference" "J8"
 			(at 58.42 44.4501 0)
 			(effects
@@
 		(on_board yes)
 		(dnp no)
-		(property "Reference" "RN11"
+		(property "Reference" "RN10"
 			(at 189.865 40.64 0)
 			(effects

Commit message: BOM avi checked
Parts:
- renumbered D3 to D1, D4 to D2, D5 to D3, D6 to D4, D7 to D5, J8 to J13, J9 to J14, RN10 to RN11
Changed lines of the file:
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@@
 		(on_board yes)
 		(dnp yes)
-		(property "Reference" "J9"
+		(property "Reference" "J14"
 			(at 214.0712 103.6828 0)
 			(effects
@@
 		(on_board yes)
 		(dnp no)
-		(property "Reference" "D3"
+		(property "Reference" "D1"
 			(at 219.71 45.9486 0)
 			(effects
@@
 		(on_board yes)
 		(dnp no)
-		(property "Reference" "D6"
+		(property "Reference" "D4"
 			(at 219.71 60.96 0)
 			(effects
@@
 		(on_board yes)
 		(dnp no)
-		(property "Reference" "D4"
+		(property "Reference" "D2"
 			(at 219.71 51.0286 0)
 			(effects
@@
 		(on_board yes)
 		(dnp no)
-		(property "Reference" "D5"
+		(property "Reference" "D3"
 			(at 219.71 56.1086 0)
 			(effects
@@
 		(on_board yes)
 		(dnp no)
-		(property "Reference" "D7"
+		(property "Reference" "D5"
 			(at 219.71 66.2686 0)
 			(effects
@@
 		(on_board yes)
 		(dnp yes)
-		(property "Reference" "J8"
+		(property "Reference" "J13"
 			(at 58.42 44.4501 0)
 			(effects
@@
 		(on_board yes)
 		(dnp no)
-		(property "Reference" "RN10"
+		(property "Reference" "RN11"
 			(at 189.865 40.64 0)
 			(effects

Commit message: EPS needs flash to self update with bootloader
Parts:
- renumbered J13 to J5, J14 to J6
Changed lines of the file:
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@@
 		(on_board yes)
 		(dnp yes)
-		(property "Reference" "J14"
+		(property "Reference" "J6"
 			(at 214.0712 103.6828 0)
 			(effects
@@
 		(on_board yes)
 		(dnp yes)
-		(property "Reference" "J13"
+		(property "Reference" "J5"
 			(at 58.42 44.4501 0)
 			(effects

Commit message: move SPI CS pullups to outer schema to combine multiple with RNs
Parts:
- renumbered D1 to D3, D2 to D4, D3 to D5, D4 to D6, D5 to D7, J5 to J8, J6 to J9
Changed lines of the file:
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@@
 		(on_board yes)
 		(dnp yes)
-		(property "Reference" "J6"
+		(property "Reference" "J9"
 			(at 214.0712 103.6828 0)
 			(effects
@@
 		(on_board yes)
 		(dnp no)
-		(property "Reference" "D1"
+		(property "Reference" "D3"
 			(at 219.71 45.9486 0)
 			(effects
@@
 		(on_board yes)
 		(dnp no)
-		(property "Reference" "D4"
+		(property "Reference" "D6"
 			(at 219.71 60.96 0)
 			(effects
@@
 		(on_board yes)
 		(dnp no)
-		(property "Reference" "D2"
+		(property "Reference" "D4"
 			(at 219.71 51.0286 0)
 			(effects
@@
 		(on_board yes)
 		(dnp no)
-		(property "Reference" "D3"
+		(property "Reference" "D5"
 			(at 219.71 56.1086 0)
 			(effects
@@
 		(on_board yes)
 		(dnp no)
-		(property "Reference" "D5"
+		(property "Reference" "D7"
 			(at 219.71 66.2686 0)
 			(effects
@@
 		(on_board yes)
 		(dnp yes)
-		(property "Reference" "J5"
+		(property "Reference" "J8"
 			(at 58.42 44.4501 0)
 			(effects
@@
 			(project "sci_board"
 				(path "/b4b2c88d-f6cd-4e60-862d-e21f68728580/840799ac-4fe6-4a8e-96a2-299affeec8e4/3a4f04a3-bf3f-413a-bc77-fd47ed49c088"
-					(reference "RN10")
-					(unit 1)
-				)
+					(reference "RN11")
+					(unit 1)
+				)

Commit message: 06102025 SCI lite and AVI
Parts:
- renumbered D3 to D1, D4 to D2, D5 to D3, D6 to D4, D7 to D5, J8 to J13, J9 to J14
Changed lines of the file:
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@@
 		(on_board yes)
 		(dnp yes)
-		(property "Reference" "J9"
+		(property "Reference" "J14"
 			(at 214.0712 103.6828 0)
 			(effects
@@
 		)
 		(property "Description" "Generic connector, single row, 01x04, script generated"
-			(at 213.36 106.68 0)
-			(effects
-				(font
-					(size 1.27 1.27)
-				)
-				(hide yes)
-			)
-		)
-		(property "Temperture Coefficient" ""
 			(at 213.36 106.68 0)
 			(effects
@@
 		(on_board yes)
 		(dnp no)
-		(property "Reference" "D3"
+		(property "Reference" "D1"
 			(at 219.71 45.9486 0)
 			(effects
@@
 		)
 		(property "Voltage" "2"
-			(at 204.47 46.99 0)
-			(effects
-				(font
-					(size 1.27 1.27)
-				)
-				(hide yes)
-			)
-		)
-		(property "Temperture Coefficient" ""
 			(at 204.47 46.99 0)
 			(effects
@@
 		(on_board yes)
 		(dnp no)
-		(property "Reference" "D6"
+		(property "Reference" "D4"
 			(at 219.71 60.96 0)
 			(effects
@@
 		)
 		(property "Voltage" "2"
-			(at 204.47 62.23 0)
-			(effects
-				(font
-					(size 1.27 1.27)
-				)
-				(hide yes)
-			)
-		)
-		(property "Temperture Coefficient" ""
 			(at 204.47 62.23 0)
 			(effects
@@
 		(on_board yes)
 		(dnp no)
-		(property "Reference" "D4"
+		(property "Reference" "D2"
 			(at 219.71 51.0286 0)
 			(effects
@@
 		)
 		(property "Voltage" "2"
-			(at 204.47 52.07 0)
-			(effects
-				(font
-					(size 1.27 1.27)
-				)
-				(hide yes)
-			)
-		)
-		(property "Temperture Coefficient" ""
 			(at 204.47 52.07 0)
 			(effects
@@
 		(on_board yes)
 		(dnp no)
-		(property "Reference" "D5"
+		(property "Reference" "D3"
 			(at 219.71 56.1086 0)
 			(effects
@@
 		)
 		(property "Voltage" "2"
-			(at 204.47 57.15 0)
-			(effects
-				(font
-					(size 1.27 1.27)
-				)
-				(hide yes)
-			)
-		)
-		(property "Temperture Coefficient" ""
 			(at 204.47 57.15 0)
 			(effects
@@
 		(on_board yes)
 		(dnp no)
-		(property "Reference" "D7"
+		(property "Reference" "D5"
 			(at 219.71 66.2686 0)
 			(effects
@@
 		)
 		(property "Voltage" "2"
-			(at 204.47 67.31 0)
-			(effects
-				(font
-					(size 1.27 1.27)
-				)
-				(hide yes)
-			)
-		)
-		(property "Temperture Coefficient" ""
 			(at 204.47 67.31 0)
 			(effects
@@
 		(on_board yes)
 		(dnp yes)
-		(property "Reference" "J8"
+		(property "Reference" "J13"
 			(at 58.42 44.4501 0)
 			(effects
@@
 			(at 56.515 44.45 0)
 			(effects
-				(font
-					(size 1.27 1.27)
-				)
-				(hide yes)
-			)
-		)
-		(property "Temperture Coefficient" ""
-			(at 56.515 44.45 0)
-			(effects

Commit message: all projects satisfy custom rule of min pad spacing 0.2mm to satisfy pcbway constraints
Parts:
- renumbered D1 to D3, D2 to D4, D3 to D5, D4 to D6, D5 to D7, J13 to J8, J14 to J9, RN11 to RN10
Changed lines of the file:
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@@
 		(on_board yes)
 		(dnp yes)
-		(property "Reference" "J14"
+		(property "Reference" "J9"
 			(at 214.0712 103.6828 0)
 			(effects
@@
 		(on_board yes)
 		(dnp no)
-		(property "Reference" "D1"
+		(property "Reference" "D3"
 			(at 219.71 45.9486 0)
 			(effects
@@
 		(on_board yes)
 		(dnp no)
-		(property "Reference" "D4"
+		(property "Reference" "D6"
 			(at 219.71 60.96 0)
 			(effects
@@
 		(on_board yes)
 		(dnp no)
-		(property "Reference" "D2"
+		(property "Reference" "D4"
 			(at 219.71 51.0286 0)
 			(effects
@@
 		(on_board yes)
 		(dnp no)
-		(property "Reference" "D3"
+		(property "Reference" "D5"
 			(at 219.71 56.1086 0)
 			(effects
@@
 		(on_board yes)
 		(dnp no)
-		(property "Reference" "D5"
+		(property "Reference" "D7"
 			(at 219.71 66.2686 0)
 			(effects
@@
 		(on_board yes)
 		(dnp yes)
-		(property "Reference" "J13"
+		(property "Reference" "J8"
 			(at 58.42 44.4501 0)
 			(effects
@@
 		(on_board yes)
 		(dnp no)
-		(property "Reference" "RN11"
+		(property "Reference" "RN10"
 			(at 189.865 40.64 0)
 			(effects
@@
 			(project "sci_board"
 				(path "/b4b2c88d-f6cd-4e60-862d-e21f68728580/840799ac-4fe6-4a8e-96a2-299affeec8e4/3a4f04a3-bf3f-413a-bc77-fd47ed49c088"
-					(reference "RN11")
-					(unit 1)
-				)
+					(reference "RN10")
+					(unit 1)
+				)

Commit message: EPS board add RTC battery
Parts:
- renumbered D3 to D1, D4 to D2, D5 to D3, D6 to D4, D7 to D5, J8 to J5, J9 to J6, RN10 to RN11
Changed lines of the file:
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@@
 		(on_board yes)
 		(dnp yes)
-		(property "Reference" "J9"
+		(property "Reference" "J6"
 			(at 214.0712 103.6828 0)
 			(effects
@@
 		(on_board yes)
 		(dnp no)
-		(property "Reference" "D3"
+		(property "Reference" "D1"
 			(at 219.71 45.9486 0)
 			(effects
@@
 		(on_board yes)
 		(dnp no)
-		(property "Reference" "D6"
+		(property "Reference" "D4"
 			(at 219.71 60.96 0)
 			(effects
@@
 		(on_board yes)
 		(dnp no)
-		(property "Reference" "D4"
+		(property "Reference" "D2"
 			(at 219.71 51.0286 0)
 			(effects
@@
 		(on_board yes)
 		(dnp no)
-		(property "Reference" "D5"
+		(property "Reference" "D3"
 			(at 219.71 56.1086 0)
 			(effects
@@
 		(on_board yes)
 		(dnp no)
-		(property "Reference" "D7"
+		(property "Reference" "D5"
 			(at 219.71 66.2686 0)
 			(effects
@@
 		(on_board yes)
 		(dnp yes)
-		(property "Reference" "J8"
+		(property "Reference" "J5"
 			(at 58.42 44.4501 0)
 			(effects
@@
 		(on_board yes)
 		(dnp no)
-		(property "Reference" "RN10"
+		(property "Reference" "RN11"
 			(at 189.865 40.64 0)
 			(effects

Commit message: move project to new location, update sympbol, footprint and step paths
Parts:
- renumbered D1 to D3, D2 to D4, D3 to D5, D4 to D6, D5 to D7, J5 to J8, J6 to J9
Changed lines of the file:
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@@
 		(on_board yes)
 		(dnp yes)
-		(property "Reference" "J6"
+		(property "Reference" "J9"
 			(at 214.0712 103.6828 0)
 			(effects
@@
 		(on_board yes)
 		(dnp no)
-		(property "Reference" "D1"
+		(property "Reference" "D3"
 			(at 219.71 45.9486 0)
 			(effects
@@
 		(on_board yes)
 		(dnp no)
-		(property "Reference" "D4"
+		(property "Reference" "D6"
 			(at 219.71 60.96 0)
 			(effects
@@
 		(on_board yes)
 		(dnp no)
-		(property "Reference" "D2"
+		(property "Reference" "D4"
 			(at 219.71 51.0286 0)
 			(effects
@@
 		(on_board yes)
 		(dnp no)
-		(property "Reference" "D3"
+		(property "Reference" "D5"
 			(at 219.71 56.1086 0)
 			(effects
@@
 		(on_board yes)
 		(dnp no)
-		(property "Reference" "D5"
+		(property "Reference" "D7"
 			(at 219.71 66.2686 0)
 			(effects
@@
 		(on_board yes)
 		(dnp yes)
-		(property "Reference" "J5"
+		(property "Reference" "J8"
 			(at 58.42 44.4501 0)
 			(effects
@@
 			(project "sci_board"
 				(path "/b4b2c88d-f6cd-4e60-862d-e21f68728580/840799ac-4fe6-4a8e-96a2-299affeec8e4/3a4f04a3-bf3f-413a-bc77-fd47ed49c088"
-					(reference "RN10")
-					(unit 1)
-				)
+					(reference "RN11")
+					(unit 1)
+				)
