File: avionics_board/OSC32_TCXO.kicad_sch (KiCad schematic)
At the start: 2 parts, among them X2 32.768KHZ

Commit message: cleanup pullups for reset and schmitt trigger for reset; select available thermal NTCs for avi board and use chip for voltage dividers
Parts:
- renumbered C32 to C38
Changed lines of the file:
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@@
 		(on_board yes)
 		(dnp no)
-		(property "Reference" "C32"
+		(property "Reference" "C38"
 			(at 132.461 122.6566 0)
 			(effects
@@
 			(project "sci_board"
 				(path "/b4b2c88d-f6cd-4e60-862d-e21f68728580/840799ac-4fe6-4a8e-96a2-299affeec8e4/9565b29f-739e-499d-a066-98bd4c80d38b"
-					(reference "C60")
+					(reference "C77")
 					(unit 1)
 				)

Commit message: checked BOM for sci wo switches
Parts:
- X3: renamed from X2; Tolerance (none) -> 25ppm
- renumbered C38 to C60
Changed lines of the file:
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@@
 		(on_board yes)
 		(dnp no)
-		(property "Reference" "X2"
+		(property "Reference" "X3"
 			(at 157.48 113.665 0)
 			(effects
@@
 		)
 		(property "Alt" ""
+			(at 137.16 123.19 0)
+			(effects
+				(font
+					(size 1.27 1.27)
+				)
+				(hide yes)
+			)
+		)
+		(property "Tolerance" "25ppm"
 			(at 137.16 123.19 0)
 			(effects
@@
 		(on_board yes)
 		(dnp no)
-		(property "Reference" "C38"
+		(property "Reference" "C60"
 			(at 132.461 122.6566 0)
 			(effects
@@
 			(project "sci_board"
 				(path "/b4b2c88d-f6cd-4e60-862d-e21f68728580/840799ac-4fe6-4a8e-96a2-299affeec8e4/9565b29f-739e-499d-a066-98bd4c80d38b"
-					(reference "C77")
+					(reference "C60")
 					(unit 1)
 				)
@@
 			(project "AVIONICS_BOARD"
 				(path "/f6cc00ab-17f1-4973-862f-7ac95fe70668/00000000-0000-0000-0000-00005ea31c93/00000000-0000-0000-0000-00006310c56a"
-					(reference "C38")
-					(unit 1)
-				)
+					(reference "C44")
+					(unit 1)
+				)

Commit message: 06102025 SCI lite and AVI
Parts:
- C44: renamed from C60; Temperature Coefficient (none) -> X5R; Temperture Coefficient X5R -> (none)
- renumbered X3 to X2
Changed lines of the file:
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@@
 		(on_board yes)
 		(dnp no)
-		(property "Reference" "X3"
+		(property "Reference" "X2"
 			(at 157.48 113.665 0)
 			(effects
@@
 		(on_board yes)
 		(dnp no)
-		(property "Reference" "C60"
+		(property "Reference" "C44"
 			(at 132.461 122.6566 0)
 			(effects
@@
 			)
 		)
-		(property "Temperture Coefficient" "X5R"
-			(at 129.54 123.825 0)
-			(effects
-				(font
-					(size 1.27 1.27)
-				)
-				(hide yes)
-			)
-		)
 		(property "Manufacturer" "Murata"
 			(at 129.54 123.825 0)
@@
 			(at 129.54 123.825 0)
 			(effects
+				(font
+					(size 1.27 1.27)
+				)
+				(hide yes)
+			)
+		)
+		(property "Temperature Coefficient" "X5R"
+			(at 129.54 123.825 0)
+			(effects

Commit message: all projects satisfy custom rule of min pad spacing 0.2mm to satisfy pcbway constraints
Parts:
- renumbered C44 to C77, X2 to X3
Changed lines of the file:
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@@
 		(on_board yes)
 		(dnp no)
-		(property "Reference" "X2"
+		(property "Reference" "X3"
 			(at 157.48 113.665 0)
 			(effects
@@
 		(on_board yes)
 		(dnp no)
-		(property "Reference" "C44"
+		(property "Reference" "C77"
 			(at 132.461 122.6566 0)
 			(effects
@@
 			(project "sci_board"
 				(path "/b4b2c88d-f6cd-4e60-862d-e21f68728580/840799ac-4fe6-4a8e-96a2-299affeec8e4/9565b29f-739e-499d-a066-98bd4c80d38b"
-					(reference "C60")
-					(unit 1)
-				)
+					(reference "C77")
+					(unit 1)
+				)

Commit message: EPS board add RTC battery
Parts:
- renumbered C77 to C27, X3 to X1
Changed lines of the file:
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@@
 		(on_board yes)
 		(dnp no)
-		(property "Reference" "X3"
+		(property "Reference" "X1"
 			(at 157.48 113.665 0)
 			(effects
@@
 		(on_board yes)
 		(dnp no)
-		(property "Reference" "C77"
+		(property "Reference" "C27"
 			(at 132.461 122.6566 0)
 			(effects
@@
 			(project "EPS"
 				(path "/05170af6-30ef-4c3a-b972-f098085da1bc/00000000-0000-0000-0000-00005fbffcb6/00000000-0000-0000-0000-00005fedb823"
-					(reference "C26")
-					(unit 1)
-				)
+					(reference "C27")
+					(unit 1)
+				)

Commit message: move project to new location, update sympbol, footprint and step paths
Parts:
- renumbered C27 to C60, X1 to X3
Changed lines of the file:
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@@
 		(on_board yes)
 		(dnp no)
-		(property "Reference" "X1"
+		(property "Reference" "X3"
 			(at 157.48 113.665 0)
 			(effects
@@
 		(on_board yes)
 		(dnp no)
-		(property "Reference" "C27"
+		(property "Reference" "C60"
 			(at 132.461 122.6566 0)
 			(effects
@@
 			(project "sci_board"
 				(path "/b4b2c88d-f6cd-4e60-862d-e21f68728580/840799ac-4fe6-4a8e-96a2-299affeec8e4/9565b29f-739e-499d-a066-98bd4c80d38b"
-					(reference "C77")
-					(unit 1)
-				)
+					(reference "C60")
+					(unit 1)
+				)

Commit message: VRef+ meeds to be connected to VDDA, should not be left floating
Parts:
- renumbered C60 to C77
Changed lines of the file:
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@@
 		(on_board yes)
 		(dnp no)
-		(property "Reference" "C60"
+		(property "Reference" "C77"
 			(at 132.461 122.6566 0)
 			(effects
@@
 			(project "sci_board"
 				(path "/b4b2c88d-f6cd-4e60-862d-e21f68728580/840799ac-4fe6-4a8e-96a2-299affeec8e4/9565b29f-739e-499d-a066-98bd4c80d38b"
-					(reference "C60")
+					(reference "C77")
 					(unit 1)
 				)

Commit message: SCI bodge board to correct I2C switching
Parts:
- renumbered C77 to C60
Changed lines of the file:
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@@
 		(on_board yes)
 		(dnp no)
-		(property "Reference" "C77"
+		(property "Reference" "C60"
 			(at 132.461 122.6566 0)
 			(effects
@@
 			(project "sci_board"
 				(path "/b4b2c88d-f6cd-4e60-862d-e21f68728580/840799ac-4fe6-4a8e-96a2-299affeec8e4/9565b29f-739e-499d-a066-98bd4c80d38b"
-					(reference "C77")
+					(reference "C60")
 					(unit 1)
 				)
