File: sci_board_wo_switches/camera.kicad_sch (KiCad schematic)
At the start: 7 parts, among them J3 10051922-2410EHLF

Commit message: first version of sci wo switches
Parts:
- added C26: 22pF, Capacitor_SMD:C_0402_1005Metric_Pad0.74x0.62mm_HandSolder, symbol Device:C
- added C27: 100nF, Capacitor_SMD:C_0402_1005Metric_Pad0.74x0.62mm_HandSolder, symbol Device:C
- added R12, R13: 100K, Resistor_SMD:R_0402_1005Metric_Pad0.72x0.64mm_HandSolder, symbol Device:R
Connections:
- net *RESET: now also C27.1, R12.2
- net 1V8: now also R12.1
- net DCMI_PLXCLK: now also C26.1
- net GND: now also C26.2, C27.2, R13.2
- net PWRDN: now also R13.1
