File: sci_board_wo_switches/dual_switch.kicad_sch (KiCad schematic)
At the start: 7 parts, among them U6 TPS22968QDMGRQ1

Commit message: first version of sci wo switches
Parts:
- renumbered C50 to C67, C51 to C68, C52 to C69, C53 to C70, C54 to C71, C55 to C72, U6 to U13
Changed lines of the file:
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@@
 		(dnp no)
 		(fields_autoplaced yes)
-		(property "Reference" "C52"
+		(property "Reference" "C69"
 			(at 96.52 107.9499 0)
 			(effects
@@
 		(dnp no)
 		(fields_autoplaced yes)
-		(property "Reference" "U6"
+		(property "Reference" "U13"
 			(at 147.32 86.36 0)
 			(effects
@@
 		(dnp yes)
 		(fields_autoplaced yes)
-		(property "Reference" "C50"
+		(property "Reference" "C67"
 			(at 173.99 100.3299 0)
 			(effects
@@
 		(dnp no)
 		(fields_autoplaced yes)
-		(property "Reference" "C55"
+		(property "Reference" "C72"
 			(at 187.96 107.9499 0)
 			(effects
@@
 		(dnp no)
 		(fields_autoplaced yes)
-		(property "Reference" "C53"
+		(property "Reference" "C70"
 			(at 115.57 107.9499 0)
 			(effects
@@
 		(dnp yes)
 		(fields_autoplaced yes)
-		(property "Reference" "C54"
+		(property "Reference" "C71"
 			(at 173.99 107.9499 0)
 			(effects
@@
 		(dnp no)
 		(fields_autoplaced yes)
-		(property "Reference" "C51"
+		(property "Reference" "C68"
 			(at 187.96 100.3299 0)
 			(effects
