File: sci_board_wo_switches/pmic.kicad_sch (KiCad schematic)
At the start: 18 parts, among them J1 Conn_01x03_Pin Vertical, U1 STM32L496VGTx

Commit message: EPS AVI SCI SCIwoSwitches RF AUX all updated to use RNs. BOMs completed
Parts:
- C1, C10, C11, C13, C15, C2: MANUFACTURER Murata -> (none); Manufacturer (none) -> Murata; PARTREV GRM188R61E106KA73D -> (none); Part Number (none) -> GRM188R61E106KA73D
- C12, C14, C3, C4, C5, C6, C7, C8, C9: MANUFACTURER Murata -> (none); Manufacturer (none) -> Murata; PARTREV GRM155R61E104KA87D -> (none); Part Number (none) -> GRM155R61E104KA87D
- FB1: MANUFACTURER Murata -> (none); Manufacturer (none) -> Murata; PARTREV BLM18PG121SN1D -> (none); Part Number (none) -> BLM18PG121SN1D
- J1: MANUFACTURER generic -> (none); Manufacturer (none) -> generic; PARTREV generic -> (none); Part Number (none) -> vertical
- U1: MANUFACTURER STM -> (none); Manufacturer (none) -> STM; PARTREV STM32L496VGT6 -> (none); Part Number (none) -> STM32L496VGT6

Commit message: sorting out pullups on resets and attention. replace reset with RN where possible. Introduce CN to save some parts
Parts:
- added R5: 100K, Resistor_SMD:R_0402_1005Metric_Pad0.72x0.64mm_HandSolder, symbol Device:R
- added R6: 330K, Resistor_SMD:R_0402_1005Metric_Pad0.72x0.64mm_HandSolder, symbol Device:R
- added RN5: 100K, Resistor_SMD:R_Array_Convex_2x0402, symbol Device:R_Pack02
Connections:
- net EXTR_RST: now also RN5.3 (R2.2)
- net RESET: now also RN5.4 (R1.2); no longer U1.14 (NRST)
- net VIO: now also R5.1, R6.1, RN5.1 (R1.1), RN5.2 (R2.1)
- net EXTI2 renamed ATTN_EXTI2
- net ATTN_EXTI2: now also R6.2
- new net NRST: R5.2, U1.14 (NRST)
Other:
- sheet RESET ports: added none; removed VIO

Commit message: cleanup pullups for reset and schmitt trigger for reset; select available thermal NTCs for avi board and use chip for voltage dividers
Parts:
- RN5: footprint Resistor_SMD:R_Array_Convex_2x0402 -> Common:R_Array_Convex_2x0402_widepads
Changed lines of the file:
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@@
 			)
 		)
-		(property "Footprint" "Resistor_SMD:R_Array_Convex_2x0402"
+		(property "Footprint" "Common:R_Array_Convex_2x0402_widepads"
 			(at 26.67 40.64 90)
 			(effects

Commit message: checked BOM for sci wo switches
Parts:
- removed R6: 330K, Resistor_SMD:R_0402_1005Metric_Pad0.72x0.64mm_HandSolder, symbol Device:R
- renumbered R5 to R4, RN5 to RN6
Connections:
- net I2C2_RST: now reaches U1.47 (PB10)
- no-connect marks 5 -> 4
Other:
- note removed: "SPI2_SCK"
Changed lines of the file:
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@@
 	(generator_version "9.0")
 	(paper "A4")
-	(text "SPI2_SCK"
-		(exclude_from_sim no)
-		(at 160.02 125.73 0)
-		(effects
-			(font
-				(size 1.27 1.27)
-			)
-			(justify left)
-		)
-	)
 	(junction
 		(at 99.695 17.145)
@@
 	)
 	(no_connect
-		(at 158.75 125.73)
-	)
-	(no_connect
 		(at 210.185 85.09)
 	)
@@
 		)
 	)
-	(hierarchical_label "VIO"
-		(shape input)
-		(at 85.09 118.11 0)
-		(effects
-			(font
-				(size 1.27 1.27)
-			)
-			(justify left)
-		)
-	)
 	(hierarchical_label "ENABLE_A"
 		(shape output)
@@
 		)
 	)
-	(hierarchical_label "ATTN_EXTI2"
-		(shape input)
-		(at 85.09 125.73 180)
-		(effects
-			(font
-				(size 1.27 1.27)
-			)
-			(justify right)
-		)
-	)
 	(hierarchical_label "VIO"
 		(shape input)
@@
 		)
 	)
+	(hierarchical_label "I2C2_RST"
+		(shape output)
+		(at 158.75 125.73 0)
+		(effects
+			(font
+				(size 1.27 1.27)
+			)
+			(justify left)
+		)
+	)
 	(hierarchical_label "CAN1_TX"
 		(shape input)
@@
 		(on_board yes)
 		(dnp no)
-		(property "Reference" "R5"
+		(property "Reference" "R4"
 			(at 102.87 52.705 0)
 			(effects
@@
 				)
 				(justify left)
-				(hide yes)
 			)
 		)
@@
 			)
 		)
-		(property "Datasheet" "https://www.yageo.com/upload/media/product/app/datasheet/rchip/pyu-rt_1-to-0.01_rohs_l.pdf"
+		(property "Datasheet" "https://www.yageo.com/upload/media/product/products/datasheet/rchip/PYu-RC_Group_51_RoHS_L_12.pdf"
 			(at 100.965 53.34 0)
 			(effects
@@
 			(project "sci_board_wo_switches"
 				(path "/b4b2c88d-f6cd-4e60-862d-e21f68728580/840799ac-4fe6-4a8e-96a2-299affeec8e4"
-					(reference "R5")
+					(reference "R4")
 					(unit 1)
 				)
@@
 		(on_board yes)
 		(dnp no)
-		(property "Reference" "RN5"
+		(property "Reference" "RN6"
 			(at 25.4 38.1 0)
 			(effects
@@
 			(project "sci_board_wo_switches"
 				(path "/b4b2c88d-f6cd-4e60-862d-e21f68728580/840799ac-4fe6-4a8e-96a2-299affeec8e4"
-					(reference "RN5")
+					(reference "RN6")
 					(unit 1)
 				)
@@
 					(unit 1)
 				)
-			)
-		)
-	)
-	(symbol
-		(lib_id "Device:R")
-		(at 85.09 121.92 0)
-		(unit 1)
-		(exclude_from_sim no)
-		(in_bom yes)
-		(on_board yes)
-		(dnp no)
-		(property "Reference" "R6"
-			(at 88.265 121.285 0)
-			(effects
-				(font
-					(size 1.27 1.27)
-				)
-				(justify left)
-			)
-		)
-		(property "Value" "330K"
-			(at 88.265 123.825 0)
-			(effects
-				(font
-					(size 1.27 1.27)
-				)
-				(justify left)
-			)
-		)
-		(property "Footprint" "Resistor_SMD:R_0402_1005Metric_Pad0.72x0.64mm_HandSolder"
-			(at 83.312 121.92 90)
-			(effects
-				(font
-					(size 1.27 1.27)
-				)
-				(hide yes)
-			)
-		)
-		(property "Datasheet" "https://www.yageo.com/upload/media/product/products/datasheet/rchip/PYu-RC_Group_51_RoHS_L_12.pdf"
-			(at 85.09 121.92 0)
-			(effects
-				(font
-					(size 1.27 1.27)
-				)
-				(hide yes)
-			)
-		)
-		(property "Description" "Resistor"
-			(at 85.09 121.92 0)
-			(effects
-				(font
-					(size 1.27 1.27)
-				)
-				(hide yes)
-			)
-		)
-		(property "Note" "generic pullup/down"
-			(at 85.09 121.92 0)
-			(effects
-				(font
-					(size 1.27 1.27)
-				)
-				(hide yes)
-			)
-		)
-		(property "Tolerance" "1"
-			(at 85.09 121.92 0)
-			(effects
-				(font
-					(size 1.27 1.27)
-				)
-				(hide yes)
-			)
-		)
-		(property "Manufacturer" "YAGEO"
-			(at 85.09 121.92 0)
-			(effects
-				(font
-					(size 1.27 1.27)
-				)
-				(hide yes)
-			)
-		)
-		(property "Part Number" "RC0402FR-07330KL"
-			(at 85.09 121.92 0)
-			(effects
-				(font
-					(size 1.27 1.27)
-				)
-				(hide yes)
-			)
-		)
-		(pin "2"
-		)
-		(pin "1"
-		)
-		(instances
-			(project "sci_board_wo_switches"
-				(path "/b4b2c88d-f6cd-4e60-862d-e21f68728580/840799ac-4fe6-4a8e-96a2-299affeec8e4"
-					(reference "R6")
-					(unit 1)
-				)

Commit message: move SPI CS pullups to outer schema to combine multiple with RNs
Parts:
- renumbered R4 to R5, RN6 to RN7
Changed lines of the file:
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@@
 		(on_board yes)
 		(dnp no)
-		(property "Reference" "R4"
+		(property "Reference" "R5"
 			(at 102.87 52.705 0)
 			(effects
@@
 			(project "sci_board_wo_switches"
 				(path "/b4b2c88d-f6cd-4e60-862d-e21f68728580/840799ac-4fe6-4a8e-96a2-299affeec8e4"
-					(reference "R4")
+					(reference "R5")
 					(unit 1)
 				)
@@
 		(on_board yes)
 		(dnp no)
-		(property "Reference" "RN6"
+		(property "Reference" "RN7"
 			(at 25.4 38.1 0)
 			(effects
@@
 			(project "sci_board_wo_switches"
 				(path "/b4b2c88d-f6cd-4e60-862d-e21f68728580/840799ac-4fe6-4a8e-96a2-299affeec8e4"
-					(reference "RN6")
+					(reference "RN7")
 					(unit 1)
 				)

Commit message: VRef+ meeds to be connected to VDDA, should not be left floating
Connections:
- net VDDA: now reaches C14.2, C15.2, U1.21 (VREF+)
- net VDDA: now also C10.1, C9.1, FB1.2, U1.22 (VDDA)
Changed lines of the file:
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@@
+		)
+	)
+	(label "VDDA"
+		(at 143.51 47.625 90)
+		(effects
+			(font
+				(size 1.27 1.27)
+			)
+			(justify left bottom)
 		)
 	)
@@
 		)
 	)
+	(label "VDDA"
+		(at 96.52 62.23 180)
+		(effects
+			(font
+				(size 1.27 1.27)
+			)
+			(justify right bottom)
+		)
+	)

Commit message: SCI bodge board to correct I2C switching
Connections:
- net GPIO1 renamed CAM_ENABLE_CLK
- net I2C2_RST renamed I2C1_RST
Changed lines of the file:
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@@
 		)
 	)
-	(hierarchical_label "GPIO1"
+	(hierarchical_label "CAM_ENABLE_CLK"
 		(shape output)
 		(at 158.75 171.45 0)
@@
 		)
 	)
-	(hierarchical_label "I2C2_RST"
+	(hierarchical_label "I2C1_RST"
 		(shape output)
 		(at 158.75 125.73 0)

Commit message: move legacy schema and files into inactive folders for removal
Other:
- sheet BOOT: file ../avionics_board/boot.kicad_sch -> ../common/sheets/boot.kicad_sch
- sheet DEBUG_INTERFACE: file ../avionics_board/DEBUG_INTERFACE.kicad_sch -> ../common/sheets/DEBUG_INTERFACE.kicad_sch
- sheet OSC32_TCXO: file ../avionics_board/OSC32_TCXO.kicad_sch -> ../common/sheets/OSC32_TCXO.kicad_sch
- sheet OSC_HSE_TCXO: file ../avionics_board/OSC_HSE_TCXO.kicad_sch -> ../common/sheets/OSC_HSE_TCXO.kicad_sch
- sheet RESET: file reset.kicad_sch -> ../common/sheets/reset.kicad_sch
- sheet RESET_ST: file ../avionics_board/schmitt_trigger.kicad_sch -> ../common/sheets/schmitt_trigger.kicad_sch
- sheet USB Connector: file ../avionics_board/USB.kicad_sch -> ../common/sheets/USB.kicad_sch
Changed lines of the file:
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@@
 			)
 		)
-		(property "Sheetfile" "../avionics_board/DEBUG_INTERFACE.kicad_sch"
+		(property "Sheetfile" "../common/sheets/DEBUG_INTERFACE.kicad_sch"
 			(at 231.775 161.8746 0)
 			(effects
@@
 			)
 		)
-		(property "Sheetfile" "../avionics_board/USB.kicad_sch"
+		(property "Sheetfile" "../common/sheets/USB.kicad_sch"
 			(at 193.04 92.6596 0)
 			(effects
@@
 				)
 				(justify left top)
-				(hide yes)
 			)
 		)
@@
 			)
 		)
-		(property "Sheetfile" "../avionics_board/OSC32_TCXO.kicad_sch"
+		(property "Sheetfile" "../common/sheets/OSC32_TCXO.kicad_sch"
 			(at 177.165 162.5096 0)
 			(effects
@@
 			)
 		)
-		(property "Sheetfile" "../avionics_board/boot.kicad_sch"
+		(property "Sheetfile" "../common/sheets/boot.kicad_sch"
 			(at 44.45 80.5946 0)
 			(effects
@@
 				)
 				(justify left top)
-				(hide yes)
 			)
 		)
@@
 			)
 		)
-		(property "Sheetfile" "reset.kicad_sch"
+		(property "Sheetfile" "../common/sheets/reset.kicad_sch"
 			(at 17.78 66.6246 0)
 			(effects
@@
 			)
 		)
-		(property "Sheetfile" "../avionics_board/schmitt_trigger.kicad_sch"
+		(property "Sheetfile" "../common/sheets/schmitt_trigger.kicad_sch"
 			(at 41.275 62.865 0)
 			(effects
@@
 				)
 				(justify left top)
-				(hide yes)
 			)
 		)
@@
 			)
 		)
-		(property "Sheetfile" "../avionics_board/OSC_HSE_TCXO.kicad_sch"
+		(property "Sheetfile" "../common/sheets/OSC_HSE_TCXO.kicad_sch"
 			(at 64.77 74.8796 0)
 			(effects
