File: openlst-hw/MCU.kicad_sch (KiCad schematic)
At the start: 39 parts, among them J1 Conn_02x03_Pin, J2 Conn_01x06_Pin, J3 Conn_01x03_Pin, J4 Conn_01x03_Pin, U1 CC1110, U2 MIC803, X1 27MHz

Commit message: rework COM board, add SPI ethernet for sat modem, upgrade all projects to 9.0.2
Parts:
- removed C12, C13: 100nF, Capacitor_SMD:C_0402_1005Metric_Pad0.74x0.62mm_HandSolder, symbol Device:C_Small
- removed R12, R8: 100K, Resistor_SMD:R_0402_1005Metric_Pad0.72x0.64mm_HandSolder, symbol Device:R
- removed R2, R6, R7: 1K, Resistor_SMD:R_0402_1005Metric_Pad0.72x0.64mm_HandSolder, symbol Device:R
- removed R3, R5: 10K, Resistor_SMD:R_0402_1005Metric_Pad0.72x0.64mm_HandSolder, symbol Device:R
- removed U2: MIC803, Package_TO_SOT_SMD:SOT-23_Handsoldering, symbol Project:MIC803
- added RN2: 1K, Resistor_SMD:R_Array_Convex_2x0402, symbol Device:R_Pack02
- added RN3: 10K, Resistor_SMD:R_Array_Convex_2x0402, symbol Device:R_Pack02
- D1: value ORANGE -> LED_SMD_GREEN; Part Number LTST-C191KFKT -> LTST-C191KGKT; Voltage 2.1 -> https://optoelectronics.liteon.com/upload/download/DS22-200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
- D2: value ORANGE -> LED_SMD_YELLOW; Part Number LTST-C191KFKT -> LTST-C191KSKT; Voltage 2.1 -> https://optoelectronics.liteon.com/upload/download/DS22-200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
- J2: now not fitted
- R1: value 47K -> 100K
Connections:
- net 3V3: now also RN3.3 (R2.2)
- net GND: now also RN3.4 (R1.2)
- net LED1: now also RN2.2 (R2.1)
- net LED2: now also RN2.1 (R1.1)
- net LST_RESET: now also U1.31 (RESET_N)
- net LST_RX_MODE: now also RN3.2 (R2.1)
- net LST_TX_MODE: now also RN3.1 (R1.1)
- net at D1.2 (A): now also RN2.3 (R2.2)
- net at D2.2 (A): now also RN2.4 (R1.2)
Other:
- note removed: "140ms delay"
- note removed: "3V Threshold"
- note removed: "Pulldowns to indicate active when CTS and RTS not used"
- moved on the sheet: R1

Commit message: EPS AVI SCI SCIwoSwitches RF AUX all updated to use RNs. BOMs completed
Parts:
- C1, C10, C11, C2, C3, C4, C5, C6, C7, C8, C9: Temperture Coefficient (none) -> X5R
- C12: renamed from C14; Temperture Coefficient (none) -> X5R
- J1, J2, J3, J4: Manufacturer (none) -> generic; Part Number generic -> vertical
- R1: Part Number RC0402FR-0747KL -> RC0402FR-07100KL
- RN1: renamed from RN3; Manufacturer (none) -> Panasonic; Part Number (none) -> EXB-24V103JX; Tolerance (none) -> 5
- RN2: Manufacturer (none) -> Panasonic; Part Number (none) -> EXB-24V102JX; Tolerance (none) -> 5
- renumbered R4 to R2, R9 to R3, R10 to R4, R11 to R5, R13 to R6, R14 to R7, R15 to R8

Commit message: cleanup pullups for reset and schmitt trigger for reset; select available thermal NTCs for avi board and use chip for voltage dividers
Parts:
- RN1, RN2: footprint Resistor_SMD:R_Array_Convex_2x0402 -> Common:R_Array_Convex_2x0402_widepads
Changed lines of the file:
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@@
 			)
 		)
-		(property "Footprint" "Resistor_SMD:R_Array_Convex_2x0402"
+		(property "Footprint" "Common:R_Array_Convex_2x0402_widepads"
 			(at 87.63 99.06 90)
 			(effects
@@
 			)
 		)
-		(property "Footprint" "Resistor_SMD:R_Array_Convex_2x0402"
+		(property "Footprint" "Common:R_Array_Convex_2x0402_widepads"
 			(at 267.335 142.875 90)
 			(effects

Commit message: reconcile suite
Parts:
- D1: value LED_SMD_GREEN -> GREEN
- D2: value LED_SMD_YELLOW -> YELLOW
- X1: Tolerance (none) -> 25ppm
Changed lines of the file:
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@@
+			)
+		)
+		(property "Tolerance" "25ppm"
+			(at 191.77 74.93 0)
+			(effects
+				(font
+					(size 1.27 1.27)
+				)
+				(hide yes)
 			)
 		)
@@
 			)
 		)
-		(property "Value" "LED_SMD_GREEN"
+		(property "Value" "GREEN"
 			(at 257.81 144.78 0)
 			(effects
@@
 			)
 		)
-		(property "Value" "LED_SMD_YELLOW"
+		(property "Value" "YELLOW"
 			(at 257.81 154.94 0)
 			(effects
