File: common/sheets/INTERBOARD_CONNECTOR.kicad_sch (KiCad schematic)
At the start: 1 part, among them J6 PC104 Conn_02x20_Odd_Even

Commit message: move commonly used hierarchical sheets to common/sheets for easy reuse
Parts:
- renumbered J6 to J15
Changed lines of the file:
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@@
 		(on_board yes)
 		(dnp no)
-		(property "Reference" "J6"
+		(property "Reference" "J15"
 			(at 148.59 68.1482 0)
 			(effects

Commit message: absolute paths for includes of includes or the second level common/sheet will cause problems!
Parts:
- renumbered J15 to J6
Changed lines of the file:
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@@
 		(on_board yes)
 		(dnp no)
-		(property "Reference" "J15"
+		(property "Reference" "J6"
 			(at 148.59 68.1482 0)
 			(effects
@@
 				)
 			)
-			(project "sci_board"
+			(project "sci_board_wo_switches"
 				(path "/b4b2c88d-f6cd-4e60-862d-e21f68728580/70ef1311-b406-42d7-8163-c01a0b1d3f33"
 					(reference "J6")

Commit message: move legacy schema and files into inactive folders for removal
Parts:
- renumbered J6 to J15
Changed lines of the file:
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@@
 		(on_board yes)
 		(dnp no)
-		(property "Reference" "J6"
+		(property "Reference" "J15"
 			(at 148.59 68.1482 0)
 			(effects

Commit message: moving common sheets to common, cleanup for some missed files
Parts:
- renumbered J15 to J2
Changed lines of the file:
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@@
 		(on_board yes)
 		(dnp no)
-		(property "Reference" "J15"
+		(property "Reference" "J2"
 			(at 148.59 68.1482 0)
 			(effects

Commit message: cleaning up common sheets and projects. prepare for removal of legacy path links
Parts:
- renumbered J2 to J9
Changed lines of the file:
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@@
 		(on_board yes)
 		(dnp no)
-		(property "Reference" "J2"
+		(property "Reference" "J9"
 			(at 148.59 68.1482 0)
 			(effects
