File: common/sheets/INTERBOARD_CONNECTOR.kicad_sch (KiCad schematic)
At the start: 1 part, among them J9 PC104 Conn_02x20_Odd_Even

Commit message: auxio_board: leverage more IO on aux board
Parts:
- renumbered J9 to J5
Changed lines of the file:
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@@
 		(on_board yes)
 		(dnp no)
-		(property "Reference" "J9"
+		(property "Reference" "J5"
 			(at 148.59 68.1482 0)
 			(effects
@@
 				)
 			)
-			(project "aux_board"
+			(project "auxio_board"
 				(path "/85134265-2435-454a-99c4-e49d8e69c5c2/461cab69-1065-4442-82a5-52a5533db164"
 					(reference "J5")

Commit message: add headers on sci board to accept camera hats
Parts:
- renumbered J5 to J6
Changed lines of the file:
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@@
 		(on_board yes)
 		(dnp no)
-		(property "Reference" "J5"
+		(property "Reference" "J6"
 			(at 148.59 68.1482 0)
 			(effects
@@
 				)
 			)
-			(project "sci_board_wo_switches"
+			(project "sci_board_with_hat"
 				(path "/b4b2c88d-f6cd-4e60-862d-e21f68728580/70ef1311-b406-42d7-8163-c01a0b1d3f33"
 					(reference "J6")
