File: common/sheets/dual_switch.kicad_sch (KiCad schematic)
At the start: 7 parts, among them U6 TPS22968QDMGRQ1

Commit message: move commonly used hierarchical sheets to common/sheets for easy reuse
Parts:
- removed C44, C48: 220pF, Capacitor_SMD:C_0402_1005Metric_Pad0.74x0.62mm_HandSolder, symbol Device:C
- removed C45, C49: 10uF, Capacitor_SMD:C_0603_1608Metric_Pad1.08x0.95mm_HandSolder, symbol Device:C
- removed C46: 22uF, Capacitor_SMD:C_0603_1608Metric_Pad1.08x0.95mm_HandSolder, symbol Device:C
- removed C47: 100nF, Capacitor_SMD:C_0402_1005Metric_Pad0.74x0.62mm_HandSolder, symbol Device:C
- removed U6: TPS22968QDMGRQ1, Package_SON:WSON-10-1EP_2x3mm_P0.5mm_EP0.84x2.4mm, symbol Common:TPS22968QDMGRQ1
- added C1, C5: 220pF, Capacitor_SMD:C_0402_1005Metric_Pad0.74x0.62mm_HandSolder, symbol Device:C
- added C2, C6: 10uF, Capacitor_SMD:C_0603_1608Metric_Pad1.08x0.95mm_HandSolder, symbol Device:C
- added C3: 22uF, Capacitor_SMD:C_0603_1608Metric_Pad1.08x0.95mm_HandSolder, symbol Device:C
- added C4: 100nF, Capacitor_SMD:C_0402_1005Metric_Pad0.74x0.62mm_HandSolder, symbol Device:C
- added U1: TPS22968QDMGRQ1, Package_SON:WSON-10-1EP_2x3mm_P0.5mm_EP0.84x2.4mm, symbol Common:TPS22968QDMGRQ1
Connections:
- net EN1: now also U1.2 (ON1)
- net EN2: now also U1.4 (ON2)
- net GND: now also C1.2, C2.2, C3.2, C4.2, C5.1, C6.1, U1.11 (TPAD), U1.8 (GND)
- net VBIAS: now also C4.1, U1.3 (VBIAS)
- net VIN: now also C3.1, U1.1 (VIN1), U1.5 (VIN2)
- net VOUT1: now also C2.1, U1.10 (VOUT1)
- net VOUT2: now also C6.2, U1.6 (VOUT2)
- new net: C5.2, U1.7 (CT2)
- new net: C1.1, U1.9 (CT1)

Commit message: absolute paths for includes of includes or the second level common/sheet will cause problems!
Parts:
- renumbered C1 to C44, C2 to C45, C3 to C46, C4 to C47, C5 to C48, C6 to C49, U1 to U6
Changed lines of the file:
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@@
 		(dnp no)
 		(fields_autoplaced yes)
-		(property "Reference" "C2"
+		(property "Reference" "C45"
 			(at 187.96 100.3299 0)
 			(effects
@@
 				)
 				(path "/05170af6-30ef-4c3a-b972-f098085da1bc/53211e67-c677-4be8-893d-9825fa308902/0653e279-5ac5-4fd5-819c-e8ef4edad0cf"
-					(reference "C107")
+					(reference "C92")
 					(unit 1)
 				)
@@
 				)
 				(path "/05170af6-30ef-4c3a-b972-f098085da1bc/53211e67-c677-4be8-893d-9825fa308902/a96e8afd-8b3c-4e12-820c-86caa1a14769"
-					(reference "C101")
-					(unit 1)
-				)
-			)
-			(project "openlst-hw"
+					(reference "C86")
+					(unit 1)
+				)
+			)
+			(project "comm_board"
 				(path "/a863a5ec-a5d4-4f54-be53-e8c01d5e3ac4/53f12969-e593-459a-9671-cc23a5a9aea0/158b6ecf-5b25-4ecb-8b1c-83236ab855da/0653e279-5ac5-4fd5-819c-e8ef4edad0cf"
 					(reference "C50")
@@
 		(dnp no)
 		(fields_autoplaced yes)
-		(property "Reference" "C3"
+		(property "Reference" "C46"
 			(at 96.52 107.9499 0)
 			(effects
@@
 				)
 				(path "/05170af6-30ef-4c3a-b972-f098085da1bc/53211e67-c677-4be8-893d-9825fa308902/0653e279-5ac5-4fd5-819c-e8ef4edad0cf"
-					(reference "C108")
+					(reference "C93")
 					(unit 1)
 				)
@@
 				)
 				(path "/05170af6-30ef-4c3a-b972-f098085da1bc/53211e67-c677-4be8-893d-9825fa308902/a96e8afd-8b3c-4e12-820c-86caa1a14769"
-					(reference "C102")
-					(unit 1)
-				)
-			)
-			(project "openlst-hw"
+					(reference "C87")
+					(unit 1)
+				)
+			)
+			(project "comm_board"
 				(path "/a863a5ec-a5d4-4f54-be53-e8c01d5e3ac4/53f12969-e593-459a-9671-cc23a5a9aea0/158b6ecf-5b25-4ecb-8b1c-83236ab855da/0653e279-5ac5-4fd5-819c-e8ef4edad0cf"
 					(reference "C51")
@@
 		(dnp no)
 		(fields_autoplaced yes)
-		(property "Reference" "U1"
+		(property "Reference" "U6"
 			(at 147.32 86.36 0)
 			(effects
@@
 				)
 				(path "/05170af6-30ef-4c3a-b972-f098085da1bc/53211e67-c677-4be8-893d-9825fa308902/0653e279-5ac5-4fd5-819c-e8ef4edad0cf"
-					(reference "U33")
+					(reference "U24")
 					(unit 1)
 				)
@@
 				)
 				(path "/05170af6-30ef-4c3a-b972-f098085da1bc/53211e67-c677-4be8-893d-9825fa308902/a96e8afd-8b3c-4e12-820c-86caa1a14769"
-					(reference "U32")
-					(unit 1)
-				)
-			)
-			(project "openlst-hw"
+					(reference "U23")
+					(unit 1)
+				)
+			)
+			(project "comm_board"
 				(path "/a863a5ec-a5d4-4f54-be53-e8c01d5e3ac4/53f12969-e593-459a-9671-cc23a5a9aea0/158b6ecf-5b25-4ecb-8b1c-83236ab855da/0653e279-5ac5-4fd5-819c-e8ef4edad0cf"
 					(reference "U10")
@@
 		(dnp yes)
 		(fields_autoplaced yes)
-		(property "Reference" "C1"
+		(property "Reference" "C44"
 			(at 173.99 100.3299 0)
 			(effects
@@
 				)
 				(path "/05170af6-30ef-4c3a-b972-f098085da1bc/53211e67-c677-4be8-893d-9825fa308902/0653e279-5ac5-4fd5-819c-e8ef4edad0cf"
-					(reference "C106")
+					(reference "C91")
 					(unit 1)
 				)
@@
 				)
 				(path "/05170af6-30ef-4c3a-b972-f098085da1bc/53211e67-c677-4be8-893d-9825fa308902/a96e8afd-8b3c-4e12-820c-86caa1a14769"
-					(reference "C100")
-					(unit 1)
-				)
-			)
-			(project "openlst-hw"
+					(reference "C85")
+					(unit 1)
+				)
+			)
+			(project "comm_board"
 				(path "/a863a5ec-a5d4-4f54-be53-e8c01d5e3ac4/53f12969-e593-459a-9671-cc23a5a9aea0/158b6ecf-5b25-4ecb-8b1c-83236ab855da/0653e279-5ac5-4fd5-819c-e8ef4edad0cf"
 					(reference "C49")
@@
 		(dnp yes)
 		(fields_autoplaced yes)
-		(property "Reference" "C5"
+		(property "Reference" "C48"
 			(at 173.99 107.9499 0)
 			(effects
@@
 				)
 				(path "/05170af6-30ef-4c3a-b972-f098085da1bc/53211e67-c677-4be8-893d-9825fa308902/0653e279-5ac5-4fd5-819c-e8ef4edad0cf"
-					(reference "C110")
+					(reference "C95")
 					(unit 1)
 				)
@@
 				)
 				(path "/05170af6-30ef-4c3a-b972-f098085da1bc/53211e67-c677-4be8-893d-9825fa308902/a96e8afd-8b3c-4e12-820c-86caa1a14769"
-					(reference "C104")
-					(unit 1)
-				)
-			)
-			(project "openlst-hw"
+					(reference "C89")
+					(unit 1)
+				)
+			)
+			(project "comm_board"
 				(path "/a863a5ec-a5d4-4f54-be53-e8c01d5e3ac4/53f12969-e593-459a-9671-cc23a5a9aea0/158b6ecf-5b25-4ecb-8b1c-83236ab855da/0653e279-5ac5-4fd5-819c-e8ef4edad0cf"
 					(reference "C53")
@@
 		(dnp no)
 		(fields_autoplaced yes)
-		(property "Reference" "C6"
+		(property "Reference" "C49"
 			(at 187.96 107.9499 0)
 			(effects
@@
 				)
 				(path "/05170af6-30ef-4c3a-b972-f098085da1bc/53211e67-c677-4be8-893d-9825fa308902/0653e279-5ac5-4fd5-819c-e8ef4edad0cf"
-					(reference "C111")
+					(reference "C96")
 					(unit 1)
 				)
@@
 				)
 				(path "/05170af6-30ef-4c3a-b972-f098085da1bc/53211e67-c677-4be8-893d-9825fa308902/a96e8afd-8b3c-4e12-820c-86caa1a14769"
-					(reference "C105")
-					(unit 1)
-				)
-			)
-			(project "openlst-hw"
+					(reference "C90")
+					(unit 1)
+				)
+			)
+			(project "comm_board"
 				(path "/a863a5ec-a5d4-4f54-be53-e8c01d5e3ac4/53f12969-e593-459a-9671-cc23a5a9aea0/158b6ecf-5b25-4ecb-8b1c-83236ab855da/0653e279-5ac5-4fd5-819c-e8ef4edad0cf"
 					(reference "C54")
@@
 		(dnp no)
 		(fields_autoplaced yes)
-		(property "Reference" "C4"
+		(property "Reference" "C47"
 			(at 115.57 107.9499 0)
 			(effects
@@
 				)
 				(path "/05170af6-30ef-4c3a-b972-f098085da1bc/53211e67-c677-4be8-893d-9825fa308902/0653e279-5ac5-4fd5-819c-e8ef4edad0cf"
-					(reference "C109")
+					(reference "C94")
 					(unit 1)
 				)
@@
 				)
 				(path "/05170af6-30ef-4c3a-b972-f098085da1bc/53211e67-c677-4be8-893d-9825fa308902/a96e8afd-8b3c-4e12-820c-86caa1a14769"
-					(reference "C103")
-					(unit 1)
-				)
-			)
-			(project "openlst-hw"
+					(reference "C88")
+					(unit 1)
+				)
+			)
+			(project "comm_board"
 				(path "/a863a5ec-a5d4-4f54-be53-e8c01d5e3ac4/53f12969-e593-459a-9671-cc23a5a9aea0/158b6ecf-5b25-4ecb-8b1c-83236ab855da/0653e279-5ac5-4fd5-819c-e8ef4edad0cf"
 					(reference "C52")

Commit message: move legacy schema and files into inactive folders for removal
Parts:
- renumbered C44 to C61, C45 to C62, C46 to C63, C47 to C64, C48 to C65, C49 to C66, U6 to U16
Changed lines of the file:
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@@
 		(dnp no)
 		(fields_autoplaced yes)
-		(property "Reference" "C45"
+		(property "Reference" "C62"
 			(at 187.96 100.3299 0)
 			(effects
@@
 		(dnp no)
 		(fields_autoplaced yes)
-		(property "Reference" "C46"
+		(property "Reference" "C63"
 			(at 96.52 107.9499 0)
 			(effects
@@
 		(dnp no)
 		(fields_autoplaced yes)
-		(property "Reference" "U6"
+		(property "Reference" "U16"
 			(at 147.32 86.36 0)
 			(effects
@@
 		(dnp yes)
 		(fields_autoplaced yes)
-		(property "Reference" "C44"
+		(property "Reference" "C61"
 			(at 173.99 100.3299 0)
 			(effects
@@
 		(dnp yes)
 		(fields_autoplaced yes)
-		(property "Reference" "C48"
+		(property "Reference" "C65"
 			(at 173.99 107.9499 0)
 			(effects
@@
 		(dnp no)
 		(fields_autoplaced yes)
-		(property "Reference" "C49"
+		(property "Reference" "C66"
 			(at 187.96 107.9499 0)
 			(effects
@@
 		(dnp no)
 		(fields_autoplaced yes)
-		(property "Reference" "C47"
+		(property "Reference" "C64"
 			(at 115.57 107.9499 0)
 			(effects

Commit message: moving common sheets to common, cleanup for some missed files
Parts:
- C30: renamed from C62; value 10uF -> 10u
- C31: renamed from C63; value 22uF -> 22u
- C32: renamed from C64; value 100nF -> 100n
- C34: renamed from C66; value 10uF -> 10u
- renumbered C61 to C29, C65 to C33, U16 to U6
Changed lines of the file:
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@@
 		(dnp no)
 		(fields_autoplaced yes)
-		(property "Reference" "C62"
+		(property "Reference" "C30"
 			(at 187.96 100.3299 0)
 			(effects
@@
 			)
 		)
-		(property "Value" "10uF"
+		(property "Value" "10u"
 			(at 187.96 102.8699 0)
 			(effects
@@
 		(dnp no)
 		(fields_autoplaced yes)
-		(property "Reference" "C63"
+		(property "Reference" "C31"
 			(at 96.52 107.9499 0)
 			(effects
@@
 			)
 		)
-		(property "Value" "22uF"
+		(property "Value" "22u"
 			(at 96.52 110.4899 0)
 			(effects
@@
 		(dnp no)
 		(fields_autoplaced yes)
-		(property "Reference" "U16"
+		(property "Reference" "U6"
 			(at 147.32 86.36 0)
 			(effects
@@
 		(dnp yes)
 		(fields_autoplaced yes)
-		(property "Reference" "C61"
+		(property "Reference" "C29"
 			(at 173.99 100.3299 0)
 			(effects
@@
 		(dnp yes)
 		(fields_autoplaced yes)
-		(property "Reference" "C65"
+		(property "Reference" "C33"
 			(at 173.99 107.9499 0)
 			(effects
@@
 		(dnp no)
 		(fields_autoplaced yes)
-		(property "Reference" "C66"
+		(property "Reference" "C34"
 			(at 187.96 107.9499 0)
 			(effects
@@
 			)
 		)
-		(property "Value" "10uF"
+		(property "Value" "10u"
 			(at 187.96 110.4899 0)
 			(effects
@@
 		(dnp no)
 		(fields_autoplaced yes)
-		(property "Reference" "C64"
+		(property "Reference" "C32"
 			(at 115.57 107.9499 0)
 			(effects
@@
 			)
 		)
-		(property "Value" "100nF"
+		(property "Value" "100n"
 			(at 115.57 110.4899 0)
 			(effects

Commit message: cleaning up common sheets and projects. prepare for removal of legacy path links
Parts:
- renumbered C29 to C1, C30 to C2, C31 to C3, C32 to C4, C33 to C5, C34 to C6, U6 to U1
Changed lines of the file:
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@@
 		(dnp no)
 		(fields_autoplaced yes)
-		(property "Reference" "C30"
+		(property "Reference" "C2"
 			(at 187.96 100.3299 0)
 			(effects
@@
 		(dnp no)
 		(fields_autoplaced yes)
-		(property "Reference" "C31"
+		(property "Reference" "C3"
 			(at 96.52 107.9499 0)
 			(effects
@@
 		(dnp no)
 		(fields_autoplaced yes)
-		(property "Reference" "U6"
+		(property "Reference" "U1"
 			(at 147.32 86.36 0)
 			(effects
@@
 		(dnp yes)
 		(fields_autoplaced yes)
-		(property "Reference" "C29"
+		(property "Reference" "C1"
 			(at 173.99 100.3299 0)
 			(effects
@@
 		(dnp yes)
 		(fields_autoplaced yes)
-		(property "Reference" "C33"
+		(property "Reference" "C5"
 			(at 173.99 107.9499 0)
 			(effects
@@
 		(dnp no)
 		(fields_autoplaced yes)
-		(property "Reference" "C34"
+		(property "Reference" "C6"
 			(at 187.96 107.9499 0)
 			(effects
@@
 		(dnp no)
 		(fields_autoplaced yes)
-		(property "Reference" "C32"
+		(property "Reference" "C4"
 			(at 115.57 107.9499 0)
 			(effects
