File: common/sheets/dual_switch.kicad_sch (KiCad schematic)
At the start: 7 parts, among them U1 TPS22968QDMGRQ1

Commit message: add headers on sci board to accept camera hats
Parts:
- C44: renamed from C1; now fitted
- C48: renamed from C5; now fitted
- renumbered C2 to C45, C3 to C46, C4 to C47, C6 to C49, U1 to U6
Changed lines of the file:
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@@
 		(dnp no)
 		(fields_autoplaced yes)
-		(property "Reference" "C2"
+		(property "Reference" "C45"
 			(at 187.96 100.3299 0)
 			(effects
@@
 				)
 			)
-			(project "sci_board_wo_switches"
+			(project "sci_board_with_hat"
 				(path "/b4b2c88d-f6cd-4e60-862d-e21f68728580/bffa887c-2d4a-4897-aa07-de3665bc885a/0653e279-5ac5-4fd5-819c-e8ef4edad0cf"
 					(reference "C45")
@@
 				)
 				(path "/b4b2c88d-f6cd-4e60-862d-e21f68728580/bffa887c-2d4a-4897-aa07-de3665bc885a/a96e8afd-8b3c-4e12-820c-86caa1a14769"
-					(reference "C76")
+					(reference "C83")
 					(unit 1)
 				)
@@
 		(dnp no)
 		(fields_autoplaced yes)
-		(property "Reference" "C3"
+		(property "Reference" "C46"
 			(at 96.52 107.9499 0)
 			(effects
@@
 				)
 			)
-			(project "sci_board_wo_switches"
+			(project "sci_board_with_hat"
 				(path "/b4b2c88d-f6cd-4e60-862d-e21f68728580/bffa887c-2d4a-4897-aa07-de3665bc885a/0653e279-5ac5-4fd5-819c-e8ef4edad0cf"
 					(reference "C46")
@@
 				)
 				(path "/b4b2c88d-f6cd-4e60-862d-e21f68728580/bffa887c-2d4a-4897-aa07-de3665bc885a/a96e8afd-8b3c-4e12-820c-86caa1a14769"
-					(reference "C77")
+					(reference "C84")
 					(unit 1)
 				)
@@
 		(dnp no)
 		(fields_autoplaced yes)
-		(property "Reference" "U1"
+		(property "Reference" "U6"
 			(at 147.32 86.36 0)
 			(effects
@@
 				)
 			)
-			(project "sci_board_wo_switches"
+			(project "sci_board_with_hat"
 				(path "/b4b2c88d-f6cd-4e60-862d-e21f68728580/bffa887c-2d4a-4897-aa07-de3665bc885a/0653e279-5ac5-4fd5-819c-e8ef4edad0cf"
 					(reference "U6")
@@
 				)
 				(path "/b4b2c88d-f6cd-4e60-862d-e21f68728580/bffa887c-2d4a-4897-aa07-de3665bc885a/a96e8afd-8b3c-4e12-820c-86caa1a14769"
-					(reference "U18")
+					(reference "U19")
 					(unit 1)
 				)
@@
 		(in_bom yes)
 		(on_board yes)
-		(dnp yes)
+		(dnp no)
 		(fields_autoplaced yes)
-		(property "Reference" "C1"
+		(property "Reference" "C44"
 			(at 173.99 100.3299 0)
 			(effects
@@
 				)
 			)
-			(project "sci_board_wo_switches"
+			(project "sci_board_with_hat"
 				(path "/b4b2c88d-f6cd-4e60-862d-e21f68728580/bffa887c-2d4a-4897-aa07-de3665bc885a/0653e279-5ac5-4fd5-819c-e8ef4edad0cf"
 					(reference "C44")
@@
 				)
 				(path "/b4b2c88d-f6cd-4e60-862d-e21f68728580/bffa887c-2d4a-4897-aa07-de3665bc885a/a96e8afd-8b3c-4e12-820c-86caa1a14769"
-					(reference "C75")
+					(reference "C82")
 					(unit 1)
 				)
@@
 		(in_bom yes)
 		(on_board yes)
-		(dnp yes)
+		(dnp no)
 		(fields_autoplaced yes)
-		(property "Reference" "C5"
+		(property "Reference" "C48"
 			(at 173.99 107.9499 0)
 			(effects
@@
 				)
 			)
-			(project "sci_board_wo_switches"
+			(project "sci_board_with_hat"
 				(path "/b4b2c88d-f6cd-4e60-862d-e21f68728580/bffa887c-2d4a-4897-aa07-de3665bc885a/0653e279-5ac5-4fd5-819c-e8ef4edad0cf"
 					(reference "C48")
@@
 				)
 				(path "/b4b2c88d-f6cd-4e60-862d-e21f68728580/bffa887c-2d4a-4897-aa07-de3665bc885a/a96e8afd-8b3c-4e12-820c-86caa1a14769"
-					(reference "C79")
+					(reference "C86")
 					(unit 1)
 				)
@@
 		(dnp no)
 		(fields_autoplaced yes)
-		(property "Reference" "C6"
+		(property "Reference" "C49"
 			(at 187.96 107.9499 0)
 			(effects
@@
 				)
 			)
-			(project "sci_board_wo_switches"
+			(project "sci_board_with_hat"
 				(path "/b4b2c88d-f6cd-4e60-862d-e21f68728580/bffa887c-2d4a-4897-aa07-de3665bc885a/0653e279-5ac5-4fd5-819c-e8ef4edad0cf"
 					(reference "C49")
@@
 				)
 				(path "/b4b2c88d-f6cd-4e60-862d-e21f68728580/bffa887c-2d4a-4897-aa07-de3665bc885a/a96e8afd-8b3c-4e12-820c-86caa1a14769"
-					(reference "C80")
+					(reference "C87")
 					(unit 1)
 				)
@@
 		(dnp no)
 		(fields_autoplaced yes)
-		(property "Reference" "C4"
+		(property "Reference" "C47"
 			(at 115.57 107.9499 0)
 			(effects
@@
 				)
 			)
-			(project "sci_board_wo_switches"
+			(project "sci_board_with_hat"
 				(path "/b4b2c88d-f6cd-4e60-862d-e21f68728580/bffa887c-2d4a-4897-aa07-de3665bc885a/0653e279-5ac5-4fd5-819c-e8ef4edad0cf"
 					(reference "C47")
@@
 				)
 				(path "/b4b2c88d-f6cd-4e60-862d-e21f68728580/bffa887c-2d4a-4897-aa07-de3665bc885a/a96e8afd-8b3c-4e12-820c-86caa1a14769"
-					(reference "C78")
-					(unit 1)
-				)
+					(reference "C85")
+					(unit 1)
+				)
