File: common/sheets/i2c_power_switch.kicad_sch (KiCad schematic)
At the start: 11 parts, among them U25 MCP23008T-E/SS, U26 INA226AIDGSR, U27 INA226AIDGSR

Commit message: auxio_board: leverage more IO on aux board
Connections:
- net 3V3: now also R32.1, U26.10 (IN+); no longer C100.1, R33.1, U27.10 (IN+), U27.6 (VS)
- net 3V3_CORE: now also C100.1, U27.6 (VS); no longer R32.1, U26.10 (IN+)
- net VBUS: now also R33.1, U27.10 (IN+); no longer C102.1, R33.2, U27.8 (VBUS), U27.9 (IN-)
- net 3V3_STM_CORE renamed 3V3_METERED
- new net VBUS_METERED: C102.1, R33.2, U27.8 (VBUS), U27.9 (IN-)
Changed lines of the file:
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@@
 		)
 	)
-	(label "VBUS"
+	(label "VBUS_METERED"
 		(at 205.74 105.41 180)
 		(effects
@@
 		)
 	)
+	(label "3V3_METERED"
+		(at 205.74 70.485 180)
+		(effects
+			(font
+				(size 1.27 1.27)
+			)
+			(justify right bottom)
+		)
+	)
 	(label "ENABLE5"
 		(at 95.25 39.37 0)
@@
 		)
 	)
-	(label "VBUS"
+	(label "VBUS_METERED"
 		(at 205.105 136.525 180)
 		(effects
@@
 		)
 	)
-	(label "VBUS"
+	(label "VBUS_METERED"
 		(at 205.105 132.715 180)
 		(effects
@@
 		)
 	)
+	(label "3V3_METERED"
+		(at 205.74 74.295 180)
+		(effects
+			(font
+				(size 1.27 1.27)
+			)
+			(justify right bottom)
+		)
+	)
 	(label "ENABLE3"
 		(at 95.25 44.45 0)
@@
 		)
 	)
-	(label "VBUS"
+	(label "VBUS_METERED"
 		(at 205.74 100.965 180)
 		(effects
@@
 		)
 	)
-	(label "VBUS"
+	(label "3V3_METERED"
+		(at 206.375 43.18 180)
+		(effects
+			(font
+				(size 1.27 1.27)
+			)
+			(justify right bottom)
+		)
+	)
+	(label "VBUS_METERED"
 		(at 114.935 91.44 180)
 		(effects
@@
 			)
 			(justify right bottom)
+		)
+	)
+	(label "3V3_METERED"
+		(at 43.18 90.805 180)
+		(effects
+			(font
+				(size 1.27 1.27)
+			)
+			(justify right bottom)
+		)
+	)
+	(label "3V3_METERED"
+		(at 53.34 115.57 0)
+		(effects
+			(font
+				(size 1.27 1.27)
+			)
+			(justify left bottom)
 		)
 	)
@@
 		)
 	)
-	(label "VBUS"
+	(label "VBUS_METERED"
 		(at 125.095 116.205 0)
 		(effects
@@
 			)
 			(justify left bottom)
+		)
+	)
+	(label "3V3_METERED"
+		(at 206.375 39.37 180)
+		(effects
+			(font
+				(size 1.27 1.27)
+			)
+			(justify right bottom)
 		)
 	)
@@
 		)
 	)
-	(hierarchical_label "3V3_STM_CORE"
-		(shape input)
-		(at 43.18 90.805 180)
-		(effects
-			(font
-				(size 1.27 1.27)
-			)
-			(justify right)
-		)
-	)
 	(hierarchical_label "GND"
 		(shape input)
@@
 		)
 	)
-	(hierarchical_label "3V3_STM_CORE"
-		(shape input)
-		(at 206.375 43.18 180)
-		(effects
-			(font
-				(size 1.27 1.27)
-			)
-			(justify right)
-		)
-	)
 	(hierarchical_label "VOUT7"
 		(shape output)
@@
 		)
 	)
+	(hierarchical_label "3V3"
+		(shape input)
+		(at 43.18 93.345 180)
+		(effects
+			(font
+				(size 1.27 1.27)
+			)
+			(justify right)
+		)
+	)
+	(hierarchical_label "VOUT5"
+		(shape output)
+		(at 224.79 92.075 0)
+		(effects
+			(font
+				(size 1.27 1.27)
+			)
+			(justify left)
+		)
+	)
+	(hierarchical_label "SCL"
+		(shape input)
+		(at 127 106.68 180)
+		(effects
+			(font
+				(size 1.27 1.27)
+			)
+			(justify right)
+		)
+	)
+	(hierarchical_label "VOUT3"
+		(shape output)
+		(at 224.79 60.96 0)
+		(effects
+			(font
+				(size 1.27 1.27)
+			)
+			(justify left)
+		)
+	)
+	(hierarchical_label "VOUT2"
+		(shape output)
+		(at 224.79 70.485 0)
+		(effects
+			(font
+				(size 1.27 1.27)
+			)
+			(justify left)
+		)
+	)
+	(hierarchical_label "INT"
+		(shape output)
+		(at 111.76 45.085 270)
+		(effects
+			(font
+				(size 1.27 1.27)
+			)
+			(justify right)
+		)
+	)
+	(hierarchical_label "PM_A10"
+		(shape input)
+		(at 55.245 85.725 180)
+		(effects
+			(font
+				(size 1.27 1.27)
+			)
+			(justify right)
+		)
+	)
+	(hierarchical_label "GND"
+		(shape input)
+		(at 64.77 52.07 180)
+		(effects
+			(font
+				(size 1.27 1.27)
+			)
+			(justify right)
+		)
+	)
+	(hierarchical_label "GND"
+		(shape input)
+		(at 224.79 74.295 0)
+		(effects
+			(font
+				(size 1.27 1.27)
+			)
+			(justify left)
+		)
+	)
+	(hierarchical_label "VBUS"
+		(shape input)
+		(at 114.935 93.98 180)
+		(effects
+			(font
+				(size 1.27 1.27)
+			)
+			(justify right)
+		)
+	)
 	(hierarchical_label "3V3_CORE"
 		(shape input)
-		(at 43.18 93.345 180)
-		(effects
-			(font
-				(size 1.27 1.27)
-			)
-			(justify right)
-		)
-	)
-	(hierarchical_label "VOUT5"
-		(shape output)
-		(at 224.79 92.075 0)
-		(effects
-			(font
-				(size 1.27 1.27)
-			)
-			(justify left)
-		)
-	)
-	(hierarchical_label "SCL"
-		(shape input)
-		(at 127 106.68 180)
-		(effects
-			(font
-				(size 1.27 1.27)
-			)
-			(justify right)
-		)
-	)
-	(hierarchical_label "VOUT3"
-		(shape output)
-		(at 224.79 60.96 0)
-		(effects
-			(font
-				(size 1.27 1.27)
-			)
-			(justify left)
-		)
-	)
-	(hierarchical_label "3V3_STM_CORE"
-		(shape input)
-		(at 205.74 74.295 180)
-		(effects
-			(font
-				(size 1.27 1.27)
-			)
-			(justify right)
-		)
-	)
-	(hierarchical_label "VOUT2"
-		(shape output)
-		(at 224.79 70.485 0)
+		(at 98.425 80.645 90)
 		(effects
 			(font
@@
 	(hierarchical_label "INT"
 		(shape output)
-		(at 111.76 45.085 270)
-		(effects
-			(font
-				(size 1.27 1.27)
-			)
-			(justify right)
-		)
-	)
-	(hierarchical_label "PM_A10"
-		(shape input)
-		(at 55.245 85.725 180)
-		(effects
-			(font
-				(size 1.27 1.27)
-			)
-			(justify right)
-		)
-	)
-	(hierarchical_label "GND"
-		(shape input)
-		(at 64.77 52.07 180)
-		(effects
-			(font
-				(size 1.27 1.27)
-			)
-			(justify right)
-		)
-	)
-	(hierarchical_label "3V3_STM_CORE"
-		(shape input)
-		(at 206.375 39.37 180)
-		(effects
-			(font
-				(size 1.27 1.27)
-			)
-			(justify right)
-		)
-	)
-	(hierarchical_label "GND"
-		(shape input)
-		(at 224.79 74.295 0)
-		(effects
-			(font
-				(size 1.27 1.27)
-			)
-			(justify left)
-		)
-	)
-	(hierarchical_label "3V3_STM_CORE"
-		(shape output)
-		(at 53.34 115.57 0)
-		(effects
-			(font
-				(size 1.27 1.27)
-			)
-			(justify left)
-		)
-	)
-	(hierarchical_label "3V3"
-		(shape input)
-		(at 114.935 93.98 180)
-		(effects
-			(font
-				(size 1.27 1.27)
-			)
-			(justify right)
-		)
-	)
-	(hierarchical_label "3V3_CORE"
-		(shape input)
-		(at 98.425 80.645 90)
-		(effects
-			(font
-				(size 1.27 1.27)
-			)
-			(justify left)
-		)
-	)
-	(hierarchical_label "INT"
-		(shape output)
 		(at 90.805 88.265 0)
 		(effects
@@
 			)
 			(justify left)
-		)
-	)
-	(hierarchical_label "3V3_STM_CORE"
-		(shape input)
-		(at 205.74 70.485 180)
-		(effects
-			(font
-				(size 1.27 1.27)
-			)
-			(justify right)
 		)
 	)
@@
 		)
 	)
-	(hierarchical_label "3V3"
+	(hierarchical_label "3V3_CORE"
 		(shape input)
 		(at 170.18 81.28 90)
