File: common/sheets/i2c_power_switches_3v_sch.kicad_sch (KiCad schematic)
At the start: 7 parts, among them U28 MCP23008T-E/SS, U29 INA226

Commit message: auxio_board: leverage more IO on aux board
Changed lines of the file:
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@@
+		)
+	)
+	(label "ENABLE_1"
+		(at 136.525 43.18 180)
+		(effects
+			(font
+				(size 1.27 1.27)
+			)
+			(justify right bottom)
+		)
+	)
+	(label "ENABLE_5"
+		(at 83.185 42.545 0)
+		(effects
+			(font
+				(size 1.27 1.27)
+			)
+			(justify left bottom)
+		)
+	)
+	(label "ENABLE_3"
+		(at 83.185 47.625 0)
+		(effects
+			(font
+				(size 1.27 1.27)
+			)
+			(justify left bottom)
 		)
 	)
@@
 		)
 	)
+	(label "ENABLE_3"
+		(at 136.525 72.39 180)
+		(effects
+			(font
+				(size 1.27 1.27)
+			)
+			(justify right bottom)
+		)
+	)
+	(label "ENABLE_6"
+		(at 83.185 40.005 0)
+		(effects
+			(font
+				(size 1.27 1.27)
+			)
+			(justify left bottom)
+		)
+	)
+	(label "ENABLE_7"
+		(at 83.185 37.465 0)
+		(effects
+			(font
+				(size 1.27 1.27)
+			)
+			(justify left bottom)
+		)
+	)
 	(label "VBUS"
 		(at 136.525 78.74 180)
@@
 		)
 	)
+	(label "ENABLE_0"
+		(at 136.525 39.37 180)
+		(effects
+			(font
+				(size 1.27 1.27)
+			)
+			(justify right bottom)
+		)
+	)
+	(label "ENABLE_4"
+		(at 83.185 45.085 0)
+		(effects
+			(font
+				(size 1.27 1.27)
+			)
+			(justify left bottom)
+		)
+	)
+	(label "ENABLE_7"
+		(at 193.675 73.025 180)
+		(effects
+			(font
+				(size 1.27 1.27)
+			)
+			(justify right bottom)
+		)
+	)
 	(label "VBUS"
 		(at 41.275 118.745 0)
@@
 		)
 	)
+	(label "ENABLE_5"
+		(at 193.675 43.18 180)
+		(effects
+			(font
+				(size 1.27 1.27)
+			)
+			(justify right bottom)
+		)
+	)
 	(label "VBUS"
 		(at 31.115 93.98 180)
@@
 		)
 	)
+	(label "ENABLE_1"
+		(at 83.185 52.705 0)
+		(effects
+			(font
+				(size 1.27 1.27)
+			)
+			(justify left bottom)
+		)
+	)
 	(label "VBUS"
 		(at 193.675 48.895 180)
@@
 		)
 	)
+	(label "ENABLE_2"
+		(at 83.185 50.165 0)
+		(effects
+			(font
+				(size 1.27 1.27)
+			)
+			(justify left bottom)
+		)
+	)
+	(label "ENABLE_4"
+		(at 193.675 39.37 180)
+		(effects
+			(font
+				(size 1.27 1.27)
+			)
+			(justify right bottom)
+		)
+	)
 	(label "VBUS"
 		(at 193.675 82.55 180)
@@
 		)
 	)
+	(label "ENABLE_0"
+		(at 83.185 55.245 0)
+		(effects
+			(font
+				(size 1.27 1.27)
+			)
+			(justify left bottom)
+		)
+	)
 	(label "VBUS"
 		(at 136.525 48.895 180)
@@
 	(label "VBUS"
 		(at 136.525 52.705 180)
+		(effects
+			(font
+				(size 1.27 1.27)
+			)
+			(justify right bottom)
+		)
+	)
+	(label "ENABLE_2"
+		(at 136.525 69.215 180)
+		(effects
+			(font
+				(size 1.27 1.27)
+			)
+			(justify right bottom)
+		)
+	)
+	(label "ENABLE_6"
+		(at 193.675 69.215 180)
 		(effects
 			(font
@@
 		)
 	)
-	(hierarchical_label "VOUT_B"
+	(hierarchical_label "VOUT_1"
 		(shape output)
 		(at 155.575 48.895 0)
@@
 		)
 	)
-	(hierarchical_label "ENABLE_5"
-		(shape output)
-		(at 83.185 42.545 0)
-		(effects
-			(font
-				(size 1.27 1.27)
-			)
-			(justify left)
-		)
-	)
 	(hierarchical_label "INT"
 		(shape output)
@@
 		)
 	)
-	(hierarchical_label "VOUT_C"
+	(hierarchical_label "VOUT_2"
 		(shape output)
 		(at 155.575 69.215 0)
@@
 		)
 	)
-	(hierarchical_label "ENABLE_1"
-		(shape output)
-		(at 83.185 52.705 0)
-		(effects
-			(font
-				(size 1.27 1.27)
-			)
-			(justify left)
-		)
-	)
 	(hierarchical_label "VIN"
 		(shape input)
@@
 			)
 			(justify left)
-		)
-	)
-	(hierarchical_label "ENABLE_6"
-		(shape output)
-		(at 83.185 40.005 0)
-		(effects
-			(font
-				(size 1.27 1.27)
-			)
-			(justify left)
-		)
-	)
-	(hierarchical_label "ENABLE_3"
-		(shape output)
-		(at 83.185 47.625 0)
-		(effects
-			(font
-				(size 1.27 1.27)
-			)
-			(justify left)
-		)
-	)
-	(hierarchical_label "ENABLE_2"
-		(shape output)
-		(at 83.185 50.165 0)
-		(effects
-			(font
-				(size 1.27 1.27)
-			)
-			(justify left)
-		)
-	)
-	(hierarchical_label "ENABLE_H"
-		(shape input)
-		(at 136.525 72.39 180)
-		(effects
-			(font
-				(size 1.27 1.27)
-			)
-			(justify right)
 		)
 	)
@@
 		)
 	)
-	(hierarchical_label "VOUT_E"
+	(hierarchical_label "VOUT_4"
 		(shape output)
 		(at 212.725 39.37 0)
@@
 		)
 	)
-	(hierarchical_label "ENABLE_G"
-		(shape input)
-		(at 136.525 69.215 180)
-		(effects
-			(font
-				(size 1.27 1.27)
-			)
-			(justify right)
-		)
-	)
-	(hierarchical_label "VOUT_H"
+	(hierarchical_label "VOUT_7"
 		(shape output)
 		(at 212.725 78.74 0)
@@
 		)
 	)
-	(hierarchical_label "VOUT_G"
+	(hierarchical_label "VOUT_6"
 		(shape output)
 		(at 212.725 69.215 0)
@@
 		)
 	)
-	(hierarchical_label "ENABLE_F"
-		(shape input)
-		(at 136.525 43.18 180)
-		(effects
-			(font
-				(size 1.27 1.27)
-			)
-			(justify right)
-		)
-	)
-	(hierarchical_label "VOUT_A"
+	(hierarchical_label "VOUT_0"
 		(shape output)
 		(at 155.575 39.37 0)
@@
 		)
 	)
-	(hierarchical_label "ENABLE_4"
-		(shape output)
-		(at 83.185 45.085 0)
-		(effects
-			(font
-				(size 1.27 1.27)
-			)
-			(justify left)
-		)
-	)
-	(hierarchical_label "VOUT_D"
+	(hierarchical_label "VOUT_3"
 		(shape output)
 		(at 155.575 78.74 0)
@@
 		)
 	)
-	(hierarchical_label "ENABLE_E"
-		(shape input)
-		(at 136.525 39.37 180)
-		(effects
-			(font
-				(size 1.27 1.27)
-			)
-			(justify right)
-		)
-	)
 	(hierarchical_label "GND"
 		(shape input)
@@
 		)
 	)
-	(hierarchical_label "ENABLE_7"
-		(shape output)
-		(at 83.185 37.465 0)
-		(effects
-			(font
-				(size 1.27 1.27)
-			)
-			(justify left)
-		)
-	)
-	(hierarchical_label "ENABLE_A"
-		(shape input)
-		(at 193.675 39.37 180)
-		(effects
-			(font
-				(size 1.27 1.27)
-			)
-			(justify right)
-		)
-	)
 	(hierarchical_label "GND"
 		(shape output)
@@
 		)
 	)
-	(hierarchical_label "ENABLE_D"
-		(shape input)
-		(at 193.675 73.025 180)
-		(effects
-			(font
-				(size 1.27 1.27)
-			)
-			(justify right)
-		)
-	)
-	(hierarchical_label "VOUT_F"
+	(hierarchical_label "VOUT_5"
 		(shape output)
 		(at 212.725 48.895 0)
@@
 		)
 	)
-	(hierarchical_label "ENABLE_B"
-		(shape input)
-		(at 193.675 43.18 180)
-		(effects
-			(font
-				(size 1.27 1.27)
-			)
-			(justify right)
-		)
-	)
-	(hierarchical_label "ENABLE_C"
-		(shape input)
-		(at 193.675 69.215 180)
-		(effects
-			(font
-				(size 1.27 1.27)
-			)
-			(justify right)
-		)
-	)
-	(hierarchical_label "ENABLE_0"
-		(shape output)
-		(at 83.185 55.245 0)
-		(effects
-			(font
-				(size 1.27 1.27)
-			)
-			(justify left)
-		)
-	)
